File: gdp/gdp.kicad_sch (KiCad schematic)
At the start: 20 parts, among them IC11 7406, IC3 LM393, IC8 74LS245, J3 Conn_01x32, J4 Conn_01x32

Commit message: Adds more pages, adds schema revisions
Parts:
- removed IC11: 7406, symbol 74xx_IEEE:7406
- removed IC3: LM393, symbol Comparator:LM393
- removed IC8: 74LS245, symbol 74xx_IEEE:74LS245
- removed J3, J4: Conn_01x32, symbol Connector_Generic:Conn_01x32
- removed R10, R11, R1?, R8, R9: 10K, symbol Device:R
- removed R13: 3K3, symbol Device:R
- removed R1?: 2K2, symbol Device:R
- removed R1?, R21: 330R, symbol Device:R
- removed SH1, SH2, SH3: SCHALT, symbol Switch:SW_DPST_x2
- removed ST1: 6PINCON, symbol Connector_Generic:Conn_01x06
- removed ST2: ST60F01, symbol Connector_Generic:Conn_01x06
- removed ST3: MODU2-10, symbol Connector_Generic:Conn_01x10
Connections:
- no-connect marks 5 -> 0
Other:
- added sheet 1 (1.kicad_sch)
- added sheet 2 (2.kicad_sch)

Commit message: Adds pages 4, 7, 10 (still WIP)
Other:
- added sheet 10 (10.kicad_sch)
- added sheet 3 (3.kicad_sch)
- added sheet 4 (4.kicad_sch)
- added sheet 5 (5.kicad_sch)
- added sheet 6 (6.kicad_sch)
- added sheet 7 (7.kicad_sch)
- added sheet 8 (8.kicad_sch)
- added sheet 9 (9.kicad_sch)
Changed lines of the file:
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@@
 (kicad_sch (version 20230121) (generator eeschema)
   (paper "A4")
+  (sheet (at 67.31 24.765) (size 33.655 13.97) (fields_autoplaced)
+    (stroke (width 0.1524) (type solid))
+    (fill (color 0 0 0 0.0000))
+    (property "Sheetname" "8" (at 67.31 24.0534 0)
+      (effects (font (size 1.27 1.27)) (justify left bottom))
+    )
+    (property "Sheetfile" "8.kicad_sch" (at 67.31 39.3196 0)
+      (effects (font (size 1.27 1.27)) (justify left top))
+    )
+    (instances
+      (project "gdp"
+        (path "/95aff260-2720-4733-a81d-a7a2136fdd14" (page "9"))
+      )
+    )
+  )
+  (sheet (at 73.66 49.53) (size 33.02 13.97) (fields_autoplaced)
+    (stroke (width 0.1524) (type solid))
+    (fill (color 0 0 0 0.0000))
+    (property "Sheetname" "9" (at 73.66 48.8184 0)
+      (effects (font (size 1.27 1.27)) (justify left bottom))
+    )
+    (property "Sheetfile" "9.kicad_sch" (at 73.66 64.0846 0)
+      (effects (font (size 1.27 1.27)) (justify left top))
+    )
+    (instances
+      (project "gdp"
+        (path "/95aff260-2720-4733-a81d-a7a2136fdd14" (page "10"))
+      )
+    )
+  )
+  (sheet (at 24.13 172.72) (size 37.465 14.605) (fields_autoplaced)
+    (stroke (width 0.1524) (type solid))
+    (fill (color 0 0 0 0.0000))
+    (property "Sheetname" "7" (at 24.13 172.0084 0)
+      (effects (font (size 1.27 1.27)) (justify left bottom))
+    )
+    (property "Sheetfile" "7.kicad_sch" (at 24.13 187.9096 0)
+      (effects (font (size 1.27 1.27)) (justify left top))
+    )
+    (instances
+      (project "gdp"
+        (path "/95aff260-2720-4733-a81d-a7a2136fdd14" (page "8"))
+      )
+    )
+  )
+  (sheet (at 25.4 74.295) (size 37.465 15.24) (fields_autoplaced)
+    (stroke (width 0.1524) (type solid))
+    (fill (color 0 0 0 0.0000))
+    (property "Sheetname" "3" (at 25.4 73.5834 0)
+      (effects (font (size 1.27 1.27)) (justify left bottom))
+    )
+    (property "Sheetfile" "3.kicad_sch" (at 25.4 90.1196 0)
+      (effects (font (size 1.27 1.27)) (justify left top))
+    )
+    (instances
+      (project "gdp"
+        (path "/95aff260-2720-4733-a81d-a7a2136fdd14" (page "4"))
+      )
+    )
+  )
+  (sheet (at 67.945 75.565) (size 37.465 12.7) (fields_autoplaced)
+    (stroke (width 0.1524) (type solid))
+    (fill (color 0 0 0 0.0000))
+    (property "Sheetname" "10" (at 67.945 74.8534 0)
+      (effects (font (size 1.27 1.27)) (justify left bottom))
+    )
+    (property "Sheetfile" "10.kicad_sch" (at 67.945 88.8496 0)
+      (effects (font (size 1.27 1.27)) (justify left top))
+    )
+    (instances
+      (project "gdp"
+        (path "/95aff260-2720-4733-a81d-a7a2136fdd14" (page "11"))
+      )
+    )
+  )
+  (sheet (at 24.765 126.365) (size 36.83 14.605) (fields_autoplaced)
+    (stroke (width 0.1524) (type solid))
+    (fill (color 0 0 0 0.0000))
+    (property "Sheetname" "5" (at 24.765 125.6534 0)
+      (effects (font (size 1.27 1.27)) (justify left bottom))
+    )
+    (property "Sheetfile" "5.kicad_sch" (at 24.765 141.5546 0)
+      (effects (font (size 1.27 1.27)) (justify left top))
+    )
+    (instances
+      (project "gdp"
+        (path "/95aff260-2720-4733-a81d-a7a2136fdd14" (page "6"))
+      )
+    )
+  )
+  (sheet (at 24.765 150.495) (size 36.195 15.24) (fields_autoplaced)
+    (stroke (width 0.1524) (type solid))
+    (fill (color 0 0 0 0.0000))
+    (property "Sheetname" "6" (at 24.765 149.7834 0)
+      (effects (font (size 1.27 1.27)) (justify left bottom))
+    )
+    (property "Sheetfile" "6.kicad_sch" (at 24.765 166.3196 0)
+      (effects (font (size 1.27 1.27)) (justify left top))
+    )
+    (instances
+      (project "gdp"
+        (path "/95aff260-2720-4733-a81d-a7a2136fdd14" (page "7"))
+      )
+    )
+  )
+  (sheet (at 26.67 100.33) (size 36.83 16.51) (fields_autoplaced)
+    (stroke (width 0.1524) (type solid))
+    (fill (color 0 0 0 0.0000))
+    (property "Sheetname" "4" (at 26.67 99.6184 0)
+      (effects (font (size 1.27 1.27)) (justify left bottom))
+    )
+    (property "Sheetfile" "4.kicad_sch" (at 26.67 117.4246 0)
+      (effects (font (size 1.27 1.27)) (justify left top))
+    )
+    (instances
+      (project "gdp"
+        (path "/95aff260-2720-4733-a81d-a7a2136fdd14" (page "5"))
+      )
+    )
+  )
   (sheet (at 24.765 48.895) (size 36.83 16.51) (fields_autoplaced)
     (stroke (width 0.1524) (type solid))
@@
     (instances
       (project "gdp"
-        (path "/95aff260-2720-4733-a81d-a7a2136fdd14" (page "2"))
+        (path "/95aff260-2720-4733-a81d-a7a2136fdd14" (page "3"))
       )
     )
@@
     (instances
       (project "gdp"
-        (path "/95aff260-2720-4733-a81d-a7a2136fdd14" (page "1"))
+        (path "/95aff260-2720-4733-a81d-a7a2136fdd14" (page "2"))
       )
     )
   )
   (sheet_instances
-    (path "/" (page "0"))
+    (path "/" (page "1"))
   )
 )

Commit message: Fixes sheet sizes
Other:
- added sheet 11 (11.kicad_sch)
- added sheet 12 (12.kicad_sch)
- added sheet 13 (13.kicad_sch)
- added sheet 14 (14.kicad_sch)
- company: (none) -> Oddbit Retro
- title: (none) -> PARTNER GDP
Changed lines of the file:
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@@
 (kicad_sch (version 20230121) (generator eeschema)
   (paper "A4")
-  (sheet (at 67.31 24.765) (size 33.655 13.97) (fields_autoplaced)
+  (title_block
+    (title "PARTNER GDP")
+    (company "Oddbit Retro")
+  )
+  (sheet (at 67.31 151.13) (size 31.75 15.875) (fields_autoplaced)
+    (stroke (width 0.1524) (type solid))
+    (fill (color 0 0 0 0.0000))
+    (property "Sheetname" "13" (at 67.31 150.4184 0)
+      (effects (font (size 1.27 1.27)) (justify left bottom))
+    )
+    (property "Sheetfile" "13.kicad_sch" (at 67.31 167.5896 0)
+      (effects (font (size 1.27 1.27)) (justify left top))
+    )
+    (instances
+      (project "gdp"
+        (path "/95aff260-2720-4733-a81d-a7a2136fdd14" (page "14"))
+      )
+    )
+  )
+  (sheet (at 67.31 24.765) (size 31.75 15.875) (fields_autoplaced)
     (stroke (width 0.1524) (type solid))
     (fill (color 0 0 0 0.0000))
@@
       (effects (font (size 1.27 1.27)) (justify left bottom))
     )
-    (property "Sheetfile" "8.kicad_sch" (at 67.31 39.3196 0)
+    (property "Sheetfile" "8.kicad_sch" (at 67.31 41.3496 0)
       (effects (font (size 1.27 1.27)) (justify left top))
     )
@@
     )
   )
-  (sheet (at 73.66 49.53) (size 33.02 13.97) (fields_autoplaced)
-    (stroke (width 0.1524) (type solid))
-    (fill (color 0 0 0 0.0000))
-    (property "Sheetname" "9" (at 73.66 48.8184 0)
-      (effects (font (size 1.27 1.27)) (justify left bottom))
-    )
-    (property "Sheetfile" "9.kicad_sch" (at 73.66 64.0846 0)
+  (sheet (at 67.31 50.8) (size 31.75 15.875) (fields_autoplaced)
+    (stroke (width 0.1524) (type solid))
+    (fill (color 0 0 0 0.0000))
+    (property "Sheetname" "9" (at 67.31 50.0884 0)
+      (effects (font (size 1.27 1.27)) (justify left bottom))
+    )
+    (property "Sheetfile" "9.kicad_sch" (at 67.31 67.3846 0)
       (effects (font (size 1.27 1.27)) (justify left top))
     )
@@
     )
   )
-  (sheet (at 24.13 172.72) (size 37.465 14.605) (fields_autoplaced)
-    (stroke (width 0.1524) (type solid))
-    (fill (color 0 0 0 0.0000))
-    (property "Sheetname" "7" (at 24.13 172.0084 0)
-      (effects (font (size 1.27 1.27)) (justify left bottom))
-    )
-    (property "Sheetfile" "7.kicad_sch" (at 24.13 187.9096 0)
+  (sheet (at 67.31 125.73) (size 31.75 15.875) (fields_autoplaced)
+    (stroke (width 0.1524) (type solid))
+    (fill (color 0 0 0 0.0000))
+    (property "Sheetname" "12" (at 67.31 125.0184 0)
+      (effects (font (size 1.27 1.27)) (justify left bottom))
+    )
+    (property "Sheetfile" "12.kicad_sch" (at 67.31 142.1896 0)
+      (effects (font (size 1.27 1.27)) (justify left top))
+    )
+    (instances
+      (project "gdp"
+        (path "/95aff260-2720-4733-a81d-a7a2136fdd14" (page "13"))
+      )
+    )
+  )
+  (sheet (at 24.765 172.72) (size 31.75 15.875) (fields_autoplaced)
+    (stroke (width 0.1524) (type solid))
+    (fill (color 0 0 0 0.0000))
+    (property "Sheetname" "7" (at 24.765 172.0084 0)
+      (effects (font (size 1.27 1.27)) (justify left bottom))
+    )
+    (property "Sheetfile" "7.kicad_sch" (at 24.765 189.3046 0)
       (effects (font (size 1.27 1.27)) (justify left top))
     )
@@
     )
   )
-  (sheet (at 25.4 74.295) (size 37.465 15.24) (fields_autoplaced)
-    (stroke (width 0.1524) (type solid))
-    (fill (color 0 0 0 0.0000))
-    (property "Sheetname" "3" (at 25.4 73.5834 0)
-      (effects (font (size 1.27 1.27)) (justify left bottom))
-    )
-    (property "Sheetfile" "3.kicad_sch" (at 25.4 90.1196 0)
+  (sheet (at 24.765 74.295) (size 31.75 15.875) (fields_autoplaced)
+    (stroke (width 0.1524) (type solid))
+    (fill (color 0 0 0 0.0000))
+    (property "Sheetname" "3" (at 24.765 73.5834 0)
+      (effects (font (size 1.27 1.27)) (justify left bottom))
+    )
+    (property "Sheetfile" "3.kicad_sch" (at 24.765 90.8796 0)
       (effects (font (size 1.27 1.27)) (justify left top))
     )
@@
     )
   )
-  (sheet (at 67.945 75.565) (size 37.465 12.7) (fields_autoplaced)
-    (stroke (width 0.1524) (type solid))
-    (fill (color 0 0 0 0.0000))
-    (property "Sheetname" "10" (at 67.945 74.8534 0)
-      (effects (font (size 1.27 1.27)) (justify left bottom))
-    )
-    (property "Sheetfile" "10.kicad_sch" (at 67.945 88.8496 0)
+  (sheet (at 67.31 172.72) (size 31.75 15.875) (fields_autoplaced)
+    (stroke (width 0.1524) (type solid))
+    (fill (color 0 0 0 0.0000))
+    (property "Sheetname" "14" (at 67.31 172.0084 0)
+      (effects (font (size 1.27 1.27)) (justify left bottom))
+    )
+    (property "Sheetfile" "14.kicad_sch" (at 67.31 189.3046 0)
+      (effects (font (size 1.27 1.27)) (justify left top))
+    )
+    (instances
+      (project "gdp"
+        (path "/95aff260-2720-4733-a81d-a7a2136fdd14" (page "15"))
+      )
+    )
+  )
+  (sheet (at 67.31 75.565) (size 31.75 15.875) (fields_autoplaced)
+    (stroke (width 0.1524) (type solid))
+    (fill (color 0 0 0 0.0000))
+    (property "Sheetname" "10" (at 67.31 74.8534 0)
+      (effects (font (size 1.27 1.27)) (justify left bottom))
+    )
+    (property "Sheetfile" "10.kicad_sch" (at 67.31 92.1496 0)
       (effects (font (size 1.27 1.27)) (justify left top))
     )
@@
     )
   )
-  (sheet (at 24.765 126.365) (size 36.83 14.605) (fields_autoplaced)
+  (sheet (at 24.765 126.365) (size 31.75 15.875) (fields_autoplaced)
     (stroke (width 0.1524) (type solid))
     (fill (color 0 0 0 0.0000))
@@
       (effects (font (size 1.27 1.27)) (justify left bottom))
     )
-    (property "Sheetfile" "5.kicad_sch" (at 24.765 141.5546 0)
+    (property "Sheetfile" "5.kicad_sch" (at 24.765 142.9496 0)
       (effects (font (size 1.27 1.27)) (justify left top))
     )
@@
     )
   )
-  (sheet (at 24.765 150.495) (size 36.195 15.24) (fields_autoplaced)
+  (sheet (at 24.765 150.495) (size 31.75 15.875) (fields_autoplaced)
     (stroke (width 0.1524) (type solid))
     (fill (color 0 0 0 0.0000))
@@
       (effects (font (size 1.27 1.27)) (justify left bottom))
     )
-    (property "Sheetfile" "6.kicad_sch" (at 24.765 166.3196 0)
+    (property "Sheetfile" "6.kicad_sch" (at 24.765 167.0796 0)
       (effects (font (size 1.27 1.27)) (justify left top))
     )
@@
     )
   )
-  (sheet (at 26.67 100.33) (size 36.83 16.51) (fields_autoplaced)
-    (stroke (width 0.1524) (type solid))
-    (fill (color 0 0 0 0.0000))
-    (property "Sheetname" "4" (at 26.67 99.6184 0)
-      (effects (font (size 1.27 1.27)) (justify left bottom))
-    )
-    (property "Sheetfile" "4.kicad_sch" (at 26.67 117.4246 0)
+  (sheet (at 67.31 100.33) (size 31.75 15.875) (fields_autoplaced)
+    (stroke (width 0.1524) (type solid))
+    (fill (color 0 0 0 0.0000))
+    (property "Sheetname" "11" (at 67.31 99.6184 0)
+      (effects (font (size 1.27 1.27)) (justify left bottom))
+    )
+    (property "Sheetfile" "11.kicad_sch" (at 67.31 116.9146 0)
+      (effects (font (size 1.27 1.27)) (justify left top))
+    )
+    (instances
+      (project "gdp"
+        (path "/95aff260-2720-4733-a81d-a7a2136fdd14" (page "12"))
+      )
+    )
+  )
+  (sheet (at 24.765 100.33) (size 31.75 15.875) (fields_autoplaced)
+    (stroke (width 0.1524) (type solid))
+    (fill (color 0 0 0 0.0000))
+    (property "Sheetname" "4" (at 24.765 99.6184 0)
+      (effects (font (size 1.27 1.27)) (justify left bottom))
+    )
+    (property "Sheetfile" "4.kicad_sch" (at 24.765 116.9146 0)
       (effects (font (size 1.27 1.27)) (justify left top))
     )
@@
     )
   )
-  (sheet (at 24.765 48.895) (size 36.83 16.51) (fields_autoplaced)
+  (sheet (at 24.765 48.895) (size 31.75 15.875) (fields_autoplaced)
     (stroke (width 0.1524) (type solid))
     (fill (color 0 0 0 0.0000))
@@
       (effects (font (size 1.27 1.27)) (justify left bottom))
     )
-    (property "Sheetfile" "2.kicad_sch" (at 24.765 65.9896 0)
+    (property "Sheetfile" "2.kicad_sch" (at 24.765 65.4796 0)
       (effects (font (size 1.27 1.27)) (justify left top))
     )
@@
     )
   )
-  (sheet (at 26.035 23.495) (size 35.56 15.875) (fields_autoplaced)
-    (stroke (width 0.1524) (type solid))
-    (fill (color 0 0 0 0.0000))
-    (property "Sheetname" "1" (at 26.035 22.7834 0)
-      (effects (font (size 1.27 1.27)) (justify left bottom))
-    )
-    (property "Sheetfile" "1.kicad_sch" (at 26.035 39.9546 0)
-      (effects (font (size 1.27 1.27)) (justify left top))
-    )
-    (instances
+  (sheet (at 24.765 23.495) (size 31.75 15.875)
+    (stroke (width 0.1524) (type solid))
+    (fill (color 0 0 0 0.0000))
+    (property "Sheetname" "1" (at 24.765 22.7834 0)
+      (effects (font (size 1.27 1.27)) (justify left bottom))
+    )
+    (property "Sheetfile" "1.kicad_sch" (at 24.765 40.0796 0)
+      (effects (font (size 1.27 1.27)) (justify left top))
+    )
+    (property "Text" "BUS + KEYBOARD INTERFACE" (at 40.64 31.75 0)
+      (effects (font (size 1.27 1.27) bold))
+    )
+    (instances
