File: gdp/6.kicad_sch (KiCad schematic)
At the start: 0 parts

Commit message: Adds pages 4, 7, 10 (still WIP)
Other:
- title: Partner GDP -> (none)
Changed lines of the file:
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@@
 (kicad_sch (version 20230121) (generator eeschema)
   (paper "A4")
-  (title_block
-    (title "Partner GDP")
-  )
 )

Commit message: Adds Sheet 5
Parts:
- added U9: 74LS83, symbol 74xx:74LS83
Connections:
- new net +5V: U9.5 (VCC)
- new net GND: U9.12 (GND)
Other:
- company: (none) -> Oddbit Retro
- title: (none) -> PARTNER GDP: GDP SCROLL + CAS MUX
Changed lines of the file:
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@@
 	(generator_version "8.0")
 	(paper "A4")
+	(title_block
+		(title "PARTNER GDP: GDP SCROLL + CAS MUX")
+		(company "Oddbit Retro")
+		(comment 1 "NARISAL: MIHA GRČAR")
+	)
+	(symbol
+		(lib_id "power:GNDD")
+		(at 80.01 87.63 0)
+		(unit 1)
+		(exclude_from_sim no)
+		(in_bom yes)
+		(on_board yes)
+		(dnp no)
+		(fields_autoplaced yes)
+		(property "Reference" "#PWR0103"
+			(at 80.01 93.98 0)
+			(effects
+				(font
+					(size 1.27 1.27)
+				)
+				(hide yes)
+			)
+		)
+		(property "Value" "GND"
+			(at 80.01 91.44 0)
+			(effects
+				(font
+					(size 1.27 1.27)
+				)
+			)
+		)
+		(property "Footprint" ""
+			(at 80.01 87.63 0)
+			(effects
+				(font
+					(size 1.27 1.27)
+				)
+				(hide yes)
+			)
+		)
+		(property "Datasheet" ""
+			(at 80.01 87.63 0)
+			(effects
+				(font
+					(size 1.27 1.27)
+				)
+				(hide yes)
+			)
+		)
+		(property "Description" "Power symbol creates a global label with name \"GNDD\" , digital ground"
+			(at 80.01 87.63 0)
+			(effects
+				(font
+					(size 1.27 1.27)
+				)
+				(hide yes)
+			)
+		)
+		(pin "1"
+		)
+		(instances
+			(project "gdp"
+				(path "/95aff260-2720-4733-a81d-a7a2136fdd14/d5ea0e5f-1e62-4ebe-9548-dbc71a82a27b"
+					(reference "#PWR0103")
+					(unit 1)
+				)
+			)
+		)
+	)
+	(symbol
+		(lib_id "power:+5V")
+		(at 80.01 46.99 0)
+		(unit 1)
+		(exclude_from_sim no)
+		(in_bom yes)
+		(on_board yes)
+		(dnp no)
+		(fields_autoplaced yes)
+		(property "Reference" "#PWR0102"
+			(at 80.01 50.8 0)
+			(effects
+				(font
+					(size 1.27 1.27)
+				)
+				(hide yes)
+			)
+		)
+		(property "Value" "+5V"
+			(at 80.01 41.91 0)
+			(effects
+				(font
+					(size 1.27 1.27)
+				)
+			)
+		)
+		(property "Footprint" ""
+			(at 80.01 46.99 0)
+			(effects
+				(font
+					(size 1.27 1.27)
+				)
+				(hide yes)
+			)
+		)
+		(property "Datasheet" ""
+			(at 80.01 46.99 0)
+			(effects
+				(font
+					(size 1.27 1.27)
+				)
+				(hide yes)
+			)
+		)
+		(property "Description" "Power symbol creates a global label with name \"+5V\""
+			(at 80.01 46.99 0)
+			(effects
+				(font
+					(size 1.27 1.27)
+				)
+				(hide yes)
+			)
+		)
+		(pin "1"
+		)
+		(instances
+			(project "gdp"
+				(path "/95aff260-2720-4733-a81d-a7a2136fdd14/d5ea0e5f-1e62-4ebe-9548-dbc71a82a27b"
+					(reference "#PWR0102")
+					(unit 1)
+				)
+			)
+		)
+	)
+	(symbol
+		(lib_id "74xx:74LS83")
+		(at 80.01 67.31 0)
+		(unit 1)
+		(exclude_from_sim no)
+		(in_bom yes)
+		(on_board yes)
+		(dnp no)
+		(fields_autoplaced yes)
+		(property "Reference" "U9"
+			(at 82.2041 46.99 0)
+			(effects
+				(font
+					(size 1.27 1.27)
+				)
+				(justify left)
+			)
+		)
+		(property "Value" "74LS83"
+			(at 82.2041 49.53 0)
+			(effects
+				(font
+					(size 1.27 1.27)
+				)
+				(justify left)
+			)
+		)
+		(property "Footprint" ""
+			(at 80.01 67.31 0)
+			(effects
+				(font
+					(size 1.27 1.27)
+				)
+				(hide yes)
+			)
+		)
+		(property "Datasheet" "http://www.ti.com/lit/gpn/sn74LS83"
+			(at 44.958 53.594 0)
+			(effects
+				(font
+					(size 1.27 1.27)
+				)
+				(hide yes)
+			)
+		)
+		(property "Description" "4-bit Full Adder"
+			(at 45.212 56.896 0)
+			(effects
+				(font
+					(size 1.27 1.27)
+				)
+				(hide yes)
+			)
+		)
+		(pin "13"
+		)
+		(pin "6"
+		)
+		(pin "1"
+		)
+		(pin "12"
+		)
+		(pin "14"
+		)
+		(pin "10"
+		)
+		(pin "3"
+		)
+		(pin "8"
+		)
+		(pin "4"
+		)
+		(pin "16"
+		)
+		(pin "5"
+		)
+		(pin "9"
+		)
+		(pin "7"
+		)
+		(pin "15"
+		)
+		(pin "2"
+		)
+		(pin "11"
+		)
+		(instances
+			(project ""
+				(path "/95aff260-2720-4733-a81d-a7a2136fdd14/d5ea0e5f-1e62-4ebe-9548-dbc71a82a27b"
+					(reference "U9")
+					(unit 1)
+				)
+			)
+		)
+	)
 )

Commit message: Adds Sheet 6
Parts:
- added U10: 74LS83, symbol 74xx:74LS83
- added U11, U12, U13, U14, U15, U16: 74LS244, symbol 74xx_IEEE:74LS244
Connections:
- net +5V: now also U10.5 (VCC), U11.20 (VCC), U12.20 (VCC), U13.20 (VCC), U14.20 (VCC), U15.20 (VCC), U16.20 (VCC)
- net GND: now also U10.12 (GND), U11.10 (GND), U11.11 (I0), U12.10 (GND), U13.10 (GND), U14.10 (GND), U14.8 (I3), U15.10 (GND), U16.10 (GND), U16.8 (I3)
- net DAD0: now reaches U9.1 (A4)
- net DAD0: now also U13.11 (I0), U15.4 (I1)
- net DAD3: now reaches U9.10 (A1)
- net DAD3: now also U13.17 (I3), U16.2 (I0)
- net SCRL4: now reaches U9.11 (B1)
- net at U9.13 (C0): now also U10.14 (C4)
- net at U9.15 (S4): now also U12.17 (I3)
- net SCRL7: now reaches U9.16 (B4)
- net at U9.2 (S3): now also U12.15 (I2)
- net DAD1: now reaches U9.3 (A3)
- net DAD1: now also U13.13 (I1), U15.6 (I2)
- net SCRL6: now reaches U9.4 (B3)
- net at U9.6 (S2): now also U12.13 (I1)
- net SCRL5: now reaches U9.7 (B2)
- net DAD2: now reaches U9.8 (A2)
- net DAD2: now also U13.15 (I2), U15.8 (I3)
- net at U9.9 (S1): now also U12.11 (I0)
- new net: U10.6 (S2), U11.13 (I1)
- new net: U10.2 (S3), U11.15 (I2)
- new net: U10.15 (S4), U11.17 (I3)
- new net: U10.9 (S1), U14.6 (I2), U16.6 (I2)
- new net DAD4: U10.1 (A4), U14.2 (I0), U16.4 (I1)
- new net DAD5: U10.3 (A3), U14.4 (I1)
- new net DAD6: U10.8 (A2)
- new net GA0: U11.7 (O1), U14.14 (O2), U16.14 (O2)
- new net GA1: U11.5 (O2), U14.16 (O1), U16.16 (O1)
- new net GA2: U11.3 (O3), U14.18 (O0), U16.18 (O0)
- new net GA3: U12.9 (O0), U13.3 (O3), U15.12 (O3)
- new net GA4: U12.7 (O1), U13.5 (O2), U15.14 (O2)
- new net GA5: U12.5 (O2), U13.7 (O1), U15.16 (O1)
- new net GA6: U12.3 (O3), U13.9 (O0), U15.18 (O0)
- new net MUX1: U11.19 (~{OE}), U12.19 (~{OE})
- new net PO: U10.10 (A1)
- new net SCRL0: U10.11 (B1)
- new net SCRL1: U10.7 (B2)
- new net SCRL2: U10.4 (B3)
- new net SCRL3: U10.16 (B4)
- new net X9: U15.2 (I0)
- new net ~{NORM}: U13.19 (~{OE}), U14.1 (~{OE})
- new net ~{SHIFT}: U15.1 (~{OE}), U16.1 (~{OE})
- no-connect marks 0 -> 3
Other:
- moved on the sheet: U9

Commit message: Fixes Sheet 7
Connections:
- net GND: now also U10.13 (C0)
Changed lines of the file:
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@@
 	)
 	(junction
-		(at 195.58 38.1)
-		(diameter 0)
-		(color 0 0 0 0)
-	)
-	(junction
 		(at 203.2 104.14)
 		(diameter 0)
@@
 	)
 	(junction
+		(at 203.2 38.1)
+		(diameter 0)
+		(color 0 0 0 0)
+	)
+	(junction
 		(at 46.99 83.82)
 		(diameter 0)
@@
 	(wire
 		(pts
-			(xy 195.58 38.1) (xy 195.58 71.12)
+			(xy 203.2 38.1) (xy 203.2 71.12)
 		)
 		(stroke
@@
 	(wire
 		(pts
-			(xy 184.15 111.76) (xy 204.47 111.76)
+			(xy 181.61 111.76) (xy 204.47 111.76)
 		)
 		(stroke
@@
 	(wire
 		(pts
-			(xy 195.58 38.1) (xy 204.47 38.1)
-		)
-		(stroke
-			(width 0)
-			(type default)
-		)
-	)
-	(wire
-		(pts
 			(xy 64.77 27.94) (xy 64.77 58.42)
 		)
@@
 	(wire
 		(pts
-			(xy 204.47 71.12) (xy 195.58 71.12)
+			(xy 204.47 71.12) (xy 203.2 71.12)
 		)
 		(stroke
@@
 	(wire
 		(pts
-			(xy 184.15 104.14) (xy 203.2 104.14)
+			(xy 181.61 104.14) (xy 203.2 104.14)
 		)
 		(stroke
@@
 	(wire
 		(pts
-			(xy 184.15 38.1) (xy 195.58 38.1)
+			(xy 184.15 38.1) (xy 203.2 38.1)
 		)
 		(stroke
@@
 	(wire
 		(pts
+			(xy 203.2 38.1) (xy 204.47 38.1)
+		)
+		(stroke
+			(width 0)
+			(type default)
+		)
+	)
+	(wire
+		(pts
 			(xy 40.64 81.28) (xy 67.31 81.28)
 		)
@@
 		)
 	)
+	(wire
+		(pts
+			(xy 71.12 106.68) (xy 80.01 106.68)
+		)
+		(stroke
+			(width 0)
+			(type default)
+		)
+	)
 	(bus
 		(pts
@@
 	(wire
 		(pts
+			(xy 63.5 73.66) (xy 67.31 73.66)
+		)
+		(stroke
+			(width 0)
+			(type default)
+		)
+	)
+	(wire
+		(pts
 			(xy 204.47 50.8) (xy 190.5 50.8)
 		)
@@
 	(global_label "X9"
 		(shape input)
-		(at 184.15 111.76 180)
+		(at 181.61 111.76 180)
 		(fields_autoplaced yes)
 		(effects
@@
 		)
 		(property "Intersheetrefs" "${INTERSHEET_REFS}"
-			(at 178.7458 111.76 0)
+			(at 176.2058 111.76 0)
 			(effects
 				(font
@@
 	(global_label "~{SHIFT}"
 		(shape input)
-		(at 184.15 104.14 180)
+		(at 181.61 104.14 180)
 		(fields_autoplaced yes)
 		(effects
@@
 		)
 		(property "Intersheetrefs" "${INTERSHEET_REFS}"
-			(at 175.9638 104.14 0)
+			(at 173.4238 104.14 0)
 			(effects
 				(font
@@
 		(on_board yes)
 		(dnp no)
-		(fields_autoplaced yes)
 		(property "Reference" "U11"
-			(at 144.4341 63.5 0)
+			(at 144.272 64.77 0)
 			(effects
 				(font
@@
 		)
 		(property "Value" "74LS244"
-			(at 144.4341 66.04 0)
+			(at 144.272 67.31 0)
 			(effects
 				(font
@@
 	(symbol
 		(lib_id "power:GNDD")
-		(at 80.01 106.68 0)
+		(at 71.12 106.68 0)
 		(unit 1)
 		(exclude_from_sim no)
@@
 		(fields_autoplaced yes)
 		(property "Reference" "#PWR0103"
-			(at 80.01 113.03 0)
+			(at 71.12 113.03 0)
 			(effects
 				(font
@@
 		)
 		(property "Value" "GND"
-			(at 80.01 110.49 0)
+			(at 71.12 110.49 0)
 			(effects
 				(font
@@
 		)
 		(property "Footprint" ""
-			(at 80.01 106.68 0)
+			(at 71.12 106.68 0)
 			(effects
 				(font
@@
 		)
 		(property "Datasheet" ""
-			(at 80.01 106.68 0)
+			(at 71.12 106.68 0)
 			(effects
 				(font
@@
 		)
 		(property "Description" "Power symbol creates a global label with name \"GNDD\" , digital ground"
-			(at 80.01 106.68 0)
+			(at 71.12 106.68 0)
 			(effects
 				(font
@@
 					(unit 1)
 				)
+			)
+		)
+	)
+	(symbol
+		(lib_id "power:GNDD")
+		(at 63.5 73.66 0)
+		(unit 1)
+		(exclude_from_sim no)
+		(in_bom yes)
+		(on_board yes)
+		(dnp no)
+		(fields_autoplaced yes)
+		(property "Reference" "#PWR0108"
+			(at 63.5 80.01 0)
+			(effects
+				(font
+					(size 1.27 1.27)
+				)
+				(hide yes)
+			)
+		)
+		(property "Value" "GND"
+			(at 63.5 77.47 0)
+			(effects
+				(font
+					(size 1.27 1.27)
+				)
+			)
+		)
+		(property "Footprint" ""
+			(at 63.5 73.66 0)
+			(effects
+				(font
+					(size 1.27 1.27)
+				)
+				(hide yes)
+			)
+		)
+		(property "Datasheet" ""
+			(at 63.5 73.66 0)
+			(effects
+				(font
+					(size 1.27 1.27)
+				)
+				(hide yes)
+			)
+		)
+		(property "Description" "Power symbol creates a global label with name \"GNDD\" , digital ground"
+			(at 63.5 73.66 0)
+			(effects
+				(font
+					(size 1.27 1.27)
+				)
+				(hide yes)
+			)
+		)
+		(pin "1"
+		)
+		(instances
+			(project "gdp"
+				(path "/95aff260-2720-4733-a81d-a7a2136fdd14/d5ea0e5f-1e62-4ebe-9548-dbc71a82a27b"
+					(reference "#PWR0108")
+					(unit 1)
+				)

Commit message: Adds Sheet 8
Parts:
- removed U14, U15: 74LS244, symbol 74xx_IEEE:74LS244
- added unit 1 of U11
- added unit 1 of U12
Connections:
- net +5V: now also U11.20 (VCC), U12.20 (VCC)
- net DAD0: now also U11.4 (I1)
- net DAD1: now also U11.6 (I2)
- net DAD2: now also U11.8 (I3)
- net DAD4: now also U12.2 (I0)
- net DAD5: now also U12.4 (I1)
- net GA0: now also U12.14 (O2)
- net GA1: now also U12.16 (O1)
- net GA2: now also U12.18 (O0)
- net GA3: now also U11.12 (O3)
- net GA4: now also U11.14 (O2)
- net GA5: now also U11.16 (O1)
- net GA6: now also U11.18 (O0)
- net GND: now also U11.10 (GND), U12.10 (GND), U12.8 (I3)
- net X9: now also U11.2 (I0)
- net ~{NORM}: now also U12.1 (~{OE})
- net ~{SHIFT}: now also U11.1 (~{OE})
- net at U10.9 (S1), U16.6 (I2): now also U12.6 (I2)

Commit message: Fixes Sheet 5
Connections:
- net +5V: no longer U13.20 (VCC)
- net GND: no longer U13.10 (GND)
Changed lines of the file:
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@@
 	)
 	(symbol
-		(lib_name "74LS244_1")
+		(lib_name "74LS244_3")
 		(lib_id "74xx_IEEE:74LS244")
 		(at 224.79 50.8 0)
@@
 		)
 		(instances
-			(project "gdp"
+			(project ""
+				(path "/95aff260-2720-4733-a81d-a7a2136fdd14/1e5736c7-7f09-4d36-9f85-33f8211ca85b"
+					(reference "U13")
+					(unit 2)
+				)
 				(path "/95aff260-2720-4733-a81d-a7a2136fdd14/d5ea0e5f-1e62-4ebe-9548-dbc71a82a27b"
 					(reference "U13")

Commit message: Adds Sheet 9
Parts:
- renumbered U10 to IC10, U9 to IC14, U11 to IC18, U12 to IC18, U12 to IC25, U16 to IC25, U11 to IC32, U13 to IC32
Connections:
- net +5V: now also IC32.20 (VCC)
- net GND: now also IC32.10 (GND)
Changed lines of the file:
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@@
 		(on_board yes)
 		(dnp no)
-		(property "Reference" "U11"
+		(property "Reference" "IC18"
 			(at 144.272 64.77 0)
 			(effects
@@
 			(project ""
 				(path "/95aff260-2720-4733-a81d-a7a2136fdd14/d5ea0e5f-1e62-4ebe-9548-dbc71a82a27b"
-					(reference "U11")
+					(reference "IC18")
 					(unit 2)
 				)
@@
 		(dnp no)
 		(fields_autoplaced yes)
-		(property "Reference" "U12"
+		(property "Reference" "IC18"
 			(at 224.79 78.994 0)
+			(do_not_autoplace yes)
 			(effects
 				(font
@@
 		(property "Value" "74LS244"
 			(at 224.79 81.534 0)
+			(do_not_autoplace yes)
 			(effects
 				(font
@@
 			(project "gdp"
 				(path "/95aff260-2720-4733-a81d-a7a2136fdd14/d5ea0e5f-1e62-4ebe-9548-dbc71a82a27b"
-					(reference "U12")
+					(reference "IC18")
 					(unit 1)
 				)
@@
 		(dnp no)
 		(fields_autoplaced yes)
-		(property "Reference" "U11"
+		(property "Reference" "IC32"
 			(at 224.79 112.014 0)
+			(do_not_autoplace yes)
 			(effects
 				(font
@@
 		(property "Value" "74LS244"
 			(at 224.79 114.554 0)
+			(do_not_autoplace yes)
 			(effects
 				(font
@@
 			(project "gdp"
 				(path "/95aff260-2720-4733-a81d-a7a2136fdd14/d5ea0e5f-1e62-4ebe-9548-dbc71a82a27b"
-					(reference "U11")
+					(reference "IC32")
 					(unit 1)
 				)
@@
 		(dnp no)
 		(fields_autoplaced yes)
-		(property "Reference" "U13"
+		(property "Reference" "IC32"
 			(at 224.79 45.974 0)
+			(do_not_autoplace yes)
 			(effects
 				(font
@@
 		(property "Value" "74LS244"
 			(at 224.79 48.514 0)
+			(do_not_autoplace yes)
 			(effects
 				(font
@@
 				)
 				(path "/95aff260-2720-4733-a81d-a7a2136fdd14/d5ea0e5f-1e62-4ebe-9548-dbc71a82a27b"
-					(reference "U13")
+					(reference "IC32")
 					(unit 2)
 				)
@@
 		(dnp no)
 		(fields_autoplaced yes)
-		(property "Reference" "U9"
+		(property "Reference" "IC14"
 			(at 82.2041 20.32 0)
 			(effects
@@
 			(project ""
 				(path "/95aff260-2720-4733-a81d-a7a2136fdd14/d5ea0e5f-1e62-4ebe-9548-dbc71a82a27b"
-					(reference "U9")
+					(reference "IC14")
 					(unit 1)
 				)
@@
 		(dnp no)
 		(fields_autoplaced yes)
-		(property "Reference" "U12"
+		(property "Reference" "IC25"
 			(at 144.4341 17.78 0)
 			(effects
@@
 			(project "gdp"
 				(path "/95aff260-2720-4733-a81d-a7a2136fdd14/d5ea0e5f-1e62-4ebe-9548-dbc71a82a27b"
-					(reference "U12")
+					(reference "IC25")
 					(unit 2)
 				)
@@
 		(dnp no)
 		(fields_autoplaced yes)
-		(property "Reference" "U10"
+		(property "Reference" "IC10"
 			(at 82.2041 66.04 0)
 			(effects
@@
 			(project "gdp"
 				(path "/95aff260-2720-4733-a81d-a7a2136fdd14/d5ea0e5f-1e62-4ebe-9548-dbc71a82a27b"
-					(reference "U10")
+					(reference "IC10")
 					(unit 1)
 				)
@@
 		(dnp no)
 		(fields_autoplaced yes)
-		(property "Reference" "U16"
+		(property "Reference" "IC25"
 			(at 224.79 145.034 0)
+			(do_not_autoplace yes)
 			(effects
 				(font
@@
 		(property "Value" "74LS244"
 			(at 224.79 147.574 0)
+			(do_not_autoplace yes)
 			(effects
 				(font
@@
 			(project "gdp"
 				(path "/95aff260-2720-4733-a81d-a7a2136fdd14/d5ea0e5f-1e62-4ebe-9548-dbc71a82a27b"
-					(reference "U16")
-					(unit 1)
-				)
+					(reference "IC25")
+					(unit 1)
+				)
