File: gdp/6.kicad_sch (KiCad schematic)
At the start: 5 parts, among them IC10 74LS83, IC14 74LS83, IC18 74LS244, IC25 74LS244, IC32 74LS244

Commit message: Adds Sheet 11
Changed lines of the file:
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@@
 	(bus
 		(pts
-			(xy 256.54 163.83) (xy 265.43 163.83)
+			(xy 256.54 161.29) (xy 265.43 161.29)
 		)
 		(stroke
@@
 	(bus
 		(pts
-			(xy 256.54 152.4) (xy 256.54 163.83)
+			(xy 256.54 152.4) (xy 256.54 161.29)
 		)
 		(stroke
@@
 	(global_label "GA[0..6]"
 		(shape output)
-		(at 265.43 163.83 0)
+		(at 265.43 161.29 0)
 		(fields_autoplaced yes)
 		(effects
@@
 		)
 		(property "Intersheetrefs" "${INTERSHEET_REFS}"
-			(at 276.0958 163.83 0)
-			(effects
-				(font
+			(at 276.0958 161.29 0)
+			(effects
+				(font

Commit message: Adds Sheet 12
Connections:
- net SOUT: now reaches IC14.14 (C4)
Changed lines of the file:
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@@
 	)
 	(bus_entry
-		(at 254 119.38)
+		(at 251.46 119.38)
 		(size 2.54 2.54)
 		(stroke
@@
 	)
 	(bus_entry
-		(at 254 53.34)
+		(at 251.46 53.34)
 		(size 2.54 2.54)
 		(stroke
@@
 	)
 	(bus_entry
-		(at 254 149.86)
+		(at 251.46 149.86)
 		(size 2.54 2.54)
 		(stroke
@@
 	)
 	(bus_entry
-		(at 254 111.76)
+		(at 251.46 111.76)
 		(size 2.54 2.54)
 		(stroke
@@
 	)
 	(bus_entry
-		(at 254 48.26)
+		(at 251.46 48.26)
 		(size 2.54 2.54)
 		(stroke
@@
 	)
 	(bus_entry
-		(at 254 50.8)
+		(at 251.46 50.8)
 		(size 2.54 2.54)
 		(stroke
@@
 	)
 	(bus_entry
-		(at 254 114.3)
+		(at 251.46 114.3)
 		(size 2.54 2.54)
 		(stroke
@@
 	)
 	(bus_entry
-		(at 254 144.78)
+		(at 251.46 144.78)
 		(size 2.54 2.54)
 		(stroke
@@
 	)
 	(bus_entry
-		(at 254 116.84)
+		(at 251.46 116.84)
 		(size 2.54 2.54)
 		(stroke
@@
 	)
 	(bus_entry
-		(at 254 147.32)
+		(at 251.46 147.32)
 		(size 2.54 2.54)
 		(stroke
@@
 	)
 	(bus_entry
-		(at 254 83.82)
+		(at 251.46 83.82)
 		(size 2.54 2.54)
 		(stroke
@@
 	)
 	(bus_entry
-		(at 254 78.74)
+		(at 251.46 78.74)
 		(size 2.54 2.54)
 		(stroke
@@
 	)
 	(bus_entry
-		(at 254 81.28)
+		(at 251.46 81.28)
 		(size 2.54 2.54)
 		(stroke
@@
 	)
 	(bus_entry
-		(at 254 45.72)
+		(at 251.46 45.72)
 		(size 2.54 2.54)
 		(stroke
@@
 	(wire
 		(pts
-			(xy 245.11 116.84) (xy 254 116.84)
+			(xy 245.11 116.84) (xy 251.46 116.84)
 		)
 		(stroke
@@
 	(wire
 		(pts
-			(xy 245.11 147.32) (xy 254 147.32)
+			(xy 245.11 147.32) (xy 251.46 147.32)
 		)
 		(stroke
@@
 	(wire
 		(pts
-			(xy 245.11 78.74) (xy 254 78.74)
+			(xy 245.11 78.74) (xy 251.46 78.74)
 		)
 		(stroke
@@
 	(bus
 		(pts
-			(xy 256.54 22.86) (xy 256.54 48.26)
+			(xy 254 22.86) (xy 254 48.26)
 		)
 		(stroke
@@
 	(wire
 		(pts
-			(xy 245.11 48.26) (xy 254 48.26)
+			(xy 245.11 48.26) (xy 251.46 48.26)
 		)
 		(stroke
@@
 	(bus
 		(pts
-			(xy 256.54 81.28) (xy 256.54 83.82)
-		)
-		(stroke
-			(width 0)
-			(type default)
-		)
-	)
-	(wire
-		(pts
-			(xy 245.11 114.3) (xy 254 114.3)
+			(xy 254 81.28) (xy 254 83.82)
+		)
+		(stroke
+			(width 0)
+			(type default)
+		)
+	)
+	(wire
+		(pts
+			(xy 245.11 114.3) (xy 251.46 114.3)
 		)
 		(stroke
@@
 	(bus
 		(pts
-			(xy 256.54 55.88) (xy 256.54 81.28)
+			(xy 254 55.88) (xy 254 81.28)
 		)
 		(stroke
@@
 	(wire
 		(pts
-			(xy 245.11 81.28) (xy 254 81.28)
+			(xy 245.11 81.28) (xy 251.46 81.28)
 		)
 		(stroke
@@
 	(bus
 		(pts
-			(xy 256.54 53.34) (xy 256.54 55.88)
-		)
-		(stroke
-			(width 0)
-			(type default)
-		)
-	)
-	(bus
-		(pts
-			(xy 256.54 119.38) (xy 256.54 121.92)
+			(xy 254 53.34) (xy 254 55.88)
+		)
+		(stroke
+			(width 0)
+			(type default)
+		)
+	)
+	(bus
+		(pts
+			(xy 254 119.38) (xy 254 121.92)
 		)
 		(stroke
@@
 	(wire
 		(pts
-			(xy 245.11 83.82) (xy 254 83.82)
+			(xy 245.11 83.82) (xy 251.46 83.82)
 		)
 		(stroke
@@
 	(bus
 		(pts
-			(xy 256.54 147.32) (xy 256.54 149.86)
+			(xy 254 147.32) (xy 254 149.86)
 		)
 		(stroke
@@
 	(wire
 		(pts
-			(xy 245.11 119.38) (xy 254 119.38)
+			(xy 245.11 119.38) (xy 251.46 119.38)
 		)
 		(stroke
@@
 	(bus
 		(pts
-			(xy 256.54 114.3) (xy 256.54 116.84)
+			(xy 254 114.3) (xy 254 116.84)
 		)
 		(stroke
@@
 	(bus
 		(pts
-			(xy 256.54 116.84) (xy 256.54 119.38)
-		)
-		(stroke
-			(width 0)
-			(type default)
-		)
-	)
-	(bus
-		(pts
-			(xy 170.18 22.86) (xy 256.54 22.86)
-		)
-		(stroke
-			(width 0)
-			(type default)
-		)
-	)
-	(wire
-		(pts
-			(xy 245.11 45.72) (xy 254 45.72)
+			(xy 254 116.84) (xy 254 119.38)
+		)
+		(stroke
+			(width 0)
+			(type default)
+		)
+	)
+	(bus
+		(pts
+			(xy 170.18 22.86) (xy 254 22.86)
+		)
+		(stroke
+			(width 0)
+			(type default)
+		)
+	)
+	(wire
+		(pts
+			(xy 245.11 45.72) (xy 251.46 45.72)
 		)
 		(stroke
@@
 	(bus
 		(pts
-			(xy 256.54 149.86) (xy 256.54 152.4)
+			(xy 254 149.86) (xy 254 152.4)
 		)
 		(stroke
@@
 	(bus
 		(pts
-			(xy 256.54 161.29) (xy 265.43 161.29)
+			(xy 254 161.29) (xy 260.35 161.29)
 		)
 		(stroke
@@
 	(bus
 		(pts
-			(xy 256.54 48.26) (xy 256.54 50.8)
+			(xy 254 48.26) (xy 254 50.8)
 		)
 		(stroke
@@
 	(wire
 		(pts
+			(xy 92.71 40.64) (xy 99.06 40.64)
+		)
+		(stroke
+			(width 0)
+			(type default)
+		)
+	)
+	(wire
+		(pts
 			(xy 203.2 38.1) (xy 204.47 38.1)
 		)
@@
 	(wire
 		(pts
-			(xy 245.11 111.76) (xy 254 111.76)
-		)
-		(stroke
-			(width 0)
-			(type default)
-		)
-	)
-	(bus
-		(pts
-			(xy 256.54 83.82) (xy 256.54 86.36)
+			(xy 245.11 111.76) (xy 251.46 111.76)
+		)
+		(stroke
+			(width 0)
+			(type default)
+		)
+	)
+	(bus
+		(pts
+			(xy 254 83.82) (xy 254 86.36)
 		)
 		(stroke
@@
 	(wire
 		(pts
-			(xy 245.11 144.78) (xy 254 144.78)
-		)
-		(stroke
-			(width 0)
-			(type default)
-		)
-	)
-	(wire
-		(pts
-			(xy 245.11 53.34) (xy 254 53.34)
+			(xy 245.11 144.78) (xy 251.46 144.78)
+		)
+		(stroke
+			(width 0)
+			(type default)
+		)
+	)
+	(wire
+		(pts
+			(xy 245.11 53.34) (xy 251.46 53.34)
 		)
 		(stroke
@@
 	(bus
 		(pts
-			(xy 256.54 121.92) (xy 256.54 147.32)
+			(xy 254 121.92) (xy 254 147.32)
 		)
 		(stroke
@@
 	(bus
 		(pts
-			(xy 256.54 50.8) (xy 256.54 53.34)
+			(xy 254 50.8) (xy 254 53.34)
 		)
 		(stroke
@@
 	(wire
 		(pts
-			(xy 245.11 149.86) (xy 254 149.86)
-		)
-		(stroke
-			(width 0)
-			(type default)
-		)
-	)
-	(wire
-		(pts
-			(xy 245.11 50.8) (xy 254 50.8)
-		)
-		(stroke
-			(width 0)
-			(type default)
-		)
-	)
-	(bus
-		(pts
-			(xy 256.54 86.36) (xy 256.54 114.3)
-		)
-		(stroke
-			(width 0)
-			(type default)
-		)
-	)
-	(bus
-		(pts
-			(xy 256.54 152.4) (xy 256.54 161.29)
+			(xy 245.11 149.86) (xy 251.46 149.86)
+		)
+		(stroke
+			(width 0)
+			(type default)
+		)
+	)
+	(wire
+		(pts
+			(xy 245.11 50.8) (xy 251.46 50.8)
+		)
+		(stroke
+			(width 0)
+			(type default)
+		)
+	)
+	(bus
+		(pts
+			(xy 254 86.36) (xy 254 114.3)
+		)
+		(stroke
+			(width 0)
+			(type default)
+		)
+	)
+	(bus
+		(pts
+			(xy 254 152.4) (xy 254 161.29)
 		)
 		(stroke
@@
 	(global_label "GA[0..6]"
 		(shape output)
-		(at 265.43 161.29 0)
+		(at 260.35 161.29 0)
 		(fields_autoplaced yes)
 		(effects
@@
 		)
 		(property "Intersheetrefs" "${INTERSHEET_REFS}"
-			(at 276.0958 161.29 0)
+			(at 271.0158 161.29 0)
 			(effects
 				(font
@@
 			)
 		)
+	)
+	(global_label "SOUT"
+		(shape output)
+		(at 99.06 40.64 0)
+		(fields_autoplaced yes)
+		(effects
+			(font
+				(size 1.27 1.27)
+			)
+			(justify left)
+		)
+		(property "Intersheetrefs" "${INTERSHEET_REFS}"
+			(at 106.8833 40.64 0)
+			(effects
+				(font
+					(size 1.27 1.27)
+				)
+				(justify left)
+			)
+		)

Commit message: Fixes IC references
Parts:
- renumbered IC32 to U13
Changed lines of the file:
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@@
 		(dnp no)
 		(fields_autoplaced yes)
-		(property "Reference" "IC32"
+		(property "Reference" "U13"
 			(at 224.79 45.974 0)
 			(do_not_autoplace yes)

Commit message: Initial footprint assignment
Parts:
- IC33: renamed from IC14; footprint (none) -> Package_DIP:DIP-16_W7.62mm
- IC34: renamed from IC10; footprint (none) -> Package_DIP:DIP-16_W7.62mm
- IC35: renamed from IC25; footprint (none) -> Package_DIP:DIP-20_W7.62mm
- IC36: renamed from IC18; footprint (none) -> Package_DIP:DIP-20_W7.62mm
- IC37: renamed from IC32; footprint (none) -> Package_DIP:DIP-20_W7.62mm
- U13: footprint (none) -> Package_DIP:DIP-20_W7.62mm
