File: gdp/6.kicad_sch (KiCad schematic)
At the start: 6 parts, among them IC33 74LS83, IC34 74LS83, IC35 74LS244, IC36 74LS244, IC37 74LS244, U13 74LS244

Commit message: Fixes refs
Parts:
- renumbered IC34 to IC10, IC33 to IC14, IC36 to IC18, IC35 to IC25, IC37 to IC32
Changed lines of the file:
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@@
 		(on_board yes)
 		(dnp no)
-		(property "Reference" "IC36"
+		(property "Reference" "IC18"
 			(at 144.272 64.77 0)
 			(effects
@@
 			(project ""
 				(path "/95aff260-2720-4733-a81d-a7a2136fdd14/d5ea0e5f-1e62-4ebe-9548-dbc71a82a27b"
-					(reference  "IC18")
+					(reference "IC18")
 					(unit 2)
 				)
@@
 		(dnp no)
 		(fields_autoplaced yes)
-		(property "Reference" "IC36"
+		(property "Reference" "IC18"
 			(at 224.79 78.994 0)
 			(do_not_autoplace yes)
@@
 			(project "gdp"
 				(path "/95aff260-2720-4733-a81d-a7a2136fdd14/d5ea0e5f-1e62-4ebe-9548-dbc71a82a27b"
-					(reference  "IC18")
+					(reference "IC18")
 					(unit 1)
 				)
@@
 		(dnp no)
 		(fields_autoplaced yes)
-		(property "Reference" "IC37"
+		(property "Reference" "IC32"
 			(at 224.79 112.014 0)
 			(do_not_autoplace yes)
@@
 			(project "gdp"
 				(path "/95aff260-2720-4733-a81d-a7a2136fdd14/d5ea0e5f-1e62-4ebe-9548-dbc71a82a27b"
-					(reference  "IC32")
+					(reference "IC32")
 					(unit 1)
 				)
@@
 				)
 				(path "/95aff260-2720-4733-a81d-a7a2136fdd14/d5ea0e5f-1e62-4ebe-9548-dbc71a82a27b"
-					(reference  "IC32")
+					(reference "IC32")
 					(unit 2)
 				)
@@
 		(dnp no)
 		(fields_autoplaced yes)
-		(property "Reference" "IC33"
+		(property "Reference" "IC14"
 			(at 82.2041 20.32 0)
 			(effects
@@
 			(project ""
 				(path "/95aff260-2720-4733-a81d-a7a2136fdd14/d5ea0e5f-1e62-4ebe-9548-dbc71a82a27b"
-					(reference  "IC14")
+					(reference "IC14")
 					(unit 1)
 				)
@@
 		(dnp no)
 		(fields_autoplaced yes)
-		(property "Reference" "IC35"
+		(property "Reference" "IC25"
 			(at 144.4341 17.78 0)
 			(effects
@@
 			(project "gdp"
 				(path "/95aff260-2720-4733-a81d-a7a2136fdd14/d5ea0e5f-1e62-4ebe-9548-dbc71a82a27b"
-					(reference  "IC25")
+					(reference "IC25")
 					(unit 2)
 				)
@@
 		(dnp no)
 		(fields_autoplaced yes)
-		(property "Reference" "IC34"
+		(property "Reference" "IC10"
 			(at 82.2041 66.04 0)
 			(effects
@@
 			(project "gdp"
 				(path "/95aff260-2720-4733-a81d-a7a2136fdd14/d5ea0e5f-1e62-4ebe-9548-dbc71a82a27b"
-					(reference  "IC10")
+					(reference "IC10")
 					(unit 1)
 				)
@@
 		(dnp no)
 		(fields_autoplaced yes)
-		(property "Reference" "IC35"
+		(property "Reference" "IC25"
 			(at 224.79 145.034 0)
 			(do_not_autoplace yes)
@@
 			(project "gdp"
 				(path "/95aff260-2720-4733-a81d-a7a2136fdd14/d5ea0e5f-1e62-4ebe-9548-dbc71a82a27b"
-					(reference  "IC25")
-					(unit 1)
-				)
+					(reference "IC25")
+					(unit 1)
+				)

Commit message: Fixes "CA0" issue in schematics
Parts:
- renumbered U13 to IC32
Changed lines of the file:
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@@
 (kicad_sch
-	(version 20231120)
+	(version 20250114)
 	(generator "eeschema")
-	(generator_version "8.0")
+	(generator_version "9.0")
 	(paper "A4")
 	(title_block
@@
 	(label "GA4"
 		(at 246.38 50.8 0)
-		(fields_autoplaced yes)
 		(effects
 			(font
@@
 	(label "GA0"
 		(at 246.38 149.86 0)
-		(fields_autoplaced yes)
 		(effects
 			(font
@@
 	(label "GA4"
 		(at 246.38 116.84 0)
-		(fields_autoplaced yes)
 		(effects
 			(font
@@
 	(label "GA5"
 		(at 163.83 48.26 0)
-		(fields_autoplaced yes)
 		(effects
 			(font
@@
 	(label "GA1"
 		(at 246.38 147.32 0)
-		(fields_autoplaced yes)
 		(effects
 			(font
@@
 	(label "GA3"
 		(at 246.38 53.34 0)
-		(fields_autoplaced yes)
 		(effects
 			(font
@@
 	(label "GA5"
 		(at 246.38 48.26 0)
-		(fields_autoplaced yes)
 		(effects
 			(font
@@
 	(label "GA0"
 		(at 246.38 83.82 0)
-		(fields_autoplaced yes)
 		(effects
 			(font
@@
 	(label "GA6"
 		(at 163.83 53.34 0)
-		(fields_autoplaced yes)
 		(effects
 			(font
@@
 	(label "GA3"
 		(at 246.38 119.38 0)
-		(fields_autoplaced yes)
 		(effects
 			(font
@@
 	(label "GA6"
 		(at 246.38 111.76 0)
-		(fields_autoplaced yes)
 		(effects
 			(font
@@
 	(label "GA3"
 		(at 163.83 38.1 0)
-		(fields_autoplaced yes)
 		(effects
 			(font
@@
 	(label "GA4"
 		(at 163.83 43.18 0)
-		(fields_autoplaced yes)
 		(effects
 			(font
@@
 	(label "GA2"
 		(at 246.38 78.74 0)
-		(fields_autoplaced yes)
 		(effects
 			(font
@@
 	(label "GA2"
 		(at 246.38 144.78 0)
-		(fields_autoplaced yes)
 		(effects
 			(font
@@
 	(label "GA1"
 		(at 163.83 93.98 0)
-		(fields_autoplaced yes)
 		(effects
 			(font
@@
 	(label "GA6"
 		(at 246.38 45.72 0)
-		(fields_autoplaced yes)
 		(effects
 			(font
@@
 	(label "GA5"
 		(at 246.38 114.3 0)
-		(fields_autoplaced yes)
 		(effects
 			(font
@@
 	(label "GA2"
 		(at 163.83 99.06 0)
-		(fields_autoplaced yes)
 		(effects
 			(font
@@
 	(label "GA0"
 		(at 163.83 88.9 0)
-		(fields_autoplaced yes)
 		(effects
 			(font
@@
 	(label "GA1"
 		(at 246.38 81.28 0)
-		(fields_autoplaced yes)
 		(effects
 			(font
@@
 		(dnp no)
 		(fields_autoplaced yes)
-		(property "Reference" "U13"
+		(property "Reference" "IC32"
 			(at 224.79 45.974 0)
 			(do_not_autoplace yes)
