File: gdp/8.kicad_sch (KiCad schematic)
At the start: 0 parts

Commit message: Adds pages 4, 7, 10 (still WIP)
Other:
- title: Partner GDP -> (none)
Changed lines of the file:
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@@
 (kicad_sch (version 20230121) (generator eeschema)
   (paper "A4")
-  (title_block
-    (title "Partner GDP")
-  )
 )

Commit message: Fixes Sheet 7
Other:
- company: (none) -> Oddbit Retro
- title: (none) -> PARTNER GDP: AVDC
Changed lines of the file:
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@@
 	(generator_version "8.0")
 	(paper "A4")
+	(title_block
+		(title "PARTNER GDP: AVDC")
+		(company "Oddbit Retro")
+		(comment 1 "NARISAL: MIHA GRČAR")
+	)
 )

Commit message: Adds Sheet 8
Parts:
- added IC19: SCN2674, Package_DIP:DIP-40_W15.24mm, symbol MCU_Parallax:P8X32A-D40
- added R32, R33, R34, R39, R41, R42, R45, R46, R47, R51, R53, R54: 330R, symbol Device:R
- added R48, R50: 10K, symbol Device:R
- added R49: 2K2, symbol Device:R
- added U13, U15: 74LS244, symbol 74xx_IEEE:74LS244
- added U14: 74LS245, symbol 74xx:74LS245
- added U17: 74LS367, symbol 74xx:74LS367
Connections:
- new net: IC19.2 (CE), R53.2, U17.9 (O4a)
- new net: IC19.15 (D7), R46.2, U14.9 (A7), U15.3 (O3)
- new net: IC19.39 (A2), R51.2, U17.7 (O3a)
- new net: IC19.14 (D6), R45.2, U14.8 (A6), U15.5 (O2)
- new net: IC19.13 (D5), R42.2, U14.7 (A5), U15.7 (O1)
- new net: IC19.12 (D4), R41.2, U14.6 (A4), U15.9 (O0)
- new net: IC19.9 (D1), R33.2, U13.16 (O1), U14.3 (A1)
- new net: IC19.10 (D2), R34.2, U13.14 (O2), U14.4 (A2)
- new net: IC19.38 (A1), R47.2, U17.5 (O2a)
- new net: IC19.8 (D0), R32.2, U13.18 (O0), U14.2 (A0)
- new net: IC19.11 (30), R39.2, U13.12 (O3), U14.5 (A3)
- new net: IC19.1 (RD), R48.2, U17.11 (O5b)
- new net: IC19.3 (WR), R50.2, U17.13 (O6b)
- new net: IC19.37 (A0), R49.2, U17.3 (O1a)
- new net +5V: IC19.40 (VCC), R47.1, R48.1, R51.1, R54.1, U13.20 (VCC), U14.20 (VCC), U15.20 (VCC), U17.16 (VCC)
- new net A0: U17.2 (I1)
- new net A1: U17.4 (I2)
- new net A2: U17.6 (I3)
- new net AHSYNC: IC19.19 (HSYNC)
- new net ASCD0: U13.2 (I0)
- new net ASCD1: U13.4 (I1)
- new net ASCD2: U13.6 (I2)
- new net ASCD3: U13.8 (I3)
- new net ASCD4: U15.11 (I0)
- new net ASCD5: U15.13 (I1)
- new net ASCD6: U15.15 (I2)
- new net ASCD7: U15.17 (I3)
- new net AVSCS: IC19.18 (V/CSYNC)
- new net BLANK: IC19.17 (BLANK)
- new net CURSOR: IC19.7 (CRS)
- new net D0: U14.18 (B0)
- new net D1: U14.17 (B1)
- new net D2: U14.16 (B2)
- new net D3: U14.15 (B3)
- new net D4: U14.14 (B4)
- new net D5: U14.13 (B5)
- new net D6: U14.12 (B6)
- new net D7: U14.11 (B7)
- new net DA0: IC19.34 (DA0/LG)
- new net DA1: IC19.33 (DA1/DA14)
- new net DA10: IC19.24 (DA10/UL)
- new net DA11: IC19.23 (DA11/BLI)
- new net DA12: IC19.22 (DA12/ODD)
- new net DA13: IC19.21 (DA13/LL)
- new net DA2: IC19.32 (DA2/DA15)
- new net DA3: IC19.31 (DA3/LR)
- new net DA4: IC19.30 (DA4/LA0)
- new net DA5: IC19.29 (DA5/LA1)
- new net DA6: IC19.28 (DA6/LA2)
- new net DA7: IC19.27 (DA7/LA3)
- new net DA8: IC19.26 (DA8/FL)
- new net DA9: IC19.25 (DA9/DW)
- new net GNDD: IC19.20 (GND), R32.1, R33.1, R34.1, R39.1, R41.1, R42.1, R45.1, R46.1, R49.1, R50.1, R53.1, U13.10 (GND), U14.10 (GND), U15.10 (GND), U17.8 (GND)
- new net LROW: U17.1 (OEa), U17.15 (OEb)
- new net MASTER: IC19.36 (ACLL)
- new net ~{AVDC}: U14.19 (CE), U17.10 (I4)
- new net ~{AVINT}: IC19.35 (INTR), R54.2
- new net ~{BCE}: IC19.6 (CTRL3)
- new net ~{CCLK}: IC19.16 (CCLK)
- new net ~{RDB}: IC19.5 (CTRL2)
- new net ~{RD}: U17.12 (I5)
- new net ~{ROW}: U13.1 (~{OE}), U15.19 (~{OE})
- new net ~{WDB}: IC19.4 (CTRL1)
- new net ~{WR}: U14.1 (A->B), U17.14 (I6)

Commit message: Fixes Sheet 5
Other:
- moved on the sheet: IC19, R32, R33, R34, R39, R41, R42, R45, R46, R47, R48, R49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

Commit message: Adds Sheet 9
Parts:
- removed R32, R33, R34, R39, R41, R42, R45, R46: 330R, symbol Device:R
- added RN1: 8x2K2, Resistor_THT:R_Array_SIP9, symbol Device:R_Network08
- R13: renamed from R51; value 330R -> 1K0
- R14: renamed from R48; value 10K -> 1K0
- R15: renamed from R47; value 330R -> 1K0
- R16: renamed from R54; value 330R -> 2K2
- R16: renamed from R50; value 10K -> 1K0
- R17: renamed from R49; value 2K2 -> 1K0
- R18: renamed from R53; value 330R -> 1K0
- renumbered U15 to IC13, U13 to IC13, U14 to IC16, U17 to IC4, IC19 to IC5
Connections:
- net GNDD: now also RN1.1 (common)
- net at IC13.3 (O3), IC16.9 (A7), IC5.15 (D7): now also RN1.9 (R8)
- net at IC13.5 (O2), IC16.8 (A6), IC5.14 (D6): now also RN1.8 (R7)
- net at IC13.7 (O1), IC16.7 (A5), IC5.13 (D5): now also RN1.7 (R6)
- net at IC13.9 (O0), IC16.6 (A4), IC5.12 (D4): now also RN1.6 (R5)
- net at IC13.16 (O1), IC16.3 (A1), IC5.9 (D1): now also RN1.3 (R2)
- net at IC13.14 (O2), IC16.4 (A2), IC5.10 (D2): now also RN1.4 (R3)
- net at IC13.18 (O0), IC16.2 (A0), IC5.8 (D0): now also RN1.2 (R1)
- net at IC13.12 (O3), IC16.5 (A3), IC5.11 (30): now also RN1.5 (R4)
Other:
- moved on the sheet: IC13B

Commit message: Adds Sheet 11
Other:
- moved on the sheet: R16
Changed lines of the file:
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@@
 	(wire
 		(pts
-			(xy 247.65 29.21) (xy 247.65 43.18)
+			(xy 247.65 31.75) (xy 247.65 43.18)
 		)
 		(stroke
@@
 	(wire
 		(pts
-			(xy 116.84 67.31) (xy 121.92 67.31)
-		)
-		(stroke
-			(width 0)
-			(type default)
-		)
-	)
-	(wire
-		(pts
 			(xy 72.39 119.38) (xy 72.39 49.53)
 		)
@@
 	(symbol
 		(lib_id "power:+5V")
-		(at 247.65 21.59 0)
+		(at 247.65 24.13 0)
 		(unit 1)
 		(exclude_from_sim no)
@@
 		(dnp no)
 		(property "Reference" "#PWR0132"
-			(at 247.65 25.4 0)
+			(at 247.65 27.94 0)
 			(effects
 				(font
@@
 		)
 		(property "Value" "+5V"
-			(at 247.65 17.145 0)
+			(at 247.65 19.685 0)
 			(effects
 				(font
@@
 		)
 		(property "Footprint" ""
-			(at 247.65 21.59 0)
+			(at 247.65 24.13 0)
 			(effects
 				(font
@@
 		)
 		(property "Datasheet" ""
-			(at 247.65 21.59 0)
+			(at 247.65 24.13 0)
 			(effects
 				(font
@@
 		)
 		(property "Description" ""
-			(at 247.65 21.59 0)
+			(at 247.65 24.13 0)
 			(effects
 				(font
@@
 	(symbol
 		(lib_id "Device:R")
-		(at 247.65 25.4 0)
+		(at 247.65 27.94 0)
 		(unit 1)
 		(exclude_from_sim no)
@@
 		(dnp no)
 		(property "Reference" "R16"
-			(at 248.92 24.13 0)
+			(at 248.92 26.67 0)
 			(effects
 				(font
@@
 		)
 		(property "Value" "2K2"
-			(at 248.92 26.67 0)
+			(at 248.92 29.21 0)
 			(effects
 				(font
@@
 		)
 		(property "Footprint" ""
-			(at 245.872 25.4 90)
+			(at 245.872 27.94 90)
 			(effects
 				(font
@@
 		)
 		(property "Datasheet" "~"
-			(at 247.65 25.4 0)
+			(at 247.65 27.94 0)
 			(effects
 				(font
@@
 		)
 		(property "Description" ""
-			(at 247.65 25.4 0)
+			(at 247.65 27.94 0)
 			(effects
 				(font
@@
 	(symbol
 		(lib_id "power:GNDD")
-		(at 116.84 67.31 0)
+		(at 121.92 67.31 180)
 		(unit 1)
 		(exclude_from_sim no)
@@
 		(fields_autoplaced yes)
 		(property "Reference" "#PWR0129"
-			(at 116.84 73.66 0)
+			(at 121.92 60.96 0)
 			(effects
 				(font
@@
 		)
 		(property "Value" "GNDD"
-			(at 116.84 71.12 0)
+			(at 121.92 63.5 0)
 			(effects
 				(font
@@
 		)
 		(property "Footprint" ""
-			(at 116.84 67.31 0)
+			(at 121.92 67.31 0)
 			(effects
 				(font
@@
 		)
 		(property "Datasheet" ""
-			(at 116.84 67.31 0)
+			(at 121.92 67.31 0)
 			(effects
 				(font
@@
 		)
 		(property "Description" ""
-			(at 116.84 67.31 0)
+			(at 121.92 67.31 0)
 			(effects
 				(font

Commit message: Adds Sheet 12
Parts:
- removed IC13: 74LS244, symbol 74xx_IEEE:74LS244
- removed IC16: 74LS245, symbol 74xx:74LS245
- removed IC4: 74LS367, symbol 74xx:74LS367
- removed IC5: SCN2674, Package_DIP:DIP-40_W15.24mm, symbol MCU_Parallax:P8X32A-D40
- removed R14, R15, R16, R18: 1K0, symbol Device:R
- removed R16: 2K2, symbol Device:R
- added IC13: 74LS245, symbol 74xx:74LS245
- added IC16: SCN2674, Package_DIP:DIP-40_W15.24mm, symbol MCU_Parallax:P8X32A-D40
- added IC4: 74LS244, symbol 74xx_IEEE:74LS244
- added IC5: 74LS367, symbol 74xx:74LS367
- added R16, R3, R4, R5, R6: 1K0, symbol Device:R
- R17: value 1K0 -> 2K2
Connections:
- net +5V: now also R17.1, IC13.20 (VCC), IC16.40 (VCC), IC4.20 (VCC), IC4.20 (VCC), IC5.16 (VCC), R3.1, R4.1, R5.1; no longer R13.1
- net A0: now also IC5.2 (I1)
- net A1: now also IC5.4 (I2)
- net A2: now also IC5.6 (I3)
- net AHSYNC: now also IC16.19 (HSYNC)
- net ASCD0: now also IC4.2 (I0)
- net ASCD1: now also IC4.4 (I1)
- net ASCD2: now also IC4.6 (I2)
- net ASCD3: now also IC4.8 (I3)
- net ASCD4: now also IC4.11 (I0)
- net ASCD5: now also IC4.13 (I1)
- net ASCD6: now also IC4.15 (I2)
- net ASCD7: now also IC4.17 (I3)
- net AVSCS: now also IC16.18 (V/CSYNC)
- net BLANK: now also IC16.17 (BLANK)
- net CURSOR: now also IC16.7 (CRS)
- net D0: now also IC13.18 (B0)
- net D1: now also IC13.17 (B1)
- net D2: now also IC13.16 (B2)
- net D3: now also IC13.15 (B3)
- net D4: now also IC13.14 (B4)
- net D5: now also IC13.13 (B5)
- net D6: now also IC13.12 (B6)
- net D7: now also IC13.11 (B7)
- net DA0: now also IC16.34 (DA0/LG)
- net DA1: now also IC16.33 (DA1/DA14)
- net DA10: now also IC16.24 (DA10/UL)
- net DA11: now also IC16.23 (DA11/BLI)
- net DA12: now also IC16.22 (DA12/ODD)
- net DA13: now also IC16.21 (DA13/LL)
- net DA2: now also IC16.32 (DA2/DA15)
- net DA3: now also IC16.31 (DA3/LR)
- net DA4: now also IC16.30 (DA4/LA0)
- net DA5: now also IC16.29 (DA5/LA1)
- net DA6: now also IC16.28 (DA6/LA2)
- net DA7: now also IC16.27 (DA7/LA3)
- net DA8: now also IC16.26 (DA8/FL)
- net DA9: now also IC16.25 (DA9/DW)
- net GNDD: now also R13.1, IC13.10 (GND), IC16.20 (GND), IC4.10 (GND), IC4.10 (GND), IC5.8 (GND), R16.1, R6.1; no longer R17.1
- net LROW: now also IC5.1 (OEa), IC5.15 (OEb)
- net MASTER: now also IC16.36 (ACLL)
- net ~{AVDC}: now also IC13.19 (CE), IC5.10 (I4)
- net ~{AVINT}: now also R17.2, IC16.35 (INTR)
- net ~{BCE}: now also IC16.6 (CTRL3)
- net ~{CCLK}: now also IC16.16 (CCLK)
- net ~{RDB}: now also IC16.5 (CTRL2)
- net ~{RD}: now also IC5.12 (I5)
- net ~{ROW}: now also IC4.1 (~{OE}), IC4.19 (~{OE})
- net ~{WDB}: now also IC16.4 (CTRL1)
- net ~{WR}: now also IC13.1 (A->B), IC5.14 (I6)
- net at R13.2: now also IC16.3 (WR), IC5.13 (O6b)
- net at RN1.9 (R8): now also IC13.9 (A7), IC16.15 (D7), IC4.3 (O3)
- net at RN1.8 (R7): now also IC13.8 (A6), IC16.14 (D6), IC4.5 (O2)
- net at RN1.7 (R6): now also IC13.7 (A5), IC16.13 (D5), IC4.7 (O1)
- net at RN1.6 (R5): now also IC13.6 (A4), IC16.12 (D4), IC4.9 (O0)
- net at RN1.2 (R1): now also IC13.2 (A0), IC16.8 (D0), IC4.18 (O0)
- net at RN1.3 (R2): now also IC13.3 (A1), IC16.9 (D1), IC4.16 (O1)
- net at RN1.4 (R3): now also IC13.4 (A2), IC16.10 (D2), IC4.14 (O2)
- net at RN1.5 (R4): now also IC13.5 (A3), IC16.11 (30), IC4.12 (O3)
- new net: IC16.2 (CE), IC5.9 (O4a), R16.2
- new net: IC16.39 (A2), IC5.7 (O3a), R3.2
- new net: IC16.1 (RD), IC5.11 (O5b), R5.2
- new net: IC16.37 (A0), IC5.3 (O1a), R6.2
- new net: IC16.38 (A1), IC5.5 (O2a), R4.2
