File: gdp/8.kicad_sch (KiCad schematic)
At the start: 12 parts, among them IC13 74LS245, IC16 SCN2674, IC4 74LS244, IC5 74LS367

Commit message: Fixes IC references
Parts:
- renumbered IC4 to IC13, IC13 to IC16, IC5 to IC4, IC16 to IC5
Changed lines of the file:
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@@
 		(dnp no)
 		(fields_autoplaced yes)
-		(property "Reference" "IC13"
+		(property "Reference" "IC16"
 			(at 173.6441 113.03 0)
 			(effects
@@
 			(project "gdp"
 				(path "/95aff260-2720-4733-a81d-a7a2136fdd14/1e5736c7-7f09-4d36-9f85-33f8211ca85b"
-					(reference "IC13")
+					(reference "IC16")
 					(unit 1)
 				)
@@
 		(dnp no)
 		(fields_autoplaced yes)
-		(property "Reference" "IC5"
+		(property "Reference" "IC4"
 			(at 131.7341 25.4 0)
 			(effects
@@
 			(project "gdp"
 				(path "/95aff260-2720-4733-a81d-a7a2136fdd14/1e5736c7-7f09-4d36-9f85-33f8211ca85b"
-					(reference "IC5")
+					(reference "IC4")
 					(unit 1)
 				)
@@
 		(dnp no)
 		(fields_autoplaced yes)
-		(property "Reference" "IC4"
+		(property "Reference" "IC13"
 			(at 88.9 138.684 0)
 			(do_not_autoplace yes)
@@
 			(project "gdp"
 				(path "/95aff260-2720-4733-a81d-a7a2136fdd14/1e5736c7-7f09-4d36-9f85-33f8211ca85b"
-					(reference "IC4")
+					(reference "IC13")
 					(unit 2)
 				)
@@
 		(dnp no)
 		(fields_autoplaced yes)
-		(property "Reference" "IC4"
+		(property "Reference" "IC13"
 			(at 88.9 85.344 0)
 			(do_not_autoplace yes)
@@
 			(project "gdp"
 				(path "/95aff260-2720-4733-a81d-a7a2136fdd14/1e5736c7-7f09-4d36-9f85-33f8211ca85b"
-					(reference "IC4")
+					(reference "IC13")
 					(unit 1)
 				)
@@
 		(on_board yes)
 		(dnp no)
-		(property "Reference" "IC16"
+		(property "Reference" "IC5"
 			(at 214.63 62.23 0)
 			(effects
@@
 			(project "gdp"
 				(path "/95aff260-2720-4733-a81d-a7a2136fdd14/1e5736c7-7f09-4d36-9f85-33f8211ca85b"
-					(reference "IC16")
-					(unit 1)
-				)
+					(reference "IC5")
+					(unit 1)
+				)

Commit message: Small fixes
Parts:
- renumbered R16 to R1, R13 to R2, R4 to R3, R6 to R4, R3 to R6
Changed lines of the file:
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@@
 		(on_board yes)
 		(dnp no)
-		(property "Reference" "R13"
+		(property "Reference" "R2"
 			(at 180.34 24.13 0)
 			(effects
@@
 			(project "gdp"
 				(path "/95aff260-2720-4733-a81d-a7a2136fdd14/1e5736c7-7f09-4d36-9f85-33f8211ca85b"
-					(reference "R13")
+					(reference "R2")
 					(unit 1)
 				)
@@
 		(on_board yes)
 		(dnp no)
-		(property "Reference" "R16"
+		(property "Reference" "R1"
 			(at 187.96 24.13 0)
 			(effects
@@
 			(project "gdp"
 				(path "/95aff260-2720-4733-a81d-a7a2136fdd14/1e5736c7-7f09-4d36-9f85-33f8211ca85b"
-					(reference "R16")
+					(reference "R1")
 					(unit 1)
 				)
@@
 		(on_board yes)
 		(dnp no)
-		(property "Reference" "R3"
+		(property "Reference" "R6"
 			(at 149.86 24.13 0)
 			(effects
@@
 			(project "gdp"
 				(path "/95aff260-2720-4733-a81d-a7a2136fdd14/1e5736c7-7f09-4d36-9f85-33f8211ca85b"
-					(reference "R3")
+					(reference "R6")
 					(unit 1)
 				)
@@
 		(on_board yes)
 		(dnp no)
-		(property "Reference" "R6"
+		(property "Reference" "R4"
 			(at 172.72 24.13 0)
 			(effects
@@
 			(project "gdp"
 				(path "/95aff260-2720-4733-a81d-a7a2136fdd14/1e5736c7-7f09-4d36-9f85-33f8211ca85b"
-					(reference "R6")
+					(reference "R4")
 					(unit 1)
 				)
@@
 		(on_board yes)
 		(dnp no)
-		(property "Reference" "R4"
+		(property "Reference" "R3"
 			(at 157.48 24.13 0)
 			(effects
@@
 			(project "gdp"
 				(path "/95aff260-2720-4733-a81d-a7a2136fdd14/1e5736c7-7f09-4d36-9f85-33f8211ca85b"
-					(reference "R4")
-					(unit 1)
-				)
+					(reference "R3")
+					(unit 1)
+				)

Commit message: Initial footprint assignment
Parts:
- IC46: renamed from IC13; footprint (none) -> Package_DIP:DIP-20_W7.62mm
- IC47: renamed from IC4; footprint (none) -> Package_DIP:DIP-16_W7.62mm
- IC48: renamed from IC16; footprint (none) -> Package_DIP:DIP-20_W7.62mm
- R20: renamed from R6; footprint (none) -> Resistor_THT:R_Axial_DIN0207_L6.3mm_D2.5mm_P7.62mm_Horizontal
- R21: renamed from R3; footprint (none) -> Resistor_THT:R_Axial_DIN0207_L6.3mm_D2.5mm_P7.62mm_Horizontal
- R22: renamed from R5; footprint (none) -> Resistor_THT:R_Axial_DIN0207_L6.3mm_D2.5mm_P7.62mm_Horizontal
- R23: renamed from R4; footprint (none) -> Resistor_THT:R_Axial_DIN0207_L6.3mm_D2.5mm_P7.62mm_Horizontal
- R24: renamed from R2; footprint (none) -> Resistor_THT:R_Axial_DIN0207_L6.3mm_D2.5mm_P7.62mm_Horizontal
- R25: renamed from R1; footprint (none) -> Resistor_THT:R_Axial_DIN0207_L6.3mm_D2.5mm_P7.62mm_Horizontal
- R26: renamed from R17; footprint (none) -> Resistor_THT:R_Axial_DIN0207_L6.3mm_D2.5mm_P7.62mm_Horizontal
- renumbered IC5 to IC49, RN1 to RN3
