File: gdp/8.kicad_sch (KiCad schematic)
At the start: 12 parts, among them IC46 74LS244, IC47 74LS367, IC48 74LS245, IC49 SCN2674

Commit message: Fixes refs
Parts:
- renumbered IC46 to IC13, IC48 to IC16, IC47 to IC4, IC49 to IC5, R25 to R1, R26 to R16, R24 to R2, R21 to R3, R23 to R4, R22 to R5, R20 to R6, RN3 to RN1
Changed lines of the file:
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@@
 		(on_board yes)
 		(dnp no)
-		(property "Reference" "R24"
+		(property "Reference" "R2"
 			(at 180.34 24.13 0)
 			(effects
@@
 			(project "gdp"
 				(path "/95aff260-2720-4733-a81d-a7a2136fdd14/1e5736c7-7f09-4d36-9f85-33f8211ca85b"
-					(reference  "R2")
+					(reference "R2")
 					(unit 1)
 				)
@@
 		(on_board yes)
 		(dnp no)
-		(property "Reference" "R25"
+		(property "Reference" "R1"
 			(at 187.96 24.13 0)
 			(effects
@@
 			(project "gdp"
 				(path "/95aff260-2720-4733-a81d-a7a2136fdd14/1e5736c7-7f09-4d36-9f85-33f8211ca85b"
-					(reference  "R1")
+					(reference "R1")
 					(unit 1)
 				)
@@
 		(on_board yes)
 		(dnp no)
-		(property "Reference" "R20"
+		(property "Reference" "R6"
 			(at 149.86 24.13 0)
 			(effects
@@
 			(project "gdp"
 				(path "/95aff260-2720-4733-a81d-a7a2136fdd14/1e5736c7-7f09-4d36-9f85-33f8211ca85b"
-					(reference  "R6")
+					(reference "R6")
 					(unit 1)
 				)
@@
 		(dnp no)
 		(fields_autoplaced yes)
-		(property "Reference" "IC48"
+		(property "Reference" "IC16"
 			(at 173.6441 113.03 0)
 			(effects
@@
 			(project "gdp"
 				(path "/95aff260-2720-4733-a81d-a7a2136fdd14/1e5736c7-7f09-4d36-9f85-33f8211ca85b"
-					(reference  "IC16")
+					(reference "IC16")
 					(unit 1)
 				)
@@
 		(dnp no)
 		(fields_autoplaced yes)
-		(property "Reference" "IC47"
+		(property "Reference" "IC4"
 			(at 131.7341 25.4 0)
 			(effects
@@
 			(project "gdp"
 				(path "/95aff260-2720-4733-a81d-a7a2136fdd14/1e5736c7-7f09-4d36-9f85-33f8211ca85b"
-					(reference  "IC4")
+					(reference "IC4")
 					(unit 1)
 				)
@@
 		(on_board yes)
 		(dnp no)
-		(property "Reference" "R23"
+		(property "Reference" "R4"
 			(at 172.72 24.13 0)
 			(effects
@@
 			(project "gdp"
 				(path "/95aff260-2720-4733-a81d-a7a2136fdd14/1e5736c7-7f09-4d36-9f85-33f8211ca85b"
-					(reference  "R4")
+					(reference "R4")
 					(unit 1)
 				)
@@
 		(dnp no)
 		(fields_autoplaced yes)
-		(property "Reference" "IC46"
+		(property "Reference" "IC13"
 			(at 88.9 138.684 0)
 			(do_not_autoplace yes)
@@
 			(project "gdp"
 				(path "/95aff260-2720-4733-a81d-a7a2136fdd14/1e5736c7-7f09-4d36-9f85-33f8211ca85b"
-					(reference  "IC13")
+					(reference "IC13")
 					(unit 2)
 				)
@@
 		(dnp no)
 		(fields_autoplaced yes)
-		(property "Reference" "RN3"
+		(property "Reference" "RN1"
 			(at 132.08 72.6439 0)
 			(effects
@@
 			(project "gdp"
 				(path "/95aff260-2720-4733-a81d-a7a2136fdd14/1e5736c7-7f09-4d36-9f85-33f8211ca85b"
-					(reference  "RN1")
+					(reference "RN1")
 					(unit 1)
 				)
@@
 		(on_board yes)
 		(dnp no)
-		(property "Reference" "R22"
+		(property "Reference" "R5"
 			(at 165.1 24.13 0)
 			(effects
@@
 			(project "gdp"
 				(path "/95aff260-2720-4733-a81d-a7a2136fdd14/1e5736c7-7f09-4d36-9f85-33f8211ca85b"
-					(reference  "R5")
+					(reference "R5")
 					(unit 1)
 				)
@@
 		(dnp no)
 		(fields_autoplaced yes)
-		(property "Reference" "IC46"
+		(property "Reference" "IC13"
 			(at 88.9 85.344 0)
 			(do_not_autoplace yes)
@@
 			(project "gdp"
 				(path "/95aff260-2720-4733-a81d-a7a2136fdd14/1e5736c7-7f09-4d36-9f85-33f8211ca85b"
-					(reference  "IC13")
+					(reference "IC13")
 					(unit 1)
 				)
@@
 		(on_board yes)
 		(dnp no)
-		(property "Reference" "IC49"
+		(property "Reference" "IC5"
 			(at 214.63 62.23 0)
 			(effects
@@
 			(project "gdp"
 				(path "/95aff260-2720-4733-a81d-a7a2136fdd14/1e5736c7-7f09-4d36-9f85-33f8211ca85b"
-					(reference  "IC5")
+					(reference "IC5")
 					(unit 1)
 				)
@@
 		(on_board yes)
 		(dnp no)
-		(property "Reference" "R21"
+		(property "Reference" "R3"
 			(at 157.48 24.13 0)
 			(effects
@@
 			(project "gdp"
 				(path "/95aff260-2720-4733-a81d-a7a2136fdd14/1e5736c7-7f09-4d36-9f85-33f8211ca85b"
-					(reference  "R3")
+					(reference "R3")
 					(unit 1)
 				)
@@
 		(on_board yes)
 		(dnp no)
-		(property "Reference" "R26"
+		(property "Reference" "R16"
 			(at 238.76 27.94 0)
 			(effects
@@
 			(project "gdp"
 				(path "/95aff260-2720-4733-a81d-a7a2136fdd14/1e5736c7-7f09-4d36-9f85-33f8211ca85b"
-					(reference  "R17")
-					(unit 1)
-				)
+					(reference "R16")
+					(unit 1)
+				)

Commit message: Placing footprints...
Parts:
- R1, R16, R2, R3, R4, R5, R6: footprint Resistor_THT:R_Axial_DIN0207_L6.3mm_D2.5mm_P7.62mm_Horizontal -> Resistor_THT:R_Axial_DIN0207_L6.3mm_D2.5mm_P10.16mm_Horizontal
Changed lines of the file:
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@@
 			)
 		)
-		(property "Footprint" "Resistor_THT:R_Axial_DIN0207_L6.3mm_D2.5mm_P7.62mm_Horizontal"
+		(property "Footprint" "Resistor_THT:R_Axial_DIN0207_L6.3mm_D2.5mm_P10.16mm_Horizontal"
 			(at 177.292 25.4 90)
 			(effects
@@
 			)
 		)
-		(property "Footprint" "Resistor_THT:R_Axial_DIN0207_L6.3mm_D2.5mm_P7.62mm_Horizontal"
+		(property "Footprint" "Resistor_THT:R_Axial_DIN0207_L6.3mm_D2.5mm_P10.16mm_Horizontal"
 			(at 184.912 25.4 90)
 			(effects
@@
 			)
 		)
-		(property "Footprint" "Resistor_THT:R_Axial_DIN0207_L6.3mm_D2.5mm_P7.62mm_Horizontal"
+		(property "Footprint" "Resistor_THT:R_Axial_DIN0207_L6.3mm_D2.5mm_P10.16mm_Horizontal"
 			(at 146.812 25.4 90)
 			(effects
@@
 			)
 		)
-		(property "Footprint" "Resistor_THT:R_Axial_DIN0207_L6.3mm_D2.5mm_P7.62mm_Horizontal"
+		(property "Footprint" "Resistor_THT:R_Axial_DIN0207_L6.3mm_D2.5mm_P10.16mm_Horizontal"
 			(at 169.672 25.4 90)
 			(effects
@@
 			)
 		)
-		(property "Footprint" "Resistor_THT:R_Axial_DIN0207_L6.3mm_D2.5mm_P7.62mm_Horizontal"
+		(property "Footprint" "Resistor_THT:R_Axial_DIN0207_L6.3mm_D2.5mm_P10.16mm_Horizontal"
 			(at 162.052 25.4 90)
 			(effects
@@
 			)
 		)
-		(property "Footprint" "Resistor_THT:R_Axial_DIN0207_L6.3mm_D2.5mm_P7.62mm_Horizontal"
+		(property "Footprint" "Resistor_THT:R_Axial_DIN0207_L6.3mm_D2.5mm_P10.16mm_Horizontal"
 			(at 154.432 25.4 90)
 			(effects
@@
 			)
 		)
-		(property "Footprint" "Resistor_THT:R_Axial_DIN0207_L6.3mm_D2.5mm_P7.62mm_Horizontal"
+		(property "Footprint" "Resistor_THT:R_Axial_DIN0207_L6.3mm_D2.5mm_P10.16mm_Horizontal"
 			(at 235.712 29.21 90)
 			(effects

Commit message: Maps footprints PCB -> sch
Parts:
- R16: footprint Resistor_THT:R_Axial_DIN0207_L6.3mm_D2.5mm_P10.16mm_Horizontal -> GDP:R_XL
Changed lines of the file:
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@@
 			)
 		)
-		(property "Footprint" "Resistor_THT:R_Axial_DIN0207_L6.3mm_D2.5mm_P10.16mm_Horizontal"
+		(property "Footprint" "GDP:R_XL"
 			(at 235.712 29.21 90)
 			(effects
