File: gdp/7.kicad_sch (KiCad schematic)
At the start: 9 parts, among them IC1 74LS74, IC15A 74LS367, IC2 74LS42, IC21 74LS374, IC28 74LS374, IC35 74LS374, IC38 74LS74, IC48 74LS374, IC9 74LS374

Commit message: Fixes refs
Parts:
- renumbered IC38 to IC1, IC48 to IC16, IC9 to IC22, IC35 to IC25, IC2 to IC3, IC21 to IC42, IC28 to IC68, IC1 to IC8
Changed lines of the file:
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@@
 		(on_board yes)
 		(dnp no)
-		(property "Reference" "IC9"
+		(property "Reference" "IC22"
 			(at 196.85 125.095 0)
 			(effects
@@
 			(project "7"
 				(path "/8aa3aa38-5607-4b5d-be5c-e0763aff29b1"
-					(reference  "IC22")
-					(unit 1)
-				)
-			)
-			(project "gdp"
-				(path "/95aff260-2720-4733-a81d-a7a2136fdd14/953bb077-6bb4-4683-bd3b-895ed53ec170"
-					(reference  "IC9")
+					(reference "IC22")
+					(unit 1)
+				)
+			)
+			(project "gdp"
+				(path "/95aff260-2720-4733-a81d-a7a2136fdd14/953bb077-6bb4-4683-bd3b-895ed53ec170"
+					(reference "IC9")
 					(unit 1)
 				)
@@
 		(on_board yes)
 		(dnp no)
-		(property "Reference" "IC21"
+		(property "Reference" "IC42"
 			(at 124.46 22.225 0)
 			(effects
@@
 			(project "7"
 				(path "/8aa3aa38-5607-4b5d-be5c-e0763aff29b1"
-					(reference  "IC42")
-					(unit 1)
-				)
-			)
-			(project "gdp"
-				(path "/95aff260-2720-4733-a81d-a7a2136fdd14/953bb077-6bb4-4683-bd3b-895ed53ec170"
-					(reference  "IC48")
+					(reference "IC42")
+					(unit 1)
+				)
+			)
+			(project "gdp"
+				(path "/95aff260-2720-4733-a81d-a7a2136fdd14/953bb077-6bb4-4683-bd3b-895ed53ec170"
+					(reference "IC21")
 					(unit 1)
 				)
@@
 		(dnp no)
 		(fields_autoplaced yes)
-		(property "Reference" "IC1"
-			(at 122.2091 164.465 0)
+		(property "Reference" "IC8"
+			(at 122.2091 165.1 0)
 			(effects
 				(font
@@
 		)
 		(property "Value" "74LS74"
-			(at 122.2091 167.005 0)
+			(at 122.2091 167.64 0)
 			(effects
 				(font
@@
 			(project "7"
 				(path "/8aa3aa38-5607-4b5d-be5c-e0763aff29b1"
-					(reference  "IC8")
-					(unit 1)
-				)
-			)
-			(project "gdp"
-				(path "/95aff260-2720-4733-a81d-a7a2136fdd14/953bb077-6bb4-4683-bd3b-895ed53ec170"
-					(reference  "IC21")
+					(reference "IC8")
+					(unit 1)
+				)
+			)
+			(project "gdp"
+				(path "/95aff260-2720-4733-a81d-a7a2136fdd14/953bb077-6bb4-4683-bd3b-895ed53ec170"
+					(reference "IC1")
 					(unit 1)
 				)
@@
 		(on_board yes)
 		(dnp no)
-		(property "Reference" "IC2"
+		(property "Reference" "IC3"
 			(at 119.38 135.89 0)
 			(effects
@@
 			(project "7"
 				(path "/8aa3aa38-5607-4b5d-be5c-e0763aff29b1"
-					(reference  "IC3")
-					(unit 1)
-				)
-			)
-			(project "gdp"
-				(path "/95aff260-2720-4733-a81d-a7a2136fdd14/953bb077-6bb4-4683-bd3b-895ed53ec170"
-					(reference  "IC1")
+					(reference "IC3")
+					(unit 1)
+				)
+			)
+			(project "gdp"
+				(path "/95aff260-2720-4733-a81d-a7a2136fdd14/953bb077-6bb4-4683-bd3b-895ed53ec170"
+					(reference "IC2")
 					(unit 1)
 				)
@@
 		(on_board yes)
 		(dnp no)
-		(property "Reference" "IC38"
+		(property "Reference" "IC1"
 			(at 80.01 172.72 0)
 			(effects
@@
 			(project "gdp"
 				(path "/95aff260-2720-4733-a81d-a7a2136fdd14/953bb077-6bb4-4683-bd3b-895ed53ec170"
-					(reference  "IC21")
+					(reference "IC1")
 					(unit 3)
 				)
@@
 		(on_board yes)
 		(dnp no)
-		(property "Reference" "IC28"
+		(property "Reference" "IC68"
 			(at 196.85 22.225 0)
 			(effects
@@
 			(project "7"
 				(path "/8aa3aa38-5607-4b5d-be5c-e0763aff29b1"
-					(reference  "IC68")
-					(unit 1)
-				)
-			)
-			(project "gdp"
-				(path "/95aff260-2720-4733-a81d-a7a2136fdd14/953bb077-6bb4-4683-bd3b-895ed53ec170"
-					(reference  "IC28")
+					(reference "IC68")
+					(unit 1)
+				)
+			)
+			(project "gdp"
+				(path "/95aff260-2720-4733-a81d-a7a2136fdd14/953bb077-6bb4-4683-bd3b-895ed53ec170"
+					(reference "IC28")
 					(unit 1)
 				)
@@
 		(on_board yes)
 		(dnp no)
-		(property "Reference" "IC48"
+		(property "Reference" "IC16"
 			(at 124.46 73.66 0)
 			(effects
@@
 			(project "7"
 				(path "/8aa3aa38-5607-4b5d-be5c-e0763aff29b1"
-					(reference  "IC16")
-					(unit 1)
-				)
-			)
-			(project "gdp"
-				(path "/95aff260-2720-4733-a81d-a7a2136fdd14/953bb077-6bb4-4683-bd3b-895ed53ec170"
-					(reference  "IC2")
+					(reference "IC16")
+					(unit 1)
+				)
+			)
+			(project "gdp"
+				(path "/95aff260-2720-4733-a81d-a7a2136fdd14/953bb077-6bb4-4683-bd3b-895ed53ec170"
+					(reference "IC48")
 					(unit 1)
 				)
@@
 		(on_board yes)
 		(dnp no)
-		(property "Reference" "IC35"
+		(property "Reference" "IC25"
 			(at 196.85 73.66 0)
 			(effects
@@
 			(project "7"
 				(path "/8aa3aa38-5607-4b5d-be5c-e0763aff29b1"
-					(reference  "IC25")
-					(unit 1)
-				)
-			)
-			(project "gdp"
-				(path "/95aff260-2720-4733-a81d-a7a2136fdd14/953bb077-6bb4-4683-bd3b-895ed53ec170"
-					(reference  "IC35")
+					(reference "IC25")
+					(unit 1)
+				)
+			)
+			(project "gdp"
+				(path "/95aff260-2720-4733-a81d-a7a2136fdd14/953bb077-6bb4-4683-bd3b-895ed53ec170"
+					(reference "IC35")
 					(unit 1)
 				)
@@
 			(project "gdp"
 				(path "/95aff260-2720-4733-a81d-a7a2136fdd14/953bb077-6bb4-4683-bd3b-895ed53ec170"
-					(reference  "IC15")
-					(unit 1)
-				)
+					(reference "IC15")
+					(unit 1)
+				)

Commit message: Schema fixes
Changed lines of the file:
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@@
-	)
-	(junction
-		(at 119.38 102.87)
-		(diameter 0)
-		(color 0 0 0 0)
 	)
 	(junction

Commit message: Re-annotates symbols
Parts:
- removed IC1: 74LS74, Package_DIP:DIP-14_W7.62mm, symbol 74xx:74LS74
Changed lines of the file:
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@@
-	)
-	(symbol
-		(lib_id "power:+5V")
-		(at 80.01 163.83 0)
-		(unit 1)
-		(exclude_from_sim no)
-		(in_bom yes)
-		(on_board yes)
-		(dnp no)
-		(property "Reference" "#PWR087"
-			(at 80.01 167.64 0)
-			(effects
-				(font
-					(size 1.27 1.27)
-				)
-				(hide yes)
-			)
-		)
-		(property "Value" "+5V"
-			(at 80.01 159.385 0)
-			(effects
-				(font
-					(size 1.27 1.27)
-				)
-			)
-		)
-		(property "Footprint" ""
-			(at 80.01 163.83 0)
-			(effects
-				(font
-					(size 1.27 1.27)
-				)
-				(hide yes)
-			)
-		)
-		(property "Datasheet" ""
-			(at 80.01 163.83 0)
-			(effects
-				(font
-					(size 1.27 1.27)
-				)
-				(hide yes)
-			)
-		)
-		(property "Description" ""
-			(at 80.01 163.83 0)
-			(effects
-				(font
-					(size 1.27 1.27)
-				)
-				(hide yes)
-			)
-		)
-		(pin "1"
-		)
-		(instances
-			(project "gdp"
-				(path "/95aff260-2720-4733-a81d-a7a2136fdd14/953bb077-6bb4-4683-bd3b-895ed53ec170"
-					(reference "#PWR087")
-					(unit 1)
-				)
-			)
-		)
-	)
-	(symbol
-		(lib_id "power:GNDD")
-		(at 80.01 184.15 0)
-		(unit 1)
-		(exclude_from_sim no)
-		(in_bom yes)
-		(on_board yes)
-		(dnp no)
-		(fields_autoplaced yes)
-		(property "Reference" "#PWR088"
-			(at 80.01 190.5 0)
-			(effects
-				(font
-					(size 1.27 1.27)
-				)
-				(hide yes)
-			)
-		)
-		(property "Value" "GNDD"
-			(at 80.01 187.96 0)
-			(effects
-				(font
-					(size 1.27 1.27)
-				)
-				(hide yes)
-			)
-		)
-		(property "Footprint" ""
-			(at 80.01 184.15 0)
-			(effects
-				(font
-					(size 1.27 1.27)
-				)
-				(hide yes)
-			)
-		)
-		(property "Datasheet" ""
-			(at 80.01 184.15 0)
-			(effects
-				(font
-					(size 1.27 1.27)
-				)
-				(hide yes)
-			)
-		)
-		(property "Description" ""
-			(at 80.01 184.15 0)
-			(effects
-				(font
-					(size 1.27 1.27)
-				)
-				(hide yes)
-			)
-		)
-		(pin "1"
-		)
-		(instances
-			(project "gdp"
-				(path "/95aff260-2720-4733-a81d-a7a2136fdd14/953bb077-6bb4-4683-bd3b-895ed53ec170"
-					(reference "#PWR088")
-					(unit 1)
-				)
-			)
-		)
 	)
 	(symbol
@@
 				)
 			)
-		)
-	)
-	(symbol
-		(lib_id "74xx:74LS74")
-		(at 80.01 173.99 0)
-		(unit 3)
-		(exclude_from_sim no)
-		(in_bom yes)
-		(on_board yes)
-		(dnp no)
-		(property "Reference" "IC1"
-			(at 80.01 172.72 0)
-			(effects
-				(font
-					(size 1.27 1.27)
-				)
-			)
-		)
-		(property "Value" "74LS74"
-			(at 80.01 175.26 0)
-			(effects
-				(font
-					(size 1.27 1.27)
-				)
-			)
-		)
-		(property "Footprint" "Package_DIP:DIP-14_W7.62mm"
-			(at 80.01 173.99 0)
-			(effects
-				(font
-					(size 1.27 1.27)
-				)
-				(hide yes)
-			)
-		)
-		(property "Datasheet" "N/A"
-			(at 80.01 173.99 0)
-			(effects
-				(font
-					(size 1.27 1.27)
-				)
-				(hide yes)
-			)
-		)
-		(property "Description" "N/A"
-			(at 80.01 173.99 0)
-			(effects
-				(font
-					(size 1.27 1.27)
-				)
-				(hide yes)
-			)
-		)
-		(pin "1"
-		)
-		(pin "2"
-		)
-		(pin "3"
-		)
-		(pin "4"
-		)
-		(pin "5"
-		)
-		(pin "6"
-		)
-		(pin "10"
-		)
-		(pin "11"
-		)
-		(pin "12"
-		)
-		(pin "13"
-		)
-		(pin "8"
-		)
-		(pin "9"
-		)
-		(pin "14"
-		)
-		(pin "7"
-		)
-		(instances
-			(project "gdp"
-				(path "/95aff260-2720-4733-a81d-a7a2136fdd14/953bb077-6bb4-4683-bd3b-895ed53ec170"
-					(reference "IC1")
-					(unit 3)
-				)
-			)

Commit message: Fixes GND
Connections:
- net GNDD renamed GND
Changed lines of the file:
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@@
 			)
 		)
-		(property "Value" "GNDD"
+		(property "Value" "GND"
 			(at 119.38 106.68 0)
 			(effects

Commit message: Fixes "CA0" issue in schematics
Parts:
- renumbered IC8 to IC1, IC15A to IC15, IC3 to IC2, IC42 to IC21, IC68 to IC28, IC25 to IC35, IC16 to IC48, IC22 to IC9
Changed lines of the file:
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@@
 (kicad_sch
-	(version 20231120)
+	(version 20250114)
 	(generator "eeschema")
-	(generator_version "8.0")
+	(generator_version "9.0")
 	(paper "A4")
 	(title_block
@@
 	(label "D4"
 		(at 173.99 142.875 0)
-		(fields_autoplaced yes)
 		(effects
 			(font
@@
 	(label "D2"
 		(at 173.99 34.925 0)
-		(fields_autoplaced yes)
 		(effects
 			(font
@@
 	(label "D4"
 		(at 173.99 40.005 0)
-		(fields_autoplaced yes)
 		(effects
 			(font
@@
 	(label "D6"
 		(at 173.99 45.085 0)
-		(fields_autoplaced yes)
 		(effects
 			(font
@@
 	(label "D5"
 		(at 173.99 145.415 0)
-		(fields_autoplaced yes)
 		(effects
 			(font
@@
 	(label "D2"
 		(at 173.99 137.795 0)
-		(fields_autoplaced yes)
 		(effects
 			(font
@@
 	(label "D0"
 		(at 173.99 29.845 0)
-		(fields_autoplaced yes)
 		(effects
 			(font
@@
 	(label "D3"
 		(at 173.99 140.335 0)
-		(fields_autoplaced yes)
 		(effects
 			(font
@@
 	(label "D7"
 		(at 173.99 47.625 0)
-		(fields_autoplaced yes)
 		(effects
 			(font
@@
 	(label "D1"
 		(at 173.99 135.255 0)
-		(fields_autoplaced yes)
 		(effects
 			(font
@@
 	(label "D1"
 		(at 173.99 32.385 0)
-		(fields_autoplaced yes)
 		(effects
 			(font
@@
 	(label "D7"
 		(at 173.99 99.06 0)
-		(fields_autoplaced yes)
 		(effects
 			(font
@@
 	(label "D0"
 		(at 173.99 81.28 0)
-		(fields_autoplaced yes)
 		(effects
 			(font
@@
 	(label "D5"
 		(at 173.99 93.98 0)
-		(fields_autoplaced yes)
 		(effects
 			(font
@@
 	(label "D7"
 		(at 173.99 150.495 0)
-		(fields_autoplaced yes)
 		(effects
 			(font
@@
 	(label "D3"
 		(at 173.99 88.9 0)
-		(fields_autoplaced yes)
 		(effects
 			(font
@@
 	(label "D7"
 		(at 164.465 172.085 0)
-		(fields_autoplaced yes)
 		(effects
 			(font
@@
 	(label "D6"
 		(at 173.99 96.52 0)
-		(fields_autoplaced yes)
 		(effects
 			(font
@@
 	(label "D2"
 		(at 173.99 86.36 0)
-		(fields_autoplaced yes)
 		(effects
 			(font
@@
 	(label "D4"
 		(at 164.465 177.165 0)
-		(fields_autoplaced yes)
 		(effects
 			(font
@@
 	(label "D3"
 		(at 173.99 37.465 0)
-		(fields_autoplaced yes)
 		(effects
 			(font
@@
 	(label "D4"
 		(at 173.99 91.44 0)
-		(fields_autoplaced yes)
 		(effects
 			(font
@@
 	(label "D1"
 		(at 173.99 83.82 0)
-		(fields_autoplaced yes)
 		(effects
 			(font
@@
 	(label "D6"
 		(at 173.99 147.955 0)
-		(fields_autoplaced yes)
 		(effects
 			(font
@@
 	(label "D5"
 		(at 173.99 42.545 0)
-		(fields_autoplaced yes)
 		(effects
 			(font
@@
 	(label "D0"
 		(at 173.99 132.715 0)
-		(fields_autoplaced yes)
 		(effects
 			(font
@@
 		(on_board yes)
 		(dnp no)
-		(property "Reference" "#PWR?"
+		(property "Reference" "#PWR090"
 			(at 119.38 22.225 0)
 			(effects
@@
 		(on_board yes)
 		(dnp no)
-		(property "Reference" "#PWR?"
+		(property "Reference" "#PWR0102"
 			(at 191.77 73.66 0)
 			(effects
@@
 		(dnp no)
 		(fields_autoplaced yes)
-		(property "Reference" "#PWR?"
+		(property "Reference" "#PWR096"
 			(at 119.38 160.655 0)
 			(effects
@@
 		(dnp no)
 		(fields_autoplaced yes)
-		(property "Reference" "#PWR?"
+		(property "Reference" "#PWR093"
 			(at 119.38 109.22 0)
 			(effects
@@
 		(on_board yes)
 		(dnp no)
-		(property "Reference" "IC22"
+		(property "Reference" "IC9"
 			(at 196.85 125.095 0)
 			(effects
@@
 		(dnp no)
 		(fields_autoplaced yes)
-		(property "Reference" "#PWR?"
+		(property "Reference" "#PWR0103"
 			(at 191.77 109.22 0)
 			(effects
@@
 		(dnp no)
 		(fields_autoplaced yes)
-		(property "Reference" "#PWR?"
+		(property "Reference" "#PWR091"
 			(at 119.38 57.785 0)
 			(effects
@@
 		(on_board yes)
 		(dnp no)
-		(property "Reference" "#PWR?"
+		(property "Reference" "#PWR0100"
 			(at 191.77 22.225 0)
 			(effects
@@
 		(on_board yes)
 		(dnp no)
-		(property "Reference" "IC42"
+		(property "Reference" "IC21"
 			(at 124.46 22.225 0)
 			(effects
@@
 		(dnp no)
 		(fields_autoplaced yes)
-		(property "Reference" "IC8"
+		(property "Reference" "IC1"
 			(at 122.2091 165.1 0)
 			(effects
@@
 		(on_board yes)
 		(dnp no)
-		(property "Reference" "#PWR?"
+		(property "Reference" "#PWR095"
 			(at 119.38 125.095 0)
 			(effects
@@
 		(on_board yes)
 		(dnp no)
-		(property "Reference" "IC3"
+		(property "Reference" "IC2"
 			(at 119.38 135.89 0)
 			(effects
@@
 		(dnp no)
 		(fields_autoplaced yes)
-		(property "Reference" "#PWR?"
+		(property "Reference" "#PWR0101"
 			(at 191.77 57.785 0)
 			(effects
@@
 		(on_board yes)
 		(dnp no)
-		(property "Reference" "#PWR?"
+		(property "Reference" "#PWR097"
 			(at 151.765 160.655 0)
 			(effects
@@
 		(on_board yes)
 		(dnp no)
-		(property "Reference" "#PWR?"
+		(property "Reference" "#PWR0104"
 			(at 191.77 125.095 0)
 			(effects
@@
 		(on_board yes)
 		(dnp no)
-		(property "Reference" "IC68"
+		(property "Reference" "IC28"
 			(at 196.85 22.225 0)
 			(effects
@@
 		(on_board yes)
 		(dnp no)
-		(property "Reference" "#PWR?"
+		(property "Reference" "#PWR092"
 			(at 119.38 73.66 0)
 			(effects
@@
 		(on_board yes)
 		(dnp no)
-		(property "Reference" "#PWR?"
+		(property "Reference" "#PWR089"
 			(at 110.49 169.545 0)
 			(effects
@@
 		(on_board yes)
 		(dnp no)
-		(property "Reference" "IC16"
+		(property "Reference" "IC48"
 			(at 124.46 73.66 0)
 			(effects
@@
 		(dnp no)
 		(fields_autoplaced yes)
-		(property "Reference" "#PWR?"
+		(property "Reference" "#PWR0105"
 			(at 191.77 160.655 0)
 			(effects
@@
 		(on_board yes)
 		(dnp no)
-		(property "Reference" "IC25"
+		(property "Reference" "IC35"
 			(at 196.85 73.66 0)
 			(effects
@@
 		(on_board yes)
 		(dnp no)
-		(property "Reference" "IC15A"
+		(property "Reference" "IC15"
 			(at 151.511 165.735 0)
 			(effects
@@
 		(dnp no)
 		(fields_autoplaced yes)
-		(property "Reference" "#PWR?"
+		(property "Reference" "#PWR094"
 			(at 119.38 109.22 0)
 			(effects
@@
 		(dnp no)
 		(fields_autoplaced yes)
-		(property "Reference" "#PWR?"
+		(property "Reference" "#PWR099"
 			(at 179.07 135.255 0)
 			(effects
@@
 		(dnp no)
 		(fields_autoplaced yes)
-		(property "Reference" "#PWR?"
+		(property "Reference" "#PWR098"
 			(at 151.765 188.595 0)
 			(effects
@@
 		)
 	)
+	(embedded_fonts no)
 )
