File: gdp/5.kicad_sch (KiCad schematic)
At the start: 0 parts

Commit message: Adds pages 4, 7, 10 (still WIP)
Other:
- title: Partner GDP -> (none)
Changed lines of the file:
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@@
 (kicad_sch (version 20230121) (generator eeschema)
   (paper "A4")
-  (title_block
-    (title "Partner GDP")
-  )
 )

Commit message: Adds Sheet 5
Parts:
- added R10, R14, R15, R16, R17, R21, R24, R25, R26, R27, R28, R29, R30, R31, R8, R9: 330R, symbol Device:R
- added U3, U4: 74LS166, symbol 74xx:74LS166
- added U5, U6: 74LS30, symbol 74xx:74LS30
- added U7, U8: 74LS538, symbol 74xx:74LS166
Connections:
- new net: U3.1 (Ds), U4.13 (Qh)
- new net +5V: R10.1, R14.1, R15.1, R16.1, R17.1, R21.1, R24.1, R25.1, R26.1, R27.1, R28.1, R29.1, R30.1, R31.1, R8.1, R9.1, U3.16 (VCC), U4.1 (Ds), U4.16 (VCC), U5.14 (VCC), U6.14 (VCC), U7.20 (VCC), U8.20 (VCC)
- new net ALL1: U8.15 (G3)
- new net DOUT1: U6.8
- new net DOUT2: U5.8
- new net GDO0: R21.2, U3.14 (H), U6.12
- new net GDO1: R17.2, U3.12 (G), U6.11
- new net GDO10: R26.2, U4.11 (F), U5.6
- new net GDO11: R27.2, U4.10 (E), U5.5
- new net GDO12: R28.2, U4.5 (D), U5.4
- new net GDO13: R29.2, U4.4 (C), U5.3
- new net GDO14: R30.2, U4.3 (B), U5.2
- new net GDO15: R31.2, U4.2 (A), U5.1
- new net GDO2: R16.2, U3.11 (F), U6.6
- new net GDO3: R15.2, U3.10 (E), U6.5
- new net GDO4: R14.2, U3.5 (D), U6.4
- new net GDO5: R10.2, U3.4 (C), U6.3
- new net GDO6: R9.2, U3.3 (B), U6.2
- new net GDO7: R8.2, U3.2 (A), U6.1
- new net GDO8: R24.2, U4.14 (H), U5.12
- new net GDO9: R25.2, U4.12 (G), U5.11
- new net GND: U3.6 (CE), U3.8 (GND), U4.6 (CE), U4.8 (GND), U5.7 (GND), U6.7 (GND), U7.10 (GND), U7.4 (OE1), U7.5 (OE2), U8.10 (GND), U8.4 (OE1), U8.5 (OE2)
- new net OC: U7.14 (G2), U8.14 (G2)
- new net RAS0: U7.3 (Y0)
- new net RAS1: U7.2 (Y1)
- new net RAS10: U8.1 (Y2)
- new net RAS11: U8.19 (Y3)
- new net RAS12: U8.18 (Y4)
- new net RAS13: U8.8 (Y5)
- new net RAS14: U8.9 (Y6)
- new net RAS15: U8.11 (Y7)
- new net RAS2: U7.1 (Y2)
- new net RAS3: U7.19 (Y3)
- new net RAS4: U7.18 (Y4)
- new net RAS5: U7.8 (Y5)
- new net RAS6: U7.9 (Y6)
- new net RAS7: U7.11 (Y7)
- new net RAS8: U8.3 (Y0)
- new net RAS9: U8.2 (Y1)
- new net SHLD: U3.15 (PE), U4.15 (PE)
- new net X0: U7.6 (A), U8.6 (A)
- new net X1: U7.7 (B), U8.7 (B)
- new net X2: U7.17 (C), U8.17 (C)
- new net X3: U7.15 (G3), U8.13 (G1)
- new net ~{ALL16}: U7.12 (AL), U8.12 (AL)
- new net ~{ALL}: U7.13 (G1)
- new net ~{ENS}: U7.16 (G4), U8.16 (G4)
- new net ~{GVID}: U3.13 (Qh)
- new net ~{HCK}: U3.7 (Clk), U4.7 (Clk)
- new net ~{WHITE}: U3.9 (Clr), U4.9 (Clr)
Other:
- company: (none) -> Oddbit Retro
- title: (none) -> PARTNER GDP: MEMOUT + RAS/SELECT

Commit message: Fixes Sheet 5
Parts:
- added R55, R56: 2K2, symbol Device:R
Connections:
- net GND: now also R55.2, R56.2
- net SHLD: now also R56.1
- net ~{HCK}: now also R55.1

Commit message: Adds Sheet 9
Parts:
- removed R10, R14, R15, R16, R17, R21, R24, R25, R26, R27, R28, R29, R30, R31, R8, R9: 330R, symbol Device:R
- added RN2, RN3: 8x2K2, Resistor_THT:R_Array_SIP9, symbol Device:R_Network08
- renumbered U8 to IC29, U7 to IC30, U4 to IC67, U5 to IC68, U3 to IC69, U6 to IC70, R55 to R49, R56 to R53
Connections:
- net +5V: now also RN2.1 (common), RN3.1 (common)
- net GDO0: now also RN2.2 (R1)
- net GDO1: now also RN2.3 (R2)
- net GDO10: now also RN3.4 (R3)
- net GDO11: now also RN3.5 (R4)
- net GDO12: now also RN3.6 (R5)
- net GDO13: now also RN3.7 (R6)
- net GDO14: now also RN3.8 (R7)
- net GDO15: now also RN3.9 (R8)
- net GDO2: now also RN2.4 (R3)
- net GDO3: now also RN2.5 (R4)
- net GDO4: now also RN2.6 (R5)
- net GDO5: now also RN2.7 (R6)
- net GDO6: now also RN2.8 (R7)
- net GDO7: now also RN2.9 (R8)
- net GDO8: now also RN3.2 (R1)
- net GDO9: now also RN3.3 (R2)

Commit message: Adds Sheet 11
Changed lines of the file:
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@@
 	(wire
 		(pts
-			(xy 115.57 142.24) (xy 115.57 139.7)
-		)
-		(stroke
-			(width 0)
-			(type default)
-		)
-	)
-	(wire
-		(pts
 			(xy 107.95 119.38) (xy 107.95 147.32)
 		)
@@
 	(wire
 		(pts
-			(xy 115.57 139.7) (xy 113.03 139.7)
+			(xy 115.57 142.24) (xy 113.03 142.24)
 		)
 		(stroke
@@
 	(wire
 		(pts
-			(xy 113.03 50.8) (xy 115.57 50.8)
+			(xy 113.03 53.34) (xy 115.57 53.34)
 		)
 		(stroke
@@
 	(wire
 		(pts
-			(xy 115.57 53.34) (xy 115.57 50.8)
-		)
-		(stroke
-			(width 0)
-			(type default)
-		)
-	)
-	(wire
-		(pts
 			(xy 177.8 58.42) (xy 190.5 58.42)
 		)
@@
 	(symbol
 		(lib_id "power:GNDD")
-		(at 113.03 139.7 0)
+		(at 113.03 142.24 180)
 		(unit 1)
 		(exclude_from_sim no)
@@
 		(fields_autoplaced yes)
 		(property "Reference" "#PWR091"
-			(at 113.03 146.05 0)
+			(at 113.03 135.89 0)
 			(effects
 				(font
@@
 		)
 		(property "Value" "GND"
-			(at 113.03 143.51 0)
+			(at 113.03 137.16 0)
 			(effects
 				(font
@@
 		)
 		(property "Footprint" ""
-			(at 113.03 139.7 0)
+			(at 113.03 142.24 0)
 			(effects
 				(font
@@
 		)
 		(property "Datasheet" ""
-			(at 113.03 139.7 0)
+			(at 113.03 142.24 0)
 			(effects
 				(font
@@
 		)
 		(property "Description" "Power symbol creates a global label with name \"GNDD\" , digital ground"
-			(at 113.03 139.7 0)
+			(at 113.03 142.24 0)
 			(effects
 				(font
@@
 	(symbol
 		(lib_id "power:GNDD")
-		(at 113.03 50.8 0)
+		(at 113.03 53.34 180)
 		(unit 1)
 		(exclude_from_sim no)
@@
 		(fields_autoplaced yes)
 		(property "Reference" "#PWR092"
-			(at 113.03 57.15 0)
+			(at 113.03 46.99 0)
 			(effects
 				(font
@@
 		)
 		(property "Value" "GND"
-			(at 113.03 54.61 0)
+			(at 113.03 48.26 0)
 			(effects
 				(font
@@
 		)
 		(property "Footprint" ""
-			(at 113.03 50.8 0)
+			(at 113.03 53.34 0)
 			(effects
 				(font
@@
 		)
 		(property "Datasheet" ""
-			(at 113.03 50.8 0)
+			(at 113.03 53.34 0)
 			(effects
 				(font
@@
 		)
 		(property "Description" "Power symbol creates a global label with name \"GNDD\" , digital ground"
-			(at 113.03 50.8 0)
+			(at 113.03 53.34 0)
 			(effects
 				(font

Commit message: Adds Sheet 12
Other:
- moved on the sheet: IC30
Changed lines of the file:
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@@
 	)
 	(junction
-		(at 208.28 46.99)
+		(at 209.55 46.99)
 		(diameter 0)
 		(color 0 0 0 0)
@@
 	(wire
 		(pts
-			(xy 190.5 58.42) (xy 208.28 58.42)
+			(xy 190.5 58.42) (xy 209.55 58.42)
 		)
 		(stroke
@@
 	(wire
 		(pts
-			(xy 187.96 64.77) (xy 208.28 64.77)
+			(xy 187.96 64.77) (xy 209.55 64.77)
 		)
 		(stroke
@@
 	(wire
 		(pts
-			(xy 193.04 55.88) (xy 208.28 55.88)
+			(xy 193.04 55.88) (xy 209.55 55.88)
 		)
 		(stroke
@@
 	(wire
 		(pts
-			(xy 233.68 52.07) (xy 261.62 52.07)
+			(xy 234.95 52.07) (xy 261.62 52.07)
 		)
 		(stroke
@@
 	(wire
 		(pts
-			(xy 201.93 46.99) (xy 208.28 46.99)
+			(xy 201.93 46.99) (xy 209.55 46.99)
 		)
 		(stroke
@@
 	(wire
 		(pts
-			(xy 233.68 57.15) (xy 261.62 57.15)
+			(xy 234.95 57.15) (xy 261.62 57.15)
 		)
 		(stroke
@@
 	(wire
 		(pts
-			(xy 233.68 64.77) (xy 261.62 64.77)
+			(xy 234.95 64.77) (xy 261.62 64.77)
 		)
 		(stroke
@@
 	(wire
 		(pts
-			(xy 233.68 69.85) (xy 261.62 69.85)
+			(xy 234.95 69.85) (xy 261.62 69.85)
 		)
 		(stroke
@@
 	(wire
 		(pts
-			(xy 233.68 62.23) (xy 261.62 62.23)
+			(xy 234.95 62.23) (xy 261.62 62.23)
 		)
 		(stroke
@@
 	(wire
 		(pts
-			(xy 233.68 59.69) (xy 261.62 59.69)
+			(xy 234.95 59.69) (xy 261.62 59.69)
 		)
 		(stroke
@@
 	(wire
 		(pts
-			(xy 198.12 43.18) (xy 208.28 43.18)
+			(xy 198.12 43.18) (xy 209.55 43.18)
 		)
 		(stroke
@@
 	(wire
 		(pts
-			(xy 177.8 62.23) (xy 208.28 62.23)
+			(xy 177.8 62.23) (xy 209.55 62.23)
 		)
 		(stroke
@@
 	(wire
 		(pts
-			(xy 195.58 53.34) (xy 208.28 53.34)
+			(xy 195.58 53.34) (xy 209.55 53.34)
 		)
 		(stroke
@@
 	(wire
 		(pts
-			(xy 233.68 54.61) (xy 261.62 54.61)
+			(xy 234.95 54.61) (xy 261.62 54.61)
 		)
 		(stroke
@@
 	(wire
 		(pts
-			(xy 208.28 46.99) (xy 208.28 49.53)
+			(xy 234.95 67.31) (xy 261.62 67.31)
 		)
 		(stroke
@@
 	(wire
 		(pts
-			(xy 233.68 67.31) (xy 261.62 67.31)
+			(xy 110.49 55.88) (xy 115.57 55.88)
 		)
 		(stroke
@@
 	(wire
 		(pts
-			(xy 110.49 55.88) (xy 115.57 55.88)
+			(xy 209.55 46.99) (xy 209.55 49.53)
 		)
 		(stroke
@@
 	(wire
 		(pts
-			(xy 182.88 69.85) (xy 208.28 69.85)
+			(xy 182.88 69.85) (xy 209.55 69.85)
 		)
 		(stroke
@@
 	(wire
 		(pts
-			(xy 185.42 67.31) (xy 208.28 67.31)
+			(xy 185.42 67.31) (xy 209.55 67.31)
 		)
 		(stroke
@@
 	(symbol
 		(lib_id "power:GNDD")
-		(at 220.98 81.28 0)
+		(at 222.25 81.28 0)
 		(unit 1)
 		(exclude_from_sim no)
@@
 		(fields_autoplaced yes)
 		(property "Reference" "#PWR095"
-			(at 220.98 87.63 0)
+			(at 222.25 87.63 0)
 			(effects
 				(font
@@
 		)
 		(property "Value" "GND"
-			(at 220.98 85.09 0)
+			(at 222.25 85.09 0)
 			(effects
 				(font
@@
 		)
 		(property "Footprint" ""
-			(at 220.98 81.28 0)
+			(at 222.25 81.28 0)
 			(effects
 				(font
@@
 		)
 		(property "Datasheet" ""
-			(at 220.98 81.28 0)
+			(at 222.25 81.28 0)
 			(effects
 				(font
@@
 		)
 		(property "Description" "Power symbol creates a global label with name \"GNDD\" , digital ground"
-			(at 220.98 81.28 0)
+			(at 222.25 81.28 0)
 			(effects
 				(font
@@
 	(symbol
 		(lib_id "power:+5V")
-		(at 220.98 30.48 0)
+		(at 222.25 30.48 0)
 		(unit 1)
 		(exclude_from_sim no)
@@
 		(fields_autoplaced yes)
 		(property "Reference" "#PWR094"
-			(at 220.98 34.29 0)
+			(at 222.25 34.29 0)
 			(effects
 				(font
@@
 		)
 		(property "Value" "+5V"
-			(at 220.98 25.4 0)
+			(at 222.25 25.4 0)
 			(effects
 				(font
@@
 		)
 		(property "Footprint" ""
-			(at 220.98 30.48 0)
+			(at 222.25 30.48 0)
 			(effects
 				(font
@@
 		)
 		(property "Datasheet" ""
-			(at 220.98 30.48 0)
+			(at 222.25 30.48 0)
 			(effects
 				(font
@@
 		)
 		(property "Description" "Power symbol creates a global label with name \"+5V\""
-			(at 220.98 30.48 0)
+			(at 222.25 30.48 0)
 			(effects
 				(font
@@
 		(lib_name "74LS166_1")
 		(lib_id "74xx:74LS166")
-		(at 220.98 55.88 0)
+		(at 222.25 55.88 0)
 		(unit 1)
 		(exclude_from_sim no)
@@
 		(fields_autoplaced yes)
 		(property "Reference" "IC30"
-			(at 226.822 30.988 0)
+			(at 228.092 30.988 0)
 			(do_not_autoplace yes)
 			(effects
@@
 		)
 		(property "Value" "74LS538"
-			(at 226.822 33.528 0)
+			(at 228.092 33.528 0)
 			(do_not_autoplace yes)
 			(effects
@@
 		)
 		(property "Footprint" ""
-			(at 220.98 55.88 0)
+			(at 222.25 55.88 0)
 			(effects
 				(font
@@
 		)
 		(property "Datasheet" "N/A"
-			(at 180.34 53.848 0)
+			(at 181.61 53.848 0)
 			(effects
 				(font
@@
 		)
 		(property "Description" "Decoder"
-			(at 180.34 50.292 0)
+			(at 181.61 50.292 0)
 			(effects
 				(font
