File: gdp/5.kicad_sch (KiCad schematic)
At the start: 10 parts, among them IC29 74LS538, IC30 74LS538, IC67 74LS166, IC68 74LS30, IC69 74LS166, IC70 74LS30

Commit message: Initial footprint assignment
Parts:
- IC27: renamed from IC70; footprint (none) -> Package_DIP:DIP-14_W7.62mm
- IC28: renamed from IC68; footprint (none) -> Package_DIP:DIP-14_W7.62mm
- IC29: renamed from IC69; footprint (none) -> Package_DIP:DIP-16_W7.62mm
- IC30: renamed from IC67; footprint (none) -> Package_DIP:DIP-16_W7.62mm
- IC31: renamed from IC30; footprint (none) -> Package_DIP:DIP-20_W7.62mm
- IC32: renamed from IC29; footprint (none) -> Package_DIP:DIP-20_W7.62mm
- R18: renamed from R49; footprint (none) -> Resistor_THT:R_Axial_DIN0207_L6.3mm_D2.5mm_P7.62mm_Horizontal
- R19: renamed from R53; footprint (none) -> Resistor_THT:R_Axial_DIN0207_L6.3mm_D2.5mm_P7.62mm_Horizontal
- renumbered RN2 to RN1, RN3 to RN2
