File: gdp/5.kicad_sch (KiCad schematic)
At the start: 10 parts, among them IC27 74LS30, IC28 74LS30, IC29 74LS166, IC30 74LS166, IC31 74LS538, IC32 74LS538

Commit message: Fixes refs
Parts:
- renumbered IC32 to IC29, IC31 to IC30, IC30 to IC67, IC28 to IC68, IC29 to IC69, IC27 to IC70, R18 to R49, R19 to R53, RN1 to RN2, RN2 to RN3
Changed lines of the file:
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@@
 		(dnp no)
 		(fields_autoplaced yes)
-		(property "Reference" "IC30"
+		(property "Reference" "IC67"
 			(at 134.112 132.588 0)
 			(do_not_autoplace yes)
@@
 			(project "gdp"
 				(path "/95aff260-2720-4733-a81d-a7a2136fdd14/c2399418-5be2-4a84-8b56-c34f01a784cb"
-					(reference  "IC67")
+					(reference "IC67")
 					(unit 1)
 				)
@@
 		(dnp no)
 		(fields_autoplaced yes)
-		(property "Reference" "RN2"
+		(property "Reference" "RN3"
 			(at 87.63 119.6339 0)
 			(effects
@@
 			(project "gdp"
 				(path "/95aff260-2720-4733-a81d-a7a2136fdd14/c2399418-5be2-4a84-8b56-c34f01a784cb"
-					(reference  "RN3")
+					(reference "RN3")
 					(unit 1)
 				)
@@
 		(on_board yes)
 		(dnp no)
-		(property "Reference" "IC28"
+		(property "Reference" "IC68"
 			(at 55.88 185.42 0)
 			(effects
@@
 			(project "gdp"
 				(path "/95aff260-2720-4733-a81d-a7a2136fdd14/c2399418-5be2-4a84-8b56-c34f01a784cb"
-					(reference  "IC68")
+					(reference "IC68")
 					(unit 2)
 				)
@@
 		(on_board yes)
 		(dnp no)
-		(property "Reference" "IC28"
+		(property "Reference" "IC68"
 			(at 53.594 155.956 0)
 			(effects
@@
 			(project ""
 				(path "/95aff260-2720-4733-a81d-a7a2136fdd14/c2399418-5be2-4a84-8b56-c34f01a784cb"
-					(reference  "IC68")
+					(reference "IC68")
 					(unit 1)
 				)
@@
 		(dnp no)
 		(fields_autoplaced yes)
-		(property "Reference" "IC29"
+		(property "Reference" "IC69"
 			(at 134.112 43.688 0)
 			(do_not_autoplace yes)
@@
 			(project ""
 				(path "/95aff260-2720-4733-a81d-a7a2136fdd14/c2399418-5be2-4a84-8b56-c34f01a784cb"
-					(reference  "IC69")
+					(reference "IC69")
 					(unit 1)
 				)
@@
 		(dnp no)
 		(fields_autoplaced yes)
-		(property "Reference" "IC32"
+		(property "Reference" "IC29"
 			(at 228.092 102.108 0)
 			(do_not_autoplace yes)
@@
 			(project "gdp"
 				(path "/95aff260-2720-4733-a81d-a7a2136fdd14/c2399418-5be2-4a84-8b56-c34f01a784cb"
-					(reference  "IC29")
+					(reference "IC29")
 					(unit 1)
 				)
@@
 		(on_board yes)
 		(dnp no)
-		(property "Reference" "IC27"
+		(property "Reference" "IC70"
 			(at 55.88 96.52 0)
 			(effects
@@
 			(project "gdp"
 				(path "/95aff260-2720-4733-a81d-a7a2136fdd14/c2399418-5be2-4a84-8b56-c34f01a784cb"
-					(reference  "IC70")
+					(reference "IC70")
 					(unit 2)
 				)
@@
 		(dnp no)
 		(fields_autoplaced yes)
-		(property "Reference" "IC31"
+		(property "Reference" "IC30"
 			(at 228.092 30.988 0)
 			(do_not_autoplace yes)
@@
 			(project "gdp"
 				(path "/95aff260-2720-4733-a81d-a7a2136fdd14/c2399418-5be2-4a84-8b56-c34f01a784cb"
-					(reference  "IC30")
+					(reference "IC30")
 					(unit 1)
 				)
@@
 		(on_board yes)
 		(dnp no)
-		(property "Reference" "R19"
+		(property "Reference" "R53"
 			(at 121.92 118.11 0)
 			(effects
@@
 			(project "gdp"
 				(path "/95aff260-2720-4733-a81d-a7a2136fdd14/c2399418-5be2-4a84-8b56-c34f01a784cb"
-					(reference  "R53")
+					(reference "R53")
 					(unit 1)
 				)
@@
 		(on_board yes)
 		(dnp no)
-		(property "Reference" "R18"
+		(property "Reference" "R49"
 			(at 121.92 111.76 0)
 			(effects
@@
 			(project "gdp"
 				(path "/95aff260-2720-4733-a81d-a7a2136fdd14/c2399418-5be2-4a84-8b56-c34f01a784cb"
-					(reference  "R49")
+					(reference "R49")
 					(unit 1)
 				)
@@
 		(dnp no)
 		(fields_autoplaced yes)
-		(property "Reference" "RN1"
+		(property "Reference" "RN2"
 			(at 87.63 30.7339 0)
 			(effects
@@
 			(project ""
 				(path "/95aff260-2720-4733-a81d-a7a2136fdd14/c2399418-5be2-4a84-8b56-c34f01a784cb"
-					(reference  "RN2")
+					(reference "RN2")
 					(unit 1)
 				)
@@
 		(on_board yes)
 		(dnp no)
-		(property "Reference" "IC27"
+		(property "Reference" "IC70"
 			(at 53.594 67.056 0)
 			(effects
@@
 			(project "gdp"
 				(path "/95aff260-2720-4733-a81d-a7a2136fdd14/c2399418-5be2-4a84-8b56-c34f01a784cb"
-					(reference  "IC70")
-					(unit 1)
-				)
+					(reference "IC70")
+					(unit 1)
+				)

Commit message: Placing footprints...
Parts:
- R49, R53: footprint Resistor_THT:R_Axial_DIN0207_L6.3mm_D2.5mm_P7.62mm_Horizontal -> Resistor_THT:R_Axial_DIN0207_L6.3mm_D2.5mm_P10.16mm_Horizontal
Changed lines of the file:
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@@
 			)
 		)
-		(property "Footprint" "Resistor_THT:R_Axial_DIN0207_L6.3mm_D2.5mm_P7.62mm_Horizontal"
+		(property "Footprint" "Resistor_THT:R_Axial_DIN0207_L6.3mm_D2.5mm_P10.16mm_Horizontal"
 			(at 123.19 121.158 90)
 			(effects
@@
 			)
 		)
-		(property "Footprint" "Resistor_THT:R_Axial_DIN0207_L6.3mm_D2.5mm_P7.62mm_Horizontal"
+		(property "Footprint" "Resistor_THT:R_Axial_DIN0207_L6.3mm_D2.5mm_P10.16mm_Horizontal"
 			(at 123.19 114.808 90)
 			(effects

Commit message: Maps footprints PCB -> sch
Parts:
- R49, R53: footprint Resistor_THT:R_Axial_DIN0207_L6.3mm_D2.5mm_P10.16mm_Horizontal -> GDP:R_XL
- renumbered RN3 to RN2, RN2 to RN3
Changed lines of the file:
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@@
 		(dnp no)
 		(fields_autoplaced yes)
-		(property "Reference" "RN3"
+		(property "Reference" "RN2"
 			(at 87.63 119.6339 0)
 			(effects
@@
 			(project "gdp"
 				(path "/95aff260-2720-4733-a81d-a7a2136fdd14/c2399418-5be2-4a84-8b56-c34f01a784cb"
-					(reference "RN3")
+					(reference "RN2")
 					(unit 1)
 				)
@@
 			)
 		)
-		(property "Footprint" "Resistor_THT:R_Axial_DIN0207_L6.3mm_D2.5mm_P10.16mm_Horizontal"
+		(property "Footprint" "GDP:R_XL"
 			(at 123.19 121.158 90)
 			(effects
@@
 			)
 		)
-		(property "Footprint" "Resistor_THT:R_Axial_DIN0207_L6.3mm_D2.5mm_P10.16mm_Horizontal"
+		(property "Footprint" "GDP:R_XL"
 			(at 123.19 114.808 90)
 			(effects
@@
 		(dnp no)
 		(fields_autoplaced yes)
-		(property "Reference" "RN2"
+		(property "Reference" "RN3"
 			(at 87.63 30.7339 0)
 			(effects
@@
 			(project ""
 				(path "/95aff260-2720-4733-a81d-a7a2136fdd14/c2399418-5be2-4a84-8b56-c34f01a784cb"
-					(reference "RN2")
-					(unit 1)
-				)
+					(reference "RN3")
+					(unit 1)
+				)

Commit message: Final fixes
Parts:
- IC68, IC70: now in the parts list
Connections:
- net GDO0: now also IC70.3; no longer IC70.12
- net GDO1: now also IC70.2; no longer IC70.11
- net GDO10: now also IC68.5; no longer IC68.6
- net GDO11: now also IC68.4; no longer IC68.5
- net GDO12: now also IC68.6; no longer IC68.4
- net GDO13: now also IC68.2; no longer IC68.3
- net GDO14: now also IC68.3; no longer IC68.2
- net GDO3: now also IC70.11; no longer IC70.5
- net GDO4: now also IC70.5; no longer IC70.4
- net GDO5: now also IC70.4; no longer IC70.3
- net GDO6: now also IC70.12; no longer IC70.2
Changed lines of the file:
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@@
 	)
 	(symbol
+		(lib_name "74LS30_3")
 		(lib_id "74xx:74LS30")
 		(at 57.15 185.42 270)
 		(unit 2)
 		(exclude_from_sim no)
-		(in_bom no)
+		(in_bom yes)
 		(on_board yes)
 		(dnp no)
 		(property "Reference" "IC68"
-			(at 55.88 185.42 0)
+			(at 55.626 185.42 0)
 			(effects
 				(font
@@
 		)
 		(property "Value" "74LS30"
-			(at 58.42 185.42 0)
+			(at 58.166 185.42 0)
 			(effects
 				(font
@@
 		)
 		(property "Footprint" "Package_DIP:DIP-14_W7.62mm"
-			(at 57.15 185.42 0)
+			(at 45.212 185.42 0)
 			(effects
 				(font
@@
 		)
 		(property "Footprint" "Package_DIP:DIP-14_W7.62mm"
-			(at 54.61 165.1 0)
+			(at 54.61 153.162 0)
 			(effects
 				(font
@@
 	)
 	(symbol
+		(lib_name "74LS30_1")
 		(lib_id "74xx:74LS30")
 		(at 57.15 96.52 270)
 		(unit 2)
 		(exclude_from_sim no)
-		(in_bom no)
+		(in_bom yes)
 		(on_board yes)
 		(dnp no)
@@
 		)
 		(property "Footprint" "Package_DIP:DIP-14_W7.62mm"
-			(at 57.15 96.52 0)
+			(at 45.212 96.52 0)
 			(effects
 				(font
@@
 	)
 	(symbol
+		(lib_name "74LS30_2")
 		(lib_id "74xx:74LS30")
 		(at 54.61 76.2 180)
@@
 		)
 		(property "Footprint" "Package_DIP:DIP-14_W7.62mm"
-			(at 54.61 76.2 0)
-			(effects
-				(font
+			(at 54.61 64.262 0)
+			(effects
+				(font

Commit message: Fixes RN pin numbers
Connections:
- net GDO0: now also RN3.7 (R1); no longer RN3.2 (R1)
- net GDO10: now also RN2.6 (R3); no longer RN2.4 (R3)
- net GDO11: now also RN2.8 (R4); no longer RN2.5 (R4)
- net GDO12: now also RN2.9 (R5); no longer RN2.6 (R5)
- net GDO13: now also RN2.5 (R6); no longer RN2.7 (R6)
- net GDO14: now also RN2.2 (R7); no longer RN2.8 (R7)
- net GDO15: now also RN2.3 (R8); no longer RN2.9 (R8)
- net GDO2: now also RN3.8 (R3); no longer RN3.4 (R3)
- net GDO5: now also RN3.9 (R6); no longer RN3.7 (R6)
- net GDO6: now also RN3.4 (R7); no longer RN3.8 (R7)
- net GDO7: now also RN3.2 (R8); no longer RN3.9 (R8)
- net GDO8: now also RN2.4 (R1); no longer RN2.2 (R1)
- net GDO9: now also RN2.7 (R2); no longer RN2.3 (R2)
Changed lines of the file:
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@@
 	)
 	(symbol
+		(lib_name "R_Network08_1")
 		(lib_id "Device:R_Network08")
 		(at 77.47 31.75 0)

Commit message: Fixes "CA0" issue in schematics
Changed lines of the file:
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@@
 (kicad_sch
-	(version 20231120)
+	(version 20250114)
 	(generator "eeschema")
-	(generator_version "8.0")
+	(generator_version "9.0")
 	(paper "A4")
 	(title_block

Commit message: Fixes unconnected pads
Changed lines of the file:
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@@
 		(dnp no)
 		(property "Reference" "IC68"
-			(at 55.626 185.42 0)
+			(at 48.006 186.436 0)
 			(effects
 				(font
@@
 		)
 		(property "Value" "74LS30"
-			(at 58.166 185.42 0)
+			(at 50.546 186.436 0)
 			(effects
 				(font
@@
 		(pin "3"
 		)
+		(pin "9"
+		)
+		(pin "10"
+		)
+		(pin "13"
+		)
 		(instances
 			(project "gdp"
@@
 		)
 		(pin "3"
+		)
+		(pin "9"
+		)
+		(pin "10"
+		)
+		(pin "13"
 		)
 		(instances
@@
 		(dnp no)
 		(property "Reference" "IC70"
-			(at 55.88 96.52 0)
+			(at 48.006 97.536 0)
 			(effects
 				(font
@@
 		)
 		(property "Value" "74LS30"
-			(at 58.42 96.52 0)
+			(at 50.546 97.536 0)
 			(effects
 				(font
@@
 		)
 		(pin "3"
+		)
+		(pin "13"
+		)
+		(pin "10"
+		)
+		(pin "9"
 		)
 		(instances
@@
 		(pin "3"
 		)
-		(instances
+		(pin "10"
+		)
+		(pin "13"
+		)
+		(pin "9"
+		)
+		(instances

Commit message: Fixes several mistakes (1 mistake in the schema!)
Connections:
- net OC renamed QC
Changed lines of the file:
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@@
 		)
 	)
-	(global_label "OC"
+	(global_label "QC"
 		(shape input)
 		(at 177.8 64.77 180)
