File: gdp/1.kicad_sch (KiCad schematic)
At the start: 23 parts, among them IC1 LM393, IC3 LM393, IC8 74LS245, J3 ST32, J4 ST32, U1 7406, U2 7406

Commit message: Adds pages 4, 7, 10 (still WIP)
Changed lines of the file:
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@@
-    )
-  )
-  (global_label "VDD" (shape input) (at 167.64 52.07 90) (fields_autoplaced)
-    (effects (font (size 1.27 1.27)) (justify left))
-    (property "Intersheetrefs" "${INTERSHEET_REFS}" (at 167.64 45.4562 90)
-      (effects (font (size 1.27 1.27)) (justify left))
     )
   )
@@
     )
   )
-  (global_label "VCC" (shape input) (at 167.64 36.195 90) (fields_autoplaced)
-    (effects (font (size 1.27 1.27)) (justify left))
-    (property "Intersheetrefs" "${INTERSHEET_REFS}" (at 167.64 29.5812 90)
-      (effects (font (size 1.27 1.27)) (justify left))
-    )
-  )
   (global_label "A7" (shape output) (at 40.64 165.735 0) (fields_autoplaced)
     (effects (font (size 1.27 1.27)) (justify left))
@@
     )
   )
-  (global_label "VDD" (shape input) (at 50.165 94.615 90) (fields_autoplaced)
-    (effects (font (size 1.27 1.27)) (justify left))
-    (property "Intersheetrefs" "${INTERSHEET_REFS}" (at 50.165 88.0012 90)
-      (effects (font (size 1.27 1.27)) (justify left))
-    )
-  )
   (global_label "~{INT}" (shape input) (at 69.85 142.875 180) (fields_autoplaced)
     (effects (font (size 1.27 1.27)) (justify right))
@@
     (effects (font (size 1.27 1.27)) (justify left))
     (property "Intersheetrefs" "${INTERSHEET_REFS}" (at 96.3605 146.685 0)
-      (effects (font (size 1.27 1.27)) (justify left))
-    )
-  )
-  (global_label "VCC" (shape input) (at 60.325 94.615 90) (fields_autoplaced)
-    (effects (font (size 1.27 1.27)) (justify left))
-    (property "Intersheetrefs" "${INTERSHEET_REFS}" (at 60.325 88.0012 90)
       (effects (font (size 1.27 1.27)) (justify left))
     )
@@
   )
   (symbol (lib_id "power:+5V") (at 165.1 139.7 0) (unit 1)
-    (in_bom yes) (on_board yes) (dnp no) (fields_autoplaced)
+    (in_bom yes) (on_board yes) (dnp no)
     (property "Reference" "#PWR015" (at 165.1 143.51 0)
       (effects (font (size 1.27 1.27)) hide)
     )
-    (property "Value" "+5V" (at 165.1 134.62 0)
+    (property "Value" "+5V" (at 165.1 135.255 0)
       (effects (font (size 1.27 1.27)))
     )
@@
       (effects (font (size 1.27 1.27)) hide)
     )
-    (property "Value" "+12V" (at 204.47 47.625 0)
+    (property "Value" "+12V" (at 204.47 48.26 0)
       (effects (font (size 1.27 1.27)))
     )
@@
         )
         (path "/95aff260-2720-4733-a81d-a7a2136fdd14/fb334c08-c103-46ff-b900-c3f57a56f58c"
-          (reference "CK1") (unit 1)
+          (reference "CK23") (unit 1)
         )
       )
@@
     )
   )
+  (symbol (lib_id "power:VDD") (at 50.165 94.615 0) (unit 1)
+    (in_bom yes) (on_board yes) (dnp no)
+    (property "Reference" "#PWR023" (at 50.165 98.425 0)
+      (effects (font (size 1.27 1.27)) hide)
+    )
+    (property "Value" "VDD" (at 50.165 90.17 0)
+      (effects (font (size 1.27 1.27)))
+    )
+    (property "Footprint" "" (at 50.165 94.615 0)
+      (effects (font (size 1.27 1.27)) hide)
+    )
+    (property "Datasheet" "" (at 50.165 94.615 0)
+      (effects (font (size 1.27 1.27)) hide)
+    )
+    (pin "1")
+    (instances
+      (project "gdp"
+        (path "/95aff260-2720-4733-a81d-a7a2136fdd14/fb334c08-c103-46ff-b900-c3f57a56f58c"
+          (reference "#PWR023") (unit 1)
+        )
+      )
+    )
+  )
   (symbol (lib_id "power:+5V") (at 213.36 52.705 0) (unit 1)
+    (in_bom yes) (on_board yes) (dnp no)
+    (property "Reference" "#PWR05" (at 213.36 56.515 0)
+      (effects (font (size 1.27 1.27)) hide)
+    )
+    (property "Value" "+5V" (at 213.36 48.26 0)
+      (effects (font (size 1.27 1.27)))
+    )
+    (property "Footprint" "" (at 213.36 52.705 0)
+      (effects (font (size 1.27 1.27)) hide)
+    )
+    (property "Datasheet" "" (at 213.36 52.705 0)
+      (effects (font (size 1.27 1.27)) hide)
+    )
+    (pin "1")
+    (instances
+      (project "gdp"
+        (path "/95aff260-2720-4733-a81d-a7a2136fdd14"
+          (reference "#PWR05") (unit 1)
+        )
+        (path "/95aff260-2720-4733-a81d-a7a2136fdd14/fb334c08-c103-46ff-b900-c3f57a56f58c"
+          (reference "#PWR020") (unit 1)
+        )
+      )
+    )
+  )
+  (symbol (lib_id "power:VCC") (at 167.64 36.195 0) (unit 1)
     (in_bom yes) (on_board yes) (dnp no) (fields_autoplaced)
-    (property "Reference" "#PWR05" (at 213.36 56.515 0)
-      (effects (font (size 1.27 1.27)) hide)
-    )
-    (property "Value" "+5V" (at 213.36 47.625 0)
-      (effects (font (size 1.27 1.27)))
-    )
-    (property "Footprint" "" (at 213.36 52.705 0)
-      (effects (font (size 1.27 1.27)) hide)
-    )
-    (property "Datasheet" "" (at 213.36 52.705 0)
-      (effects (font (size 1.27 1.27)) hide)
-    )
-    (pin "1")
-    (instances
-      (project "gdp"
-        (path "/95aff260-2720-4733-a81d-a7a2136fdd14"
-          (reference "#PWR05") (unit 1)
-        )
-        (path "/95aff260-2720-4733-a81d-a7a2136fdd14/fb334c08-c103-46ff-b900-c3f57a56f58c"
-          (reference "#PWR020") (unit 1)
+    (property "Reference" "#PWR016" (at 167.64 40.005 0)
+      (effects (font (size 1.27 1.27)) hide)
+    )
+    (property "Value" "VCC" (at 167.64 31.75 0)
+      (effects (font (size 1.27 1.27)))
+    )
+    (property "Footprint" "" (at 167.64 36.195 0)
+      (effects (font (size 1.27 1.27)) hide)
+    )
+    (property "Datasheet" "" (at 167.64 36.195 0)
+      (effects (font (size 1.27 1.27)) hide)
+    )
+    (pin "1")
+    (instances
+      (project "gdp"
+        (path "/95aff260-2720-4733-a81d-a7a2136fdd14/fb334c08-c103-46ff-b900-c3f57a56f58c"
+          (reference "#PWR016") (unit 1)
         )
       )
@@
     )
   )
+  (symbol (lib_id "power:VDD") (at 167.64 52.07 0) (unit 1)
+    (in_bom yes) (on_board yes) (dnp no)
+    (property "Reference" "#PWR017" (at 167.64 55.88 0)
+      (effects (font (size 1.27 1.27)) hide)
+    )
+    (property "Value" "VDD" (at 167.64 47.625 0)
+      (effects (font (size 1.27 1.27)))
+    )
+    (property "Footprint" "" (at 167.64 52.07 0)
+      (effects (font (size 1.27 1.27)) hide)
+    )
+    (property "Datasheet" "" (at 167.64 52.07 0)
+      (effects (font (size 1.27 1.27)) hide)
+    )
+    (pin "1")
+    (instances
+      (project "gdp"
+        (path "/95aff260-2720-4733-a81d-a7a2136fdd14/fb334c08-c103-46ff-b900-c3f57a56f58c"
+          (reference "#PWR017") (unit 1)
+        )
+      )
+    )
+  )
   (symbol (lib_id "power:GNDD") (at 224.79 52.705 180) (unit 1)
     (in_bom yes) (on_board yes) (dnp no) (fields_autoplaced)
@@
     )
   )
+  (symbol (lib_id "power:VCC") (at 60.325 94.615 0) (unit 1)
+    (in_bom yes) (on_board yes) (dnp no) (fields_autoplaced)
+    (property "Reference" "#PWR022" (at 60.325 98.425 0)
+      (effects (font (size 1.27 1.27)) hide)
+    )
+    (property "Value" "VCC" (at 60.325 90.17 0)
+      (effects (font (size 1.27 1.27)))
+    )
+    (property "Footprint" "" (at 60.325 94.615 0)
+      (effects (font (size 1.27 1.27)) hide)
+    )
+    (property "Datasheet" "" (at 60.325 94.615 0)
+      (effects (font (size 1.27 1.27)) hide)
+    )
+    (pin "1")
+    (instances
+      (project "gdp"
+        (path "/95aff260-2720-4733-a81d-a7a2136fdd14/fb334c08-c103-46ff-b900-c3f57a56f58c"
+          (reference "#PWR022") (unit 1)
+        )
+      )
+    )
+  )
   (symbol (lib_id "Switch:SW_DPST_x2") (at 247.65 32.385 0) (unit 1)
     (in_bom yes) (on_board yes) (dnp no)
@@
   )
   (symbol (lib_id "power:+5V") (at 101.6 20.32 0) (unit 1)
-    (in_bom yes) (on_board yes) (dnp no) (fields_autoplaced)
+    (in_bom yes) (on_board yes) (dnp no)
     (property "Reference" "#PWR05" (at 101.6 24.13 0)
       (effects (font (size 1.27 1.27)) hide)
     )
-    (property "Value" "+5V" (at 101.6 15.24 0)
+    (property "Value" "+5V" (at 101.6 15.875 0)
       (effects (font (size 1.27 1.27)))
     )
@@
   )
   (symbol (lib_id "power:+5V") (at 264.16 127 0) (unit 1)
-    (in_bom yes) (on_board yes) (dnp no) (fields_autoplaced)
+    (in_bom yes) (on_board yes) (dnp no)
     (property "Reference" "#PWR014" (at 264.16 130.81 0)
       (effects (font (size 1.27 1.27)) hide)
     )
-    (property "Value" "+5V" (at 264.16 121.92 0)
-      (effects (font (size 1.27 1.27)))
-    )
+    (property "Value" "+5V" (at 264.16 122.555 0)
+      (effects (font (size 1.27 1.27)))
+    )

Commit message: Some minor edits
Other:
- company: (none) -> Oddbit Retro
Changed lines of the file:
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@@
   (title_block
     (title "PARTNER GDP")
+    (company "Oddbit Retro")
   )
   (junction (at 213.36 112.395) (diameter 0) (color 0 0 0 0)

Commit message: Adds Sheet 3
Parts:
- gave numbers to parts that had none: 3
- renumbered IC8 to IC1, U2 to IC11, U1 to IC11, IC3 to IC2, IC1 to IC2, R13 to R1, R21 to R2, R11 to R3, R10 to R4, R9 to R5, R8 to R6, ST2 to ST1, ST1 to ST2, J4 to ST4, J3 to ST5

Commit message: Adds Sheet 5
Other:
- title: PARTNER GDP -> PARTNER GDP: BUS + KEYBOARD INTERFACE
Changed lines of the file:
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@@
 	(paper "A4")
 	(title_block
-		(title "PARTNER GDP")
+		(title "PARTNER GDP: BUS + KEYBOARD INTERFACE")
 		(company "Oddbit Retro")
+		(comment 1 "NARISAL: MIHA GRČAR")
 	)
 	(junction

Commit message: Adds Sheet 9
Parts:
- renumbered IC2 to IC3, IC1 to IC8, R4 to R10, R3 to R11, R11 to R12, R12 to R14, R13 to R15, R2 to R21, R6 to R8, R5 to R9, ST2 to ST1, ST1 to ST2
Other:
- moved on the sheet: CK23, IC11A, IC11B, IC11G, IC3A, IC3B, IC8, R1, R10, R11, R12, R14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

Commit message: Adds Sheet 12
Other:
- moved on the sheet: CK23, IC11A, IC11B, IC11G, IC3A, IC3B, IC8, R1, R10, R11, R12, R14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

Commit message: Small fixes
Parts:
- renumbered R1 to R13
Changed lines of the file:
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@@
 		(on_board yes)
 		(dnp no)
-		(property "Reference" "R1"
+		(property "Reference" "R13"
 			(at 162.56 118.745 0)
 			(effects
@@
 			(project "gdp"
 				(path "/95aff260-2720-4733-a81d-a7a2136fdd14/fb334c08-c103-46ff-b900-c3f57a56f58c"
-					(reference "R1")
+					(reference "R13")
 					(unit 1)
 				)

Commit message: Initial footprint assignment
Parts:
- CK1: renamed from CK23; footprint (none) -> Capacitor_THT:C_Disc_D4.3mm_W1.9mm_P5.00mm
- IC1: renamed from IC8; footprint (none) -> Package_DIP:DIP-20_W7.62mm
- IC2: renamed from IC3; footprint (none) -> Package_DIP:DIP-8_W7.62mm
- IC2: footprint (none) -> Package_DIP:DIP-8_W7.62mm
- IC3: renamed from IC11; footprint (none) -> Package_DIP:DIP-14_W7.62mm
- R1: renamed from R13; footprint (none) -> Resistor_THT:R_Axial_DIN0207_L6.3mm_D2.5mm_P7.62mm_Horizontal
- R2: renamed from R21; footprint (none) -> Resistor_THT:R_Axial_DIN0207_L6.3mm_D2.5mm_P7.62mm_Horizontal
- R3: renamed from R12; footprint (none) -> Resistor_THT:R_Axial_DIN0207_L6.3mm_D2.5mm_P7.62mm_Horizontal
- R4: renamed from R14; footprint (none) -> Resistor_THT:R_Axial_DIN0207_L6.3mm_D2.5mm_P7.62mm_Horizontal
- R5: renamed from R11; footprint (none) -> Resistor_THT:R_Axial_DIN0207_L6.3mm_D2.5mm_P7.62mm_Horizontal
- R6: renamed from R10; footprint (none) -> Resistor_THT:R_Axial_DIN0207_L6.3mm_D2.5mm_P7.62mm_Horizontal
- R7: renamed from R15; footprint (none) -> Resistor_THT:R_Axial_DIN0207_L6.3mm_D2.5mm_P7.62mm_Horizontal
- R8: renamed from R9; footprint (none) -> Resistor_THT:R_Axial_DIN0207_L6.3mm_D2.5mm_P7.62mm_Horizontal
- R9: renamed from R8; footprint (none) -> Resistor_THT:R_Axial_DIN0207_L6.3mm_D2.5mm_P7.62mm_Horizontal
- SH1: footprint (none) -> Connector_PinHeader_2.54mm:PinHeader_1x02_P2.54mm_Vertical
- SH2: renamed from SH3; footprint (none) -> Connector_PinHeader_2.54mm:PinHeader_1x02_P2.54mm_Vertical
- SH3: renamed from SH2; footprint (none) -> Connector_PinHeader_2.54mm:PinHeader_1x02_P2.54mm_Vertical
- ST1: renamed from ST5; value ST32 -> 32; footprint (none) -> Connector_PinHeader_2.54mm:PinHeader_1x32_P2.54mm_Vertical
- ST2: renamed from ST4; value ST32 -> 32; footprint (none) -> Connector_PinHeader_2.54mm:PinHeader_1x32_P2.54mm_Vertical
- ST3: renamed from ST2; value ST60F01 -> 6; footprint (none) -> Connector_PinHeader_2.54mm:PinHeader_1x06_P2.54mm_Vertical
- ST4: renamed from ST1; value 6PINCON -> 6; footprint (none) -> Connector_PinHeader_2.54mm:PinHeader_1x06_P2.54mm_Vertical
- ST5: renamed from ST3; value MODU2-10 -> 10; footprint (none) -> Connector_PinHeader_2.54mm:PinHeader_1x10_P2.54mm_Vertical
