File: gdp/2.kicad_sch (KiCad schematic)
At the start: 0 parts

Commit message: Adds page 2 (created by Tomaz)
Parts:
- added IC1: 74LS85, symbol replica:74LS85
- added IC17: MK3881, symbol replica:MK3881
- added IC7: PAL16L8, symbol replica:PAL16L8
- added R18, R19, R20: 2K2, symbol Device:R
- added SH7, SH8, SH9: SCHALT1, symbol Switch:SW_DPST_x2
Connections:
- new net: IC1.13 (A2), R18.2, SH8.1 (A)
- new net: IC1.15 (A3), R20.2, SH9.1 (A)
- new net: IC1.6 (A=B), IC7.1 (A)
- new net: IC17.4 (~{CE}), IC7.14 (BC)
- new net: IC17.37 (~{M1}), IC7.17 (BF)
- new net: IC1.12 (A1), R19.2, SH7.1 (A)
- new net +5V: IC1.3 (i(A=B)), SH7.2 (B), SH8.2 (B), SH9.2 (B)
- new net A0: IC17.5 (DS)
- new net A1: IC17.6 (BAS)
- new net A2: IC7.3 (C)
- new net A3: IC7.4 (D)
- new net A4: IC7.5 (E)
- new net A5: IC1.11 (B1)
- new net A6: IC1.14 (B2)
- new net A7: IC1.1 (B3)
- new net CA1: IC17.28 (B1)
- new net CA2: IC17.29 (B2)
- new net CA3: IC17.30 (B3)
- new net CA4: IC17.31 (B4)
- new net CA5: IC17.32 (B5)
- new net CA6: IC17.33 (B6)
- new net CA7: IC17.34 (B7)
- new net D0: IC17.19 (D0)
- new net D1: IC17.20 (D1)
- new net D2: IC17.1 (D2)
- new net D3: IC17.40 (D3)
- new net D4: IC17.39 (D4)
- new net D5: IC17.38 (D5)
- new net D6: IC17.3 (D6)
- new net D7: IC17.2 (D7)
- new net FM0: IC17.12 (A3)
- new net FM1: IC17.10 (A4)
- new net GND: IC1.10 (A0), IC1.2 (i(A<B)), IC1.4 (i(A>B)), IC1.9 (B0), R18.1, R19.1, R20.1
- new net IEI: IC17.24 (INI)
- new net PHI: IC17.25 (PHI)
- new net RBNK: IC17.15 (A0)
- new net SCRLM: IC17.7 (A7)
- new net WBNK: IC17.14 (A1)
- new net XORM: IC17.13 (A2)
- new net ~{AVDC}: IC7.16 (BE)
- new net ~{AVDINT}: IC17.17 (~{BSTB})
- new net ~{AVINT}: IC17.8 (A6)
- new net ~{BUFFER}: IC7.15 (BD)
- new net ~{DIN}: IC7.18 (BG)
- new net ~{GDPINT}: IC17.16 (~{ASTB})
- new net ~{GDP}: IC7.12 (ZA)
- new net ~{GINT}: IC17.9 (A5)
- new net ~{INT}: IC17.23 (~{INT}), IC7.8 (H)
- new net ~{IORQ}: IC17.36 (~{IORQ}), IC7.9 (I)
- new net ~{MI}: IC7.7 (G)
- new net ~{RD}: IC17.35 (~{RD}), IC7.6 (F)
- new net ~{RES}: IC7.2 (B)
- new net ~{TSC}: IC7.13 (BB)
- no-connect marks 0 -> 8
Other:
- note added: "CA0"
- note added: "IE0"
- company: (none) -> Oddbit Retro
- title: Partner GDP -> PARTNER GDP

Commit message: Adds Sheet 3
Connections:
- net +5V: now also IC1.16 (VCC), IC17.26 (VCC), IC7.20 (VCC)
- net GND: now also IC1.8 (GND), IC17.11 (GND), IC7.10 (GND)
Other:
- moved on the sheet: IC1, R18, R19, R20, SH7A, SH8A, SH9A

Commit message: Adds Sheet 5
Other:
- title: PARTNER GDP -> PARTNER GDP: ADRESIRANJE + PIO
- moved on the sheet: IC1, IC17, IC7, R18, R19, R20, SH7A, SH8A, SH9A

Commit message: Adds Sheet 12
Changed lines of the file:
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@@
 	)
 	(symbol
+		(lib_name "SW_DPST_x2_2")
 		(lib_id "Switch:SW_DPST_x2")
 		(at 81.28 113.03 90)
@@
 		)
 		(pin "2"
-		)
-		(pin "3"
-		)
-		(pin "4"
 		)
 		(instances
@@
 	)
 	(symbol
+		(lib_name "SW_DPST_x2_1")
 		(lib_id "Switch:SW_DPST_x2")
 		(at 78.74 113.03 90)
@@
 		)
 		(pin "2"
-		)
-		(pin "3"
-		)
-		(pin "4"
 		)
 		(instances
@@
 		(pin "2"
 		)
-		(pin "3"
-		)
-		(pin "4"
-		)
-		(instances
+		(instances

Commit message: Adds Sheet 14 (WIP)
Connections:
- net ~{MI} renamed ~{M1}
Changed lines of the file:
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@@
 		)
 	)
-	(global_label "~{MI}"
+	(global_label "~{M1}"
 		(shape input)
 		(at 115.57 67.31 180)
@@
 		)
 		(property "Intersheetrefs" "${INTERSHEET_REFS}"
-			(at 110.5286 67.31 0)
+			(at 109.9239 67.31 0)
 			(effects
 				(font

Commit message: Initial footprint assignment
Parts:
- IC1: footprint (none) -> Package_DIP:DIP-16_W7.62mm
- IC17: footprint (none) -> Package_DIP:DIP-40_W15.24mm
- IC7: footprint (none) -> Package_DIP:DIP-20_W7.62mm
- R18, R19, R20: footprint (none) -> Resistor_THT:R_Axial_DIN0207_L6.3mm_D2.5mm_P7.62mm_Horizontal
- SH7, SH8, SH9: value SCHALT1 -> SCHALT; footprint (none) -> Connector_PinHeader_2.54mm:PinHeader_1x02_P2.54mm_Vertical
Changed lines of the file:
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@@
 			)
 		)
-		(property "Footprint" ""
+		(property "Footprint" "Resistor_THT:R_Axial_DIN0207_L6.3mm_D2.5mm_P7.62mm_Horizontal"
 			(at 71.12 136.398 90)
 			(effects
@@
 			)
 		)
-		(property "Datasheet" "~"
+		(property "Datasheet" "N/A"
 			(at 71.12 134.62 0)
 			(effects
@@
 			)
 		)
-		(property "Description" ""
+		(property "Description" "N/A"
 			(at 71.12 134.62 0)
 			(effects
@@
 			(project "gdp"
 				(path "/95aff260-2720-4733-a81d-a7a2136fdd14/ed2e3011-1fbf-423e-aa8b-2b4bbe99b1f1"
-					(reference "R18")
+					(reference "R11")
 					(unit 1)
 				)
@@
 		(dnp no)
 		(fields_autoplaced yes)
-		(property "Reference" "#PWR065"
+		(property "Reference" "#PWR032"
 			(at 187.96 144.78 0)
 			(effects
@@
 			(project "gdp"
 				(path "/95aff260-2720-4733-a81d-a7a2136fdd14/ed2e3011-1fbf-423e-aa8b-2b4bbe99b1f1"
-					(reference "#PWR065")
+					(reference "#PWR032")
 					(unit 1)
 				)
@@
 		(dnp no)
 		(fields_autoplaced yes)
-		(property "Reference" "#PWR082"
+		(property "Reference" "#PWR027"
 			(at 114.3 115.57 0)
 			(effects
@@
 			(project "gdp"
 				(path "/95aff260-2720-4733-a81d-a7a2136fdd14/ed2e3011-1fbf-423e-aa8b-2b4bbe99b1f1"
-					(reference "#PWR082")
+					(reference "#PWR027")
 					(unit 1)
 				)
@@
 		(dnp no)
 		(fields_autoplaced yes)
-		(property "Reference" "#PWR064"
+		(property "Reference" "#PWR028"
 			(at 114.3 157.48 0)
 			(effects
@@
 			(project "gdp"
 				(path "/95aff260-2720-4733-a81d-a7a2136fdd14/ed2e3011-1fbf-423e-aa8b-2b4bbe99b1f1"
-					(reference "#PWR064")
+					(reference "#PWR028")
 					(unit 1)
 				)
@@
 			)
 		)
-		(property "Footprint" ""
+		(property "Footprint" "Resistor_THT:R_Axial_DIN0207_L6.3mm_D2.5mm_P7.62mm_Horizontal"
 			(at 71.12 138.938 90)
 			(effects
@@
 			)
 		)
-		(property "Datasheet" "~"
+		(property "Datasheet" "N/A"
 			(at 71.12 137.16 0)
 			(effects
@@
 			)
 		)
-		(property "Description" ""
+		(property "Description" "N/A"
 			(at 71.12 137.16 0)
 			(effects
@@
 			(project "gdp"
 				(path "/95aff260-2720-4733-a81d-a7a2136fdd14/ed2e3011-1fbf-423e-aa8b-2b4bbe99b1f1"
-					(reference "R20")
+					(reference "R12")
 					(unit 1)
 				)
@@
 			)
 		)
-		(property "Footprint" ""
+		(property "Footprint" "Package_DIP:DIP-20_W7.62mm"
 			(at 137.16 41.91 0)
 			(effects
@@
 			)
 		)
-		(property "Datasheet" ""
+		(property "Datasheet" "N/A"
 			(at 137.16 41.91 0)
 			(effects
@@
 			)
 		)
-		(property "Description" ""
+		(property "Description" "N/A"
 			(at 138.43 45.72 0)
 			(effects
@@
 			(project "gdp"
 				(path "/95aff260-2720-4733-a81d-a7a2136fdd14/ed2e3011-1fbf-423e-aa8b-2b4bbe99b1f1"
-					(reference "IC7")
+					(reference "IC5")
 					(unit 1)
 				)
@@
 		(dnp no)
 		(fields_autoplaced yes)
-		(property "Reference" "#PWR074"
+		(property "Reference" "#PWR029"
 			(at 138.43 50.8 0)
 			(effects
@@
 			(project ""
 				(path "/95aff260-2720-4733-a81d-a7a2136fdd14/ed2e3011-1fbf-423e-aa8b-2b4bbe99b1f1"
-					(reference "#PWR074")
+					(reference "#PWR029")
 					(unit 1)
 				)
@@
 			(project "gdp"
 				(path "/95aff260-2720-4733-a81d-a7a2136fdd14/ed2e3011-1fbf-423e-aa8b-2b4bbe99b1f1"
-					(reference "#PWR01")
+					(reference "#PWR025")
 					(unit 1)
 				)
@@
 		(dnp no)
 		(fields_autoplaced yes)
-		(property "Reference" "#PWR063"
+		(property "Reference" "#PWR024"
 			(at 67.31 147.32 0)
 			(effects
@@
 			(project ""
 				(path "/95aff260-2720-4733-a81d-a7a2136fdd14/ed2e3011-1fbf-423e-aa8b-2b4bbe99b1f1"
-					(reference "#PWR063")
+					(reference "#PWR024")
 					(unit 1)
 				)
@@
 		(dnp no)
 		(fields_autoplaced yes)
-		(property "Reference" "#PWR066"
+		(property "Reference" "#PWR030"
 			(at 138.43 86.36 0)
 			(effects
@@
 			(project "gdp"
 				(path "/95aff260-2720-4733-a81d-a7a2136fdd14/ed2e3011-1fbf-423e-aa8b-2b4bbe99b1f1"
-					(reference "#PWR066")
+					(reference "#PWR030")
 					(unit 1)
 				)
@@
 			)
 		)
-		(property "Value" "SCHALT1"
+		(property "Value" "SCHALT"
 			(at 80.01 109.22 0)
 			(effects
@@
 			)
 		)
-		(property "Footprint" ""
+		(property "Footprint" "Connector_PinHeader_2.54mm:PinHeader_1x02_P2.54mm_Vertical"
 			(at 81.28 113.03 0)
 			(effects
@@
 			)
 		)
-		(property "Datasheet" "~"
+		(property "Datasheet" "N/A"
 			(at 81.28 113.03 0)
 			(effects
@@
 			)
 		)
-		(property "Description" ""
+		(property "Description" "N/A"
 			(at 81.28 113.03 0)
 			(effects
@@
 			(project "gdp"
 				(path "/95aff260-2720-4733-a81d-a7a2136fdd14/ed2e3011-1fbf-423e-aa8b-2b4bbe99b1f1"
-					(reference "SH8")
+					(reference "SH5")
 					(unit 1)
 				)
@@
 		(dnp no)
 		(fields_autoplaced yes)
-		(property "Reference" "#PWR075"
+		(property "Reference" "#PWR031"
 			(at 187.96 83.82 0)
 			(effects
@@
 			(project ""
 				(path "/95aff260-2720-4733-a81d-a7a2136fdd14/ed2e3011-1fbf-423e-aa8b-2b4bbe99b1f1"
-					(reference "#PWR075")
+					(reference "#PWR031")
 					(unit 1)
 				)
@@
 			)
 		)
-		(property "Value" "SCHALT1"
+		(property "Value" "SCHALT"
 			(at 77.47 109.22 0)
 			(effects
@@
 			)
 		)
-		(property "Footprint" ""
+		(property "Footprint" "Connector_PinHeader_2.54mm:PinHeader_1x02_P2.54mm_Vertical"
 			(at 78.74 113.03 0)
 			(effects
@@
 			)
 		)
-		(property "Datasheet" "~"
+		(property "Datasheet" "N/A"
 			(at 78.74 113.03 0)
 			(effects
@@
 			)
 		)
-		(property "Description" ""
+		(property "Description" "N/A"
 			(at 78.74 113.03 0)
 			(effects
@@
 			(project "gdp"
 				(path "/95aff260-2720-4733-a81d-a7a2136fdd14/ed2e3011-1fbf-423e-aa8b-2b4bbe99b1f1"
-					(reference "SH7")
+					(reference "SH4")
 					(unit 1)
 				)
@@
 			)
 		)
-		(property "Value" "SCHALT1"
+		(property "Value" "SCHALT"
 			(at 82.55 109.22 0)
 			(effects
@@
 			)
 		)
-		(property "Footprint" ""
+		(property "Footprint" "Connector_PinHeader_2.54mm:PinHeader_1x02_P2.54mm_Vertical"
 			(at 83.82 113.03 0)
 			(effects
@@
 			)
 		)
-		(property "Datasheet" "~"
+		(property "Datasheet" "N/A"
 			(at 83.82 113.03 0)
 			(effects
@@
 			)
 		)
-		(property "Description" ""
+		(property "Description" "N/A"
 			(at 83.82 113.03 0)
 			(effects
@@
 			(project "gdp"
 				(path "/95aff260-2720-4733-a81d-a7a2136fdd14/ed2e3011-1fbf-423e-aa8b-2b4bbe99b1f1"
-					(reference "SH9")
+					(reference "SH6")
 					(unit 1)
 				)
@@
 		(dnp no)
 		(fields_autoplaced yes)
-		(property "Reference" "#PWR081"
+		(property "Reference" "#PWR026"
 			(at 97.79 125.73 0)
 			(effects
@@
 			(project "gdp"
 				(path "/95aff260-2720-4733-a81d-a7a2136fdd14/ed2e3011-1fbf-423e-aa8b-2b4bbe99b1f1"
-					(reference "#PWR081")
+					(reference "#PWR026")
 					(unit 1)
 				)
@@
 			)
 		)
-		(property "Footprint" ""
+		(property "Footprint" "Package_DIP:DIP-40_W15.24mm"
 			(at 186.69 77.47 0)
 			(effects
@@
 			)
 		)
-		(property "Datasheet" ""
+		(property "Datasheet" "N/A"
 			(at 186.69 77.47 0)
 			(effects
@@
 			)
 		)
-		(property "Description" ""
+		(property "Description" "N/A"
 			(at 182.88 77.47 0)
 			(effects
@@
 			(project "gdp"
 				(path "/95aff260-2720-4733-a81d-a7a2136fdd14/ed2e3011-1fbf-423e-aa8b-2b4bbe99b1f1"
-					(reference "IC17")
+					(reference "IC6")
 					(unit 1)
 				)
@@
 			)
 		)
-		(property "Footprint" ""
+		(property "Footprint" "Package_DIP:DIP-16_W7.62mm"
 			(at 116.84 109.22 0)
 			(effects
@@
 			)
 		)
-		(property "Datasheet" ""
+		(property "Datasheet" "N/A"
 			(at 116.84 109.22 0)
 			(effects
@@
 			)
 		)
-		(property "Description" ""
+		(property "Description" "N/A"
 			(at 110.49 118.11 0)
 			(effects
@@
 			(project "gdp"
 				(path "/95aff260-2720-4733-a81d-a7a2136fdd14/ed2e3011-1fbf-423e-aa8b-2b4bbe99b1f1"
-					(reference "IC6")
+					(reference "IC4")
 					(unit 1)
 				)
@@
 			)
 		)
-		(property "Footprint" ""
+		(property "Footprint" "Resistor_THT:R_Axial_DIN0207_L6.3mm_D2.5mm_P7.62mm_Horizontal"
 			(at 71.12 133.858 90)
 			(effects
@@
 			)
 		)
-		(property "Datasheet" "~"
+		(property "Datasheet" "N/A"
 			(at 71.12 132.08 0)
 			(effects
@@
 			)
 		)
-		(property "Description" ""
+		(property "Description" "N/A"
 			(at 71.12 132.08 0)
 			(effects
@@
 			(project "gdp"
 				(path "/95aff260-2720-4733-a81d-a7a2136fdd14/ed2e3011-1fbf-423e-aa8b-2b4bbe99b1f1"
-					(reference "R19")
-					(unit 1)
-				)
+					(reference "R10")
+					(unit 1)
+				)
