File: gdp/2.kicad_sch (KiCad schematic)
At the start: 9 parts, among them IC1 74LS85, IC17 MK3881, IC7 PAL16L8

Commit message: Fixes refs
Parts:
- renumbered IC7 to IC23, IC17 to IC60, IC1 to IC8, R18 to R49, R19 to R53, R20 to R6, SH8 to SH10, SH7 to SH11, SH9 to SH4
Changed lines of the file:
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@@
 		(on_board yes)
 		(dnp no)
-		(property "Reference" "R18"
+		(property "Reference" "R49"
 			(at 71.12 134.62 90)
 			(effects
@@
 			(project "replica"
 				(path "/1aaa08cd-2585-4601-8223-7ea6b691e31d"
-					(reference  "R49")
-					(unit 1)
-				)
-			)
-			(project "gdp"
-				(path "/95aff260-2720-4733-a81d-a7a2136fdd14/ed2e3011-1fbf-423e-aa8b-2b4bbe99b1f1"
-					(reference  "R18")
+					(reference "R49")
+					(unit 1)
+				)
+			)
+			(project "gdp"
+				(path "/95aff260-2720-4733-a81d-a7a2136fdd14/ed2e3011-1fbf-423e-aa8b-2b4bbe99b1f1"
+					(reference "R18")
 					(unit 1)
 				)
@@
 		(on_board yes)
 		(dnp no)
-		(property "Reference" "R20"
+		(property "Reference" "R6"
 			(at 71.12 137.16 90)
 			(effects
@@
 			(project "replica"
 				(path "/1aaa08cd-2585-4601-8223-7ea6b691e31d"
-					(reference  "R6")
-					(unit 1)
-				)
-			)
-			(project "gdp"
-				(path "/95aff260-2720-4733-a81d-a7a2136fdd14/ed2e3011-1fbf-423e-aa8b-2b4bbe99b1f1"
-					(reference  "R20")
+					(reference "R6")
+					(unit 1)
+				)
+			)
+			(project "gdp"
+				(path "/95aff260-2720-4733-a81d-a7a2136fdd14/ed2e3011-1fbf-423e-aa8b-2b4bbe99b1f1"
+					(reference "R20")
 					(unit 1)
 				)
@@
 		(dnp no)
 		(fields_autoplaced yes)
-		(property "Reference" "IC7"
+		(property "Reference" "IC23"
 			(at 139.7 44.45 0)
 			(do_not_autoplace yes)
@@
 			(project "replica"
 				(path "/1aaa08cd-2585-4601-8223-7ea6b691e31d"
-					(reference  "IC23")
-					(unit 1)
-				)
-			)
-			(project "gdp"
-				(path "/95aff260-2720-4733-a81d-a7a2136fdd14/ed2e3011-1fbf-423e-aa8b-2b4bbe99b1f1"
-					(reference  "IC7")
+					(reference "IC23")
+					(unit 1)
+				)
+			)
+			(project "gdp"
+				(path "/95aff260-2720-4733-a81d-a7a2136fdd14/ed2e3011-1fbf-423e-aa8b-2b4bbe99b1f1"
+					(reference "IC7")
 					(unit 1)
 				)
@@
 		(on_board yes)
 		(dnp no)
-		(property "Reference" "SH8"
+		(property "Reference" "SH10"
 			(at 80.01 119.38 0)
 			(effects
@@
 			(project "replica"
 				(path "/1aaa08cd-2585-4601-8223-7ea6b691e31d"
-					(reference  "SH10")
-					(unit 1)
-				)
-			)
-			(project "gdp"
-				(path "/95aff260-2720-4733-a81d-a7a2136fdd14/ed2e3011-1fbf-423e-aa8b-2b4bbe99b1f1"
-					(reference  "SH8")
+					(reference "SH10")
+					(unit 1)
+				)
+			)
+			(project "gdp"
+				(path "/95aff260-2720-4733-a81d-a7a2136fdd14/ed2e3011-1fbf-423e-aa8b-2b4bbe99b1f1"
+					(reference "SH8")
 					(unit 1)
 				)
@@
 		(on_board yes)
 		(dnp no)
-		(property "Reference" "SH7"
+		(property "Reference" "SH11"
 			(at 77.47 119.38 0)
 			(effects
@@
 			(project "replica"
 				(path "/1aaa08cd-2585-4601-8223-7ea6b691e31d"
-					(reference  "SH11")
-					(unit 1)
-				)
-			)
-			(project "gdp"
-				(path "/95aff260-2720-4733-a81d-a7a2136fdd14/ed2e3011-1fbf-423e-aa8b-2b4bbe99b1f1"
-					(reference  "SH7")
+					(reference "SH11")
+					(unit 1)
+				)
+			)
+			(project "gdp"
+				(path "/95aff260-2720-4733-a81d-a7a2136fdd14/ed2e3011-1fbf-423e-aa8b-2b4bbe99b1f1"
+					(reference "SH7")
 					(unit 1)
 				)
@@
 		(on_board yes)
 		(dnp no)
-		(property "Reference" "SH9"
+		(property "Reference" "SH4"
 			(at 82.55 119.38 0)
 			(effects
@@
 			(project "replica"
 				(path "/1aaa08cd-2585-4601-8223-7ea6b691e31d"
-					(reference  "SH4")
-					(unit 1)
-				)
-			)
-			(project "gdp"
-				(path "/95aff260-2720-4733-a81d-a7a2136fdd14/ed2e3011-1fbf-423e-aa8b-2b4bbe99b1f1"
-					(reference  "SH9")
+					(reference "SH4")
+					(unit 1)
+				)
+			)
+			(project "gdp"
+				(path "/95aff260-2720-4733-a81d-a7a2136fdd14/ed2e3011-1fbf-423e-aa8b-2b4bbe99b1f1"
+					(reference "SH9")
 					(unit 1)
 				)
@@
 		(dnp no)
 		(fields_autoplaced yes)
-		(property "Reference" "IC17"
+		(property "Reference" "IC60"
 			(at 190.1541 77.47 0)
 			(effects
@@
 			(project "replica"
 				(path "/1aaa08cd-2585-4601-8223-7ea6b691e31d"
-					(reference  "IC60")
-					(unit 1)
-				)
-			)
-			(project "gdp"
-				(path "/95aff260-2720-4733-a81d-a7a2136fdd14/ed2e3011-1fbf-423e-aa8b-2b4bbe99b1f1"
-					(reference  "IC17")
+					(reference "IC60")
+					(unit 1)
+				)
+			)
+			(project "gdp"
+				(path "/95aff260-2720-4733-a81d-a7a2136fdd14/ed2e3011-1fbf-423e-aa8b-2b4bbe99b1f1"
+					(reference "IC17")
 					(unit 1)
 				)
@@
 		(dnp no)
 		(fields_autoplaced yes)
-		(property "Reference" "IC1"
+		(property "Reference" "IC8"
 			(at 116.4941 109.22 0)
 			(effects
@@
 			(project "replica"
 				(path "/1aaa08cd-2585-4601-8223-7ea6b691e31d"
-					(reference  "IC8")
-					(unit 1)
-				)
-			)
-			(project "gdp"
-				(path "/95aff260-2720-4733-a81d-a7a2136fdd14/ed2e3011-1fbf-423e-aa8b-2b4bbe99b1f1"
-					(reference  "IC6")
+					(reference "IC8")
+					(unit 1)
+				)
+			)
+			(project "gdp"
+				(path "/95aff260-2720-4733-a81d-a7a2136fdd14/ed2e3011-1fbf-423e-aa8b-2b4bbe99b1f1"
+					(reference "IC6")
 					(unit 1)
 				)
@@
 		(on_board yes)
 		(dnp no)
-		(property "Reference" "R19"
+		(property "Reference" "R53"
 			(at 71.12 132.08 90)
 			(effects
@@
 			(project "replica"
 				(path "/1aaa08cd-2585-4601-8223-7ea6b691e31d"
-					(reference  "R53")
-					(unit 1)
-				)
-			)
-			(project "gdp"
-				(path "/95aff260-2720-4733-a81d-a7a2136fdd14/ed2e3011-1fbf-423e-aa8b-2b4bbe99b1f1"
-					(reference  "R19")
-					(unit 1)
-				)
+					(reference "R53")
+					(unit 1)
+				)
+			)
+			(project "gdp"
+				(path "/95aff260-2720-4733-a81d-a7a2136fdd14/ed2e3011-1fbf-423e-aa8b-2b4bbe99b1f1"
+					(reference "R19")
+					(unit 1)
+				)

Commit message: Placing footprints...
Parts:
- R49, R53, R6: footprint Resistor_THT:R_Axial_DIN0207_L6.3mm_D2.5mm_P7.62mm_Horizontal -> Resistor_THT:R_Axial_DIN0207_L6.3mm_D2.5mm_P10.16mm_Horizontal
Changed lines of the file:
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@@
 			)
 		)
-		(property "Footprint" "Resistor_THT:R_Axial_DIN0207_L6.3mm_D2.5mm_P7.62mm_Horizontal"
+		(property "Footprint" "Resistor_THT:R_Axial_DIN0207_L6.3mm_D2.5mm_P10.16mm_Horizontal"
 			(at 71.12 136.398 90)
 			(effects
@@
 			)
 		)
-		(property "Footprint" "Resistor_THT:R_Axial_DIN0207_L6.3mm_D2.5mm_P7.62mm_Horizontal"
+		(property "Footprint" "Resistor_THT:R_Axial_DIN0207_L6.3mm_D2.5mm_P10.16mm_Horizontal"
 			(at 71.12 138.938 90)
 			(effects
@@
 			)
 		)
-		(property "Footprint" "Resistor_THT:R_Axial_DIN0207_L6.3mm_D2.5mm_P7.62mm_Horizontal"
+		(property "Footprint" "Resistor_THT:R_Axial_DIN0207_L6.3mm_D2.5mm_P10.16mm_Horizontal"
 			(at 71.12 133.858 90)
 			(effects

Commit message: Maps footprints PCB -> sch
Parts:
- IC23: footprint Package_DIP:DIP-20_W7.62mm -> Package_DIP:DIP-40_W15.24mm
- IC8: footprint Package_DIP:DIP-16_W7.62mm -> Package_DIP:DIP-20_W7.62mm
- R53: footprint Resistor_THT:R_Axial_DIN0207_L6.3mm_D2.5mm_P10.16mm_Horizontal -> GDP:R_XL
Changed lines of the file:
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@@
 			)
 		)
-		(property "Footprint" "Package_DIP:DIP-20_W7.62mm"
+		(property "Footprint" "Package_DIP:DIP-40_W15.24mm"
 			(at 137.16 41.91 0)
 			(effects
@@
 			)
 		)
-		(property "Footprint" "Package_DIP:DIP-16_W7.62mm"
+		(property "Footprint" "Package_DIP:DIP-20_W7.62mm"
 			(at 116.84 109.22 0)
 			(effects
@@
 			)
 		)
-		(property "Footprint" "Resistor_THT:R_Axial_DIN0207_L6.3mm_D2.5mm_P10.16mm_Horizontal"
+		(property "Footprint" "GDP:R_XL"
 			(at 71.12 133.858 90)
 			(effects

Commit message: Fixes footprint references in sch
Parts:
- IC60: footprint Package_DIP:DIP-40_W15.24mm -> Package_DIP:DIP-16_W7.62mm
- R49: footprint Resistor_THT:R_Axial_DIN0207_L6.3mm_D2.5mm_P10.16mm_Horizontal -> GDP:R_XL
Changed lines of the file:
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@@
 			)
 		)
-		(property "Footprint" "Resistor_THT:R_Axial_DIN0207_L6.3mm_D2.5mm_P10.16mm_Horizontal"
+		(property "Footprint" "GDP:R_XL"
 			(at 71.12 136.398 90)
 			(effects
@@
 			)
 		)
-		(property "Footprint" "Package_DIP:DIP-40_W15.24mm"
+		(property "Footprint" "Package_DIP:DIP-16_W7.62mm"
 			(at 186.69 77.47 0)
 			(effects

Commit message: Fixes Sheet 2 symbols
Parts:
- removed R49, R53: 2K2, GDP:R_XL, symbol Device:R
- removed R6: 2K2, Resistor_THT:R_Axial_DIN0207_L6.3mm_D2.5mm_P10.16mm_Horizontal, symbol Device:R
- added R18, R19, R20: 2K2, GDP:R_XL, symbol Device:R
- IC23: symbol replica:PAL16L8 -> GDP:PAL16L8
- IC60: symbol replica:MK3881 -> GDP:MK3881
- IC8: symbol replica:74LS85 -> GDP:74LS85
Connections:
- net GND: now also R18.1, R19.1, R20.1
- net at IC8.13 (A2), SH10.1 (A): now also R18.2
- net at IC8.15 (A3), SH4.1 (A): now also R20.2
- net at IC8.12 (A1), SH11.1 (A): now also R19.2

Commit message: Final fixes
Parts:
- IC17: renamed from IC60; footprint Package_DIP:DIP-16_W7.62mm -> Package_DIP:DIP-40_W15.24mm
- IC6: renamed from IC8; footprint Package_DIP:DIP-20_W7.62mm -> Package_DIP:DIP-16_W7.62mm
- IC7: renamed from IC23; footprint Package_DIP:DIP-40_W15.24mm -> Package_DIP:DIP-20_W7.62mm
- renumbered SH11 to SH7, SH10 to SH8, SH4 to SH9
Changed lines of the file:
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@@
 		(dnp no)
 		(fields_autoplaced yes)
-		(property "Reference" "#PWR032"
+		(property "Reference" "#PWR0204"
 			(at 187.96 144.78 0)
 			(effects
@@
 			(project "gdp"
 				(path "/95aff260-2720-4733-a81d-a7a2136fdd14/ed2e3011-1fbf-423e-aa8b-2b4bbe99b1f1"
-					(reference "#PWR032")
+					(reference "#PWR0204")
 					(unit 1)
 				)
@@
 		(dnp no)
 		(fields_autoplaced yes)
-		(property "Reference" "#PWR027"
+		(property "Reference" "#PWR0201"
 			(at 114.3 115.57 0)
 			(effects
@@
 			(project "gdp"
 				(path "/95aff260-2720-4733-a81d-a7a2136fdd14/ed2e3011-1fbf-423e-aa8b-2b4bbe99b1f1"
-					(reference "#PWR027")
+					(reference "#PWR0201")
 					(unit 1)
 				)
@@
 		(dnp no)
 		(fields_autoplaced yes)
-		(property "Reference" "#PWR028"
+		(property "Reference" "#PWR0199"
 			(at 114.3 157.48 0)
 			(effects
@@
 			(project "gdp"
 				(path "/95aff260-2720-4733-a81d-a7a2136fdd14/ed2e3011-1fbf-423e-aa8b-2b4bbe99b1f1"
-					(reference "#PWR028")
+					(reference "#PWR0199")
 					(unit 1)
 				)
@@
 		(on_board yes)
 		(dnp no)
-		(fields_autoplaced yes)
-		(property "Reference" "IC23"
-			(at 140.6241 41.91 0)
+		(property "Reference" "IC7"
+			(at 140.716 44.45 0)
 			(effects
 				(font
@@
 		)
 		(property "Value" "PAL16L8"
-			(at 140.6241 44.45 0)
+			(at 140.716 46.99 0)
 			(effects
 				(font
@@
 			)
 		)
-		(property "Footprint" "Package_DIP:DIP-40_W15.24mm"
+		(property "Footprint" "Package_DIP:DIP-20_W7.62mm"
 			(at 137.16 41.91 0)
 			(effects
@@
 		)
 		(instances
-			(project "replica"
-				(path "/1aaa08cd-2585-4601-8223-7ea6b691e31d"
-					(reference "IC23")
-					(unit 1)
-				)
-			)
 			(project "gdp"
 				(path "/95aff260-2720-4733-a81d-a7a2136fdd14/ed2e3011-1fbf-423e-aa8b-2b4bbe99b1f1"
@@
 		(dnp no)
 		(fields_autoplaced yes)
-		(property "Reference" "#PWR029"
+		(property "Reference" "#PWR0207"
 			(at 138.43 50.8 0)
 			(effects
@@
 		)
 		(instances
-			(project ""
-				(path "/95aff260-2720-4733-a81d-a7a2136fdd14/ed2e3011-1fbf-423e-aa8b-2b4bbe99b1f1"
-					(reference "#PWR029")
+			(project "gdp"
+				(path "/95aff260-2720-4733-a81d-a7a2136fdd14/ed2e3011-1fbf-423e-aa8b-2b4bbe99b1f1"
+					(reference "#PWR0207")
 					(unit 1)
 				)
@@
 		(dnp no)
 		(fields_autoplaced yes)
-		(property "Reference" "#PWR01"
+		(property "Reference" "#PWR0205"
 			(at 97.79 106.68 0)
 			(effects
@@
 		)
 		(instances
-			(project "replica"
-				(path "/1aaa08cd-2585-4601-8223-7ea6b691e31d"
-					(reference "#PWR01")
-					(unit 1)
-				)
-			)
-			(project "gdp"
-				(path "/95aff260-2720-4733-a81d-a7a2136fdd14/ed2e3011-1fbf-423e-aa8b-2b4bbe99b1f1"
-					(reference "#PWR025")
+			(project "gdp"
+				(path "/95aff260-2720-4733-a81d-a7a2136fdd14/ed2e3011-1fbf-423e-aa8b-2b4bbe99b1f1"
+					(reference "#PWR0205")
 					(unit 1)
 				)
@@
 		(dnp no)
 		(fields_autoplaced yes)
-		(property "Reference" "#PWR024"
+		(property "Reference" "#PWR0202"
 			(at 67.31 147.32 0)
 			(effects
@@
 		)
 		(instances
-			(project ""
-				(path "/95aff260-2720-4733-a81d-a7a2136fdd14/ed2e3011-1fbf-423e-aa8b-2b4bbe99b1f1"
-					(reference "#PWR024")
+			(project "gdp"
+				(path "/95aff260-2720-4733-a81d-a7a2136fdd14/ed2e3011-1fbf-423e-aa8b-2b4bbe99b1f1"
+					(reference "#PWR0202")
 					(unit 1)
 				)
@@
 		(dnp no)
 		(fields_autoplaced yes)
-		(property "Reference" "#PWR030"
+		(property "Reference" "#PWR0206"
 			(at 138.43 86.36 0)
 			(effects
@@
 			(project "gdp"
 				(path "/95aff260-2720-4733-a81d-a7a2136fdd14/ed2e3011-1fbf-423e-aa8b-2b4bbe99b1f1"
-					(reference "#PWR030")
+					(reference "#PWR0206")
 					(unit 1)
 				)
@@
 		(on_board yes)
 		(dnp no)
-		(property "Reference" "SH10"
+		(property "Reference" "SH8"
 			(at 80.01 119.38 0)
 			(effects
@@
 		)
 		(instances
-			(project "replica"
-				(path "/1aaa08cd-2585-4601-8223-7ea6b691e31d"
-					(reference "SH10")
-					(unit 1)
-				)
-			)
 			(project "gdp"
 				(path "/95aff260-2720-4733-a81d-a7a2136fdd14/ed2e3011-1fbf-423e-aa8b-2b4bbe99b1f1"
@@
 		(dnp no)
 		(fields_autoplaced yes)
-		(property "Reference" "#PWR031"
+		(property "Reference" "#PWR0203"
 			(at 187.96 83.82 0)
 			(effects
@@
 		)
 		(instances
-			(project ""
-				(path "/95aff260-2720-4733-a81d-a7a2136fdd14/ed2e3011-1fbf-423e-aa8b-2b4bbe99b1f1"
-					(reference "#PWR031")
+			(project "gdp"
+				(path "/95aff260-2720-4733-a81d-a7a2136fdd14/ed2e3011-1fbf-423e-aa8b-2b4bbe99b1f1"
+					(reference "#PWR0203")
 					(unit 1)
 				)
@@
 		(on_board yes)
 		(dnp no)
-		(property "Reference" "SH11"
+		(property "Reference" "SH7"
 			(at 77.47 119.38 0)
 			(effects
@@
 		)
 		(instances
-			(project "replica"
-				(path "/1aaa08cd-2585-4601-8223-7ea6b691e31d"
-					(reference "SH11")
-					(unit 1)
-				)
-			)
 			(project "gdp"
 				(path "/95aff260-2720-4733-a81d-a7a2136fdd14/ed2e3011-1fbf-423e-aa8b-2b4bbe99b1f1"
@@
 		(on_board yes)
 		(dnp no)
-		(property "Reference" "SH4"
+		(property "Reference" "SH9"
 			(at 82.55 119.38 0)
 			(effects
@@
 		)
 		(instances
-			(project "replica"
-				(path "/1aaa08cd-2585-4601-8223-7ea6b691e31d"
-					(reference "SH4")
-					(unit 1)
-				)
-			)
 			(project "gdp"
 				(path "/95aff260-2720-4733-a81d-a7a2136fdd14/ed2e3011-1fbf-423e-aa8b-2b4bbe99b1f1"
@@
 		(dnp no)
 		(fields_autoplaced yes)
-		(property "Reference" "#PWR026"
+		(property "Reference" "#PWR0200"
 			(at 97.79 125.73 0)
 			(effects
@@
 			(project "gdp"
 				(path "/95aff260-2720-4733-a81d-a7a2136fdd14/ed2e3011-1fbf-423e-aa8b-2b4bbe99b1f1"
-					(reference "#PWR026")
+					(reference "#PWR0200")
 					(unit 1)
 				)
@@
 		(dnp no)
 		(fields_autoplaced yes)
-		(property "Reference" "IC60"
+		(property "Reference" "IC17"
 			(at 190.1541 77.47 0)
 			(effects
@@
 			)
 		)
-		(property "Footprint" "Package_DIP:DIP-16_W7.62mm"
+		(property "Footprint" "Package_DIP:DIP-40_W15.24mm"
 			(at 186.69 77.47 0)
 			(effects
@@
 		)
 		(instances
-			(project "replica"
-				(path "/1aaa08cd-2585-4601-8223-7ea6b691e31d"
-					(reference "IC60")
-					(unit 1)
-				)
-			)
 			(project "gdp"
 				(path "/95aff260-2720-4733-a81d-a7a2136fdd14/ed2e3011-1fbf-423e-aa8b-2b4bbe99b1f1"
@@
 		(dnp no)
 		(fields_autoplaced yes)
-		(property "Reference" "IC8"
+		(property "Reference" "IC6"
 			(at 116.4941 109.22 0)
 			(effects
@@
 			)
 		)
-		(property "Footprint" "Package_DIP:DIP-20_W7.62mm"
+		(property "Footprint" "Package_DIP:DIP-16_W7.62mm"
 			(at 116.84 109.22 0)
 			(effects
@@
 		)
 		(instances
-			(project "replica"
-				(path "/1aaa08cd-2585-4601-8223-7ea6b691e31d"
-					(reference "IC8")
-					(unit 1)
-				)
-			)
 			(project "gdp"
 				(path "/95aff260-2720-4733-a81d-a7a2136fdd14/ed2e3011-1fbf-423e-aa8b-2b4bbe99b1f1"
@@
 		)
 	)
-	(sheet_instances
-		(path "/"
-			(page "1")
-		)
-	)

Commit message: Fixes "CA0" issue in schematics
Connections:
- net CA0: now reaches IC17.27 (B0)
- no-connect marks 8 -> 7
Other:
- note removed: "CA0"
