File: gdp/2.kicad_sch (KiCad schematic)
At the start: 9 parts, among them IC17 MK3881, IC6 74LS85, IC7 PAL16L8

Commit message: Some polishing
Connections:
- net X_IC6_5 renamed x-IC6-5
- net X_IC6_7 renamed x-IC6-7
Changed lines of the file:
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@@
 		)
 	)
-	(label "X_IC6_7"
+	(label "x-IC6-7"
 		(at 124.46 121.92 0)
 		(effects
@@
 		)
 	)
-	(label "X_IC6_5"
+	(label "x-IC6-5"
 		(at 124.46 119.38 0)
 		(effects

Commit message: Further validation sync
Connections:
- net x-IC6-5 renamed unconnected-IC6-5
- net x-IC6-7 renamed unconnected-IC6-7
Changed lines of the file:
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@@
 		)
 	)
-	(label "x-IC6-7"
+	(label "unconnected-IC6-7"
 		(at 124.46 121.92 0)
 		(effects
@@
 		)
 	)
-	(label "x-IC6-5"
+	(label "unconnected-IC6-5"
 		(at 124.46 119.38 0)
 		(effects
