File: gdp/4.kicad_sch (KiCad schematic)
At the start: 16 parts, among them IC10 4164-15, IC12 4164-15, IC13 4164-15, IC14 4164-15, IC15 4164-15, IC16 4164-15, IC17 4164-15, IC3 4164-15, IC4 4164-15, IC40 4164-15, IC5 4164-15, IC59 4164-15, IC6 4164-15, IC7 4164-15, IC8 4164-15, IC9 4164-15

Commit message: Some minor edits
Other:
- company: (none) -> Oddbit Retro
Changed lines of the file:
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@@
   (title_block
     (title "PARTNER GDP")
+    (company "Oddbit Retro")
   )
   (junction (at 116.84 13.97) (diameter 0) (color 0 0 0 0)

Commit message: Adds Sheet 5
Other:
- title: PARTNER GDP -> PARTNER GDP: GDP RAM
Changed lines of the file:
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@@
 	(paper "A4")
 	(title_block
-		(title "PARTNER GDP")
+		(title "PARTNER GDP: GDP RAM")
 		(company "Oddbit Retro")
+		(comment 1 "NARISAL: MIHA GRČAR")
 	)
 	(junction

Commit message: Adds Sheet 9
Parts:
- removed IC13: 4164-15, symbol 74xx_IEEE:74LS352
- added IC37: 4164-15, symbol 74xx_IEEE:74LS352
- renumbered IC12 to IC36, IC15 to IC38, IC10 to IC39, IC8 to IC41, IC6 to IC42, IC7 to IC43, IC14 to IC53, IC9 to IC54, IC16 to IC55, IC17 to IC56, IC3 to IC57, IC5 to IC58, IC4 to IC60
Connections:
- net +5V: now also IC37.8 (VCC)
- net GA0: now also IC37.5 (A0)
- net GA1: now also IC37.7 (A1)
- net GA2: now also IC37.6 (A2)
- net GA3: now also IC37.12 (A3)
- net GA4: now also IC37.11 (A4)
- net GA5: now also IC37.10 (A5)
- net GA6: now also IC37.13 (A6)
- net GA7: now also IC37.9 (A7)
- net GDO1: now also IC37.14 (DOUT)
- net GNDD: now also IC37.16 (GND)
- net RAS1: now also IC37.4 (RAS)
- net ~{CAS}: now also IC37.15 (CAS)
- net ~{DINX}: now also IC37.2 (DIN)
- net ~{WRITE}: now also IC37.3 (WR)
Other:
- moved on the sheet: IC36, IC38, IC39, IC40, IC41, IC42, IC43, IC53, IC54, IC55, IC56, IC57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

Commit message: Fixes Sheet 4
Connections:
- net GDO0: no longer IC54.14 (DOUT)
- net GDO1: no longer IC37.14 (DOUT), IC38.14 (DOUT), IC39.14 (DOUT), IC41.14 (DOUT), IC42.14 (DOUT), IC56.14 (DOUT), IC60.14 (DOUT)
- net GDO2: no longer IC36.14 (DOUT), IC43.14 (DOUT), IC53.14 (DOUT), IC55.14 (DOUT), IC58.14 (DOUT)
- net RAS0: no longer IC36.4 (RAS), IC43.4 (RAS), IC53.4 (RAS), IC54.4 (RAS), IC55.4 (RAS), IC57.4 (RAS), IC58.4 (RAS)
- net RAS1: no longer IC37.4 (RAS), IC38.4 (RAS), IC39.4 (RAS), IC41.4 (RAS), IC42.4 (RAS), IC56.4 (RAS), IC60.4 (RAS)
- new net GDO10: IC36.14 (DOUT)
- new net GDO11: IC37.14 (DOUT)
- new net GDO12: IC53.14 (DOUT)
- new net GDO13: IC38.14 (DOUT)
- new net GDO14: IC55.14 (DOUT)
- new net GDO15: IC56.14 (DOUT)
- new net GDO3: IC60.14 (DOUT)
- new net GDO4: IC58.14 (DOUT)
- new net GDO5: IC42.14 (DOUT)
- new net GDO6: IC43.14 (DOUT)
- new net GDO7: IC41.14 (DOUT)
- new net GDO8: IC54.14 (DOUT)
- new net GDO9: IC39.14 (DOUT)
- new net RAS10: IC36.4 (RAS)
- new net RAS11: IC37.4 (RAS)
- new net RAS12: IC53.4 (RAS)
- new net RAS13: IC38.4 (RAS)
- new net RAS14: IC55.4 (RAS)
- new net RAS15: IC56.4 (RAS)
- new net RAS2: IC57.4 (RAS)
- new net RAS3: IC60.4 (RAS)
- new net RAS4: IC58.4 (RAS)
- new net RAS5: IC42.4 (RAS)
- new net RAS6: IC43.4 (RAS)
- new net RAS7: IC41.4 (RAS)
- new net RAS8: IC54.4 (RAS)
- new net RAS9: IC39.4 (RAS)

Commit message: Initial footprint assignment
Parts:
- IC11: renamed from IC40; footprint (none) -> Package_DIP:DIP-16_W7.62mm
- IC12: renamed from IC54; footprint (none) -> Package_DIP:DIP-16_W7.62mm
- IC13: renamed from IC59; footprint (none) -> Package_DIP:DIP-16_W7.62mm
- IC14: renamed from IC39; footprint (none) -> Package_DIP:DIP-16_W7.62mm
- IC15: renamed from IC57; footprint (none) -> Package_DIP:DIP-16_W7.62mm
- IC16: renamed from IC36; footprint (none) -> Package_DIP:DIP-16_W7.62mm
- IC17: renamed from IC60; footprint (none) -> Package_DIP:DIP-16_W7.62mm
- IC18: renamed from IC37; footprint (none) -> Package_DIP:DIP-16_W7.62mm
- IC19: renamed from IC58; footprint (none) -> Package_DIP:DIP-16_W7.62mm
- IC20: renamed from IC53; footprint (none) -> Package_DIP:DIP-16_W7.62mm
- IC21: renamed from IC42; footprint (none) -> Package_DIP:DIP-16_W7.62mm
- IC22: renamed from IC38; footprint (none) -> Package_DIP:DIP-16_W7.62mm
- IC23: renamed from IC43; footprint (none) -> Package_DIP:DIP-16_W7.62mm
- IC24: renamed from IC55; footprint (none) -> Package_DIP:DIP-16_W7.62mm
- IC25: renamed from IC41; footprint (none) -> Package_DIP:DIP-16_W7.62mm
- IC26: renamed from IC56; footprint (none) -> Package_DIP:DIP-16_W7.62mm
