File: gdp/4.kicad_sch (KiCad schematic)
At the start: 16 parts, among them IC11 4164-15, IC12 4164-15, IC13 4164-15, IC14 4164-15, IC15 4164-15, IC16 4164-15, IC17 4164-15, IC18 4164-15, IC19 4164-15, IC20 4164-15, IC21 4164-15, IC22 4164-15, IC23 4164-15, IC24 4164-15, IC25 4164-15, IC26 4164-15

Commit message: Fixes refs
Parts:
- renumbered IC16 to IC36, IC18 to IC37, IC22 to IC38, IC14 to IC39, IC11 to IC40, IC25 to IC41, IC21 to IC42, IC23 to IC43, IC20 to IC53, IC12 to IC54, IC24 to IC55, IC26 to IC56, IC15 to IC57, IC19 to IC58, IC13 to IC59, IC17 to IC60
Changed lines of the file:
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@@
 		(on_board yes)
 		(dnp no)
-		(property "Reference" "IC19"
+		(property "Reference" "IC58"
 			(at 165.1 57.15 0)
 			(effects
@@
 			(project "gdp"
 				(path "/95aff260-2720-4733-a81d-a7a2136fdd14/e98871a8-cfbc-48a6-bd1b-47ad43a4804b"
-					(reference  "IC58")
+					(reference "IC58")
 					(unit 1)
 				)
@@
 		(on_board yes)
 		(dnp no)
-		(property "Reference" "IC24"
+		(property "Reference" "IC55"
 			(at 227.965 132.08 0)
 			(effects
@@
 			(project "gdp"
 				(path "/95aff260-2720-4733-a81d-a7a2136fdd14/e98871a8-cfbc-48a6-bd1b-47ad43a4804b"
-					(reference  "IC55")
+					(reference "IC55")
 					(unit 1)
 				)
@@
 		(on_board yes)
 		(dnp no)
-		(property "Reference" "IC20"
+		(property "Reference" "IC53"
 			(at 165.1 132.08 0)
 			(effects
@@
 			(project "gdp"
 				(path "/95aff260-2720-4733-a81d-a7a2136fdd14/e98871a8-cfbc-48a6-bd1b-47ad43a4804b"
-					(reference  "IC53")
+					(reference "IC53")
 					(unit 1)
 				)
@@
 		(on_board yes)
 		(dnp no)
-		(property "Reference" "IC17"
+		(property "Reference" "IC60"
 			(at 135.89 57.15 0)
 			(effects
@@
 			(project "gdp"
 				(path "/95aff260-2720-4733-a81d-a7a2136fdd14/e98871a8-cfbc-48a6-bd1b-47ad43a4804b"
-					(reference  "IC60")
+					(reference "IC60")
 					(unit 1)
 				)
@@
 		(on_board yes)
 		(dnp no)
-		(property "Reference" "IC16"
+		(property "Reference" "IC36"
 			(at 102.235 132.08 0)
 			(effects
@@
 			(project "gdp"
 				(path "/95aff260-2720-4733-a81d-a7a2136fdd14/e98871a8-cfbc-48a6-bd1b-47ad43a4804b"
-					(reference  "IC36")
+					(reference "IC36")
 					(unit 1)
 				)
@@
 		(on_board yes)
 		(dnp no)
-		(property "Reference" "IC13"
+		(property "Reference" "IC59"
 			(at 73.025 57.15 0)
 			(effects
@@
 			(project "gdp"
 				(path "/95aff260-2720-4733-a81d-a7a2136fdd14/e98871a8-cfbc-48a6-bd1b-47ad43a4804b"
-					(reference  "IC59")
+					(reference "IC59")
 					(unit 1)
 				)
@@
 		(on_board yes)
 		(dnp no)
-		(property "Reference" "IC26"
+		(property "Reference" "IC56"
 			(at 261.62 132.08 0)
 			(effects
@@
 			(project "gdp"
 				(path "/95aff260-2720-4733-a81d-a7a2136fdd14/e98871a8-cfbc-48a6-bd1b-47ad43a4804b"
-					(reference  "IC56")
+					(reference "IC56")
 					(unit 1)
 				)
@@
 		(on_board yes)
 		(dnp no)
-		(property "Reference" "IC18"
+		(property "Reference" "IC37"
 			(at 135.89 132.08 0)
 			(effects
@@
 			(project "gdp"
 				(path "/95aff260-2720-4733-a81d-a7a2136fdd14/e98871a8-cfbc-48a6-bd1b-47ad43a4804b"
-					(reference  "IC37")
+					(reference "IC37")
 					(unit 1)
 				)
@@
 		(on_board yes)
 		(dnp no)
-		(property "Reference" "IC14"
+		(property "Reference" "IC39"
 			(at 73.025 132.08 0)
 			(effects
@@
 			(project "gdp"
 				(path "/95aff260-2720-4733-a81d-a7a2136fdd14/e98871a8-cfbc-48a6-bd1b-47ad43a4804b"
-					(reference  "IC39")
+					(reference "IC39")
 					(unit 1)
 				)
@@
 		(on_board yes)
 		(dnp no)
-		(property "Reference" "IC23"
+		(property "Reference" "IC43"
 			(at 227.965 57.15 0)
 			(effects
@@
 			(project "gdp"
 				(path "/95aff260-2720-4733-a81d-a7a2136fdd14/e98871a8-cfbc-48a6-bd1b-47ad43a4804b"
-					(reference  "IC43")
+					(reference "IC43")
 					(unit 1)
 				)
@@
 		(on_board yes)
 		(dnp no)
-		(property "Reference" "IC22"
+		(property "Reference" "IC38"
 			(at 198.755 132.08 0)
 			(effects
@@
 			(project "gdp"
 				(path "/95aff260-2720-4733-a81d-a7a2136fdd14/e98871a8-cfbc-48a6-bd1b-47ad43a4804b"
-					(reference  "IC38")
+					(reference "IC38")
 					(unit 1)
 				)
@@
 		(on_board yes)
 		(dnp no)
-		(property "Reference" "IC15"
+		(property "Reference" "IC57"
 			(at 102.235 57.15 0)
 			(effects
@@
 			(project "gdp"
 				(path "/95aff260-2720-4733-a81d-a7a2136fdd14/e98871a8-cfbc-48a6-bd1b-47ad43a4804b"
-					(reference  "IC57")
+					(reference "IC57")
 					(unit 1)
 				)
@@
 		(on_board yes)
 		(dnp no)
-		(property "Reference" "IC11"
+		(property "Reference" "IC40"
 			(at 39.37 57.15 0)
 			(effects
@@
 			(project "gdp"
 				(path "/95aff260-2720-4733-a81d-a7a2136fdd14/e98871a8-cfbc-48a6-bd1b-47ad43a4804b"
-					(reference  "IC40")
+					(reference "IC40")
 					(unit 1)
 				)
@@
 		(on_board yes)
 		(dnp no)
-		(property "Reference" "IC21"
+		(property "Reference" "IC42"
 			(at 198.755 57.15 0)
 			(effects
@@
 			(project "gdp"
 				(path "/95aff260-2720-4733-a81d-a7a2136fdd14/e98871a8-cfbc-48a6-bd1b-47ad43a4804b"
-					(reference  "IC42")
+					(reference "IC42")
 					(unit 1)
 				)
@@
 		(on_board yes)
 		(dnp no)
-		(property "Reference" "IC25"
+		(property "Reference" "IC41"
 			(at 261.62 57.15 0)
 			(effects
@@
 			(project "gdp"
 				(path "/95aff260-2720-4733-a81d-a7a2136fdd14/e98871a8-cfbc-48a6-bd1b-47ad43a4804b"
-					(reference  "IC41")
+					(reference "IC41")
 					(unit 1)
 				)
@@
 		(on_board yes)
 		(dnp no)
-		(property "Reference" "IC12"
+		(property "Reference" "IC54"
 			(at 39.37 132.08 0)
 			(effects
@@
 			(project "gdp"
 				(path "/95aff260-2720-4733-a81d-a7a2136fdd14/e98871a8-cfbc-48a6-bd1b-47ad43a4804b"
-					(reference  "IC54")
-					(unit 1)
-				)
+					(reference "IC54")
+					(unit 1)
+				)
