File: gdp/13.kicad_sch (KiCad schematic)
At the start: 28 parts, among them IC63 7406, IC72 74S04, T1 2N2905A, T2 2N2905A

Commit message: Some minor edits
Other:
- company: (none) -> Oddbit Retro
- title: (none) -> PARTNER GDP
Changed lines of the file:
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@@
 (kicad_sch (version 20230121) (generator eeschema)
   (paper "A4")
+  (title_block
+    (title "PARTNER GDP")
+    (company "Oddbit Retro")
+  )
   (junction (at 185.42 90.805) (diameter 0) (color 0 0 0 0)
   )

Commit message: Adds Sheet 3
Parts:
- gave numbers to parts that had none: 9
- renumbered CK23 to CK5, ST3 to JM1, SH2 to SH15, SH2 to SH16, SH2 to SH17, SH2 to SH18, SH2 to SH19

Commit message: Adds Sheet 9
Parts:
- CK53: renamed from CK5; value U22 -> 22U
- R25: renamed from R12; value 75R -> 1K0
- R32: renamed from R11; value 120R -> 1K8
- R37: renamed from R11; value 75R -> 1K5
- R39: renamed from R11; value 120R -> 2K2
- R41: renamed from R11; value 120R -> 1K5
- R41: renamed from R11; value 120R -> 1K2
- R43: renamed from R11; value 75R -> 680R
- R46: renamed from R11; value 75R -> 1K2
- R47: renamed from R11; value 75R -> 820R
- renumbered R43 to R24, R35 to R29, R37 to R30, R44 to R31, R36 to R39, R38 to R40, JM2 to ST6, JM1 to ST7
Changed lines of the file:
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@@
 		(on_board yes)
 		(dnp no)
-		(property "Reference" "JM1"
+		(property "Reference" "ST7"
 			(at 203.835 120.015 0)
 			(effects
@@
 			(project "gdp"
 				(path "/95aff260-2720-4733-a81d-a7a2136fdd14/123266b5-995d-4527-ad06-2cb8a9732efd"
-					(reference "JM1")
+					(reference "ST7")
 					(unit 1)
 				)
@@
 		(on_board yes)
 		(dnp no)
-		(property "Reference" "R11"
+		(property "Reference" "R39"
 			(at 176.53 106.045 0)
 			(effects
@@
 			)
 		)
-		(property "Value" "120R"
+		(property "Value" "2K2"
 			(at 179.07 106.045 0)
 			(effects
@@
 			(project "gdp"
 				(path "/95aff260-2720-4733-a81d-a7a2136fdd14/123266b5-995d-4527-ad06-2cb8a9732efd"
-					(reference "R11")
+					(reference "R39")
 					(unit 1)
 				)
@@
 		(on_board yes)
 		(dnp no)
-		(property "Reference" "R11"
+		(property "Reference" "R37"
 			(at 153.67 69.85 0)
 			(effects
@@
 			)
 		)
-		(property "Value" "75R"
+		(property "Value" "1K5"
 			(at 153.67 72.39 0)
 			(effects
@@
 			(project "gdp"
 				(path "/95aff260-2720-4733-a81d-a7a2136fdd14/123266b5-995d-4527-ad06-2cb8a9732efd"
-					(reference "R11")
+					(reference "R37")
 					(unit 1)
 				)
@@
 		(on_board yes)
 		(dnp no)
-		(property "Reference" "R43"
+		(property "Reference" "R24"
 			(at 171.45 52.705 0)
 			(effects
@@
 			(project "gdp"
 				(path "/95aff260-2720-4733-a81d-a7a2136fdd14/123266b5-995d-4527-ad06-2cb8a9732efd"
-					(reference "R43")
+					(reference "R24")
 					(unit 1)
 				)
@@
 		(on_board yes)
 		(dnp no)
-		(property "Reference" "CK5"
+		(property "Reference" "CK53"
 			(at 165.735 43.815 0)
 			(effects
@@
 			)
 		)
-		(property "Value" "U22"
+		(property "Value" "22U"
 			(at 165.735 46.355 0)
 			(effects
@@
 			(project "gdp"
 				(path "/95aff260-2720-4733-a81d-a7a2136fdd14/123266b5-995d-4527-ad06-2cb8a9732efd"
-					(reference "CK5")
+					(reference "CK53")
 					(unit 1)
 				)
@@
 		(on_board yes)
 		(dnp no)
-		(property "Reference" "R11"
+		(property "Reference" "R47"
 			(at 161.925 69.85 0)
 			(effects
@@
 			)
 		)
-		(property "Value" "75R"
+		(property "Value" "820R"
 			(at 161.925 72.39 0)
 			(effects
@@
 			(project "gdp"
 				(path "/95aff260-2720-4733-a81d-a7a2136fdd14/123266b5-995d-4527-ad06-2cb8a9732efd"
-					(reference "R11")
+					(reference "R47")
 					(unit 1)
 				)
@@
 		(on_board yes)
 		(dnp no)
-		(property "Reference" "JM2"
+		(property "Reference" "ST6"
 			(at 189.23 122.555 0)
 			(effects
@@
 			(project "gdp"
 				(path "/95aff260-2720-4733-a81d-a7a2136fdd14/123266b5-995d-4527-ad06-2cb8a9732efd"
-					(reference "JM2")
+					(reference "ST6")
 					(unit 1)
 				)
@@
 		(on_board yes)
 		(dnp no)
-		(property "Reference" "R38"
+		(property "Reference" "R40"
 			(at 200.025 43.815 0)
 			(effects
@@
 			(project "gdp"
 				(path "/95aff260-2720-4733-a81d-a7a2136fdd14/123266b5-995d-4527-ad06-2cb8a9732efd"
-					(reference "R38")
+					(reference "R40")
 					(unit 1)
 				)
@@
 		(on_board yes)
 		(dnp no)
-		(property "Reference" "R12"
+		(property "Reference" "R25"
 			(at 139.7 69.85 0)
 			(effects
@@
 			)
 		)
-		(property "Value" "75R"
+		(property "Value" "1K0"
 			(at 139.7 72.39 0)
 			(effects
@@
 			(project "gdp"
 				(path "/95aff260-2720-4733-a81d-a7a2136fdd14/123266b5-995d-4527-ad06-2cb8a9732efd"
-					(reference "R12")
+					(reference "R25")
 					(unit 1)
 				)
@@
 		(on_board yes)
 		(dnp no)
-		(property "Reference" "R11"
+		(property "Reference" "R32"
 			(at 176.53 97.79 0)
 			(effects
@@
 			)
 		)
-		(property "Value" "120R"
+		(property "Value" "1K8"
 			(at 179.07 97.79 0)
 			(effects
@@
 			(project "gdp"
 				(path "/95aff260-2720-4733-a81d-a7a2136fdd14/123266b5-995d-4527-ad06-2cb8a9732efd"
-					(reference "R11")
+					(reference "R32")
 					(unit 1)
 				)
@@
 		(on_board yes)
 		(dnp no)
-		(property "Reference" "R44"
+		(property "Reference" "R31"
 			(at 200.025 70.485 0)
 			(effects
@@
 			(project "gdp"
 				(path "/95aff260-2720-4733-a81d-a7a2136fdd14/123266b5-995d-4527-ad06-2cb8a9732efd"
-					(reference "R44")
+					(reference "R31")
 					(unit 1)
 				)
@@
 		(on_board yes)
 		(dnp no)
-		(property "Reference" "R11"
+		(property "Reference" "R46"
 			(at 146.685 69.85 0)
 			(effects
@@
 			)
 		)
-		(property "Value" "75R"
+		(property "Value" "1K2"
 			(at 146.685 72.39 0)
 			(effects
@@
 			(project "gdp"
 				(path "/95aff260-2720-4733-a81d-a7a2136fdd14/123266b5-995d-4527-ad06-2cb8a9732efd"
-					(reference "R11")
+					(reference "R46")
 					(unit 1)
 				)
@@
 		(on_board yes)
 		(dnp no)
-		(property "Reference" "R36"
+		(property "Reference" "R39"
 			(at 186.69 43.815 0)
 			(effects
@@
 			(project "gdp"
 				(path "/95aff260-2720-4733-a81d-a7a2136fdd14/123266b5-995d-4527-ad06-2cb8a9732efd"
-					(reference "R36")
+					(reference "R39")
 					(unit 1)
 				)
@@
 		(on_board yes)
 		(dnp no)
-		(property "Reference" "R35"
+		(property "Reference" "R29"
 			(at 132.715 43.815 0)
 			(effects
@@
 			(project "gdp"
 				(path "/95aff260-2720-4733-a81d-a7a2136fdd14/123266b5-995d-4527-ad06-2cb8a9732efd"
-					(reference "R35")
+					(reference "R29")
 					(unit 1)
 				)
@@
 		(on_board yes)
 		(dnp no)
-		(property "Reference" "R11"
+		(property "Reference" "R43"
 			(at 132.715 69.85 0)
 			(effects
@@
 			)
 		)
-		(property "Value" "75R"
+		(property "Value" "680R"
 			(at 132.715 72.39 0)
 			(effects
@@
 			(project "gdp"
 				(path "/95aff260-2720-4733-a81d-a7a2136fdd14/123266b5-995d-4527-ad06-2cb8a9732efd"
-					(reference "R11")
+					(reference "R43")
 					(unit 1)
 				)
@@
 		(on_board yes)
 		(dnp no)
-		(property "Reference" "R11"
+		(property "Reference" "R41"
 			(at 176.53 89.535 0)
 			(effects
@@
 			)
 		)
-		(property "Value" "120R"
+		(property "Value" "1K5"
 			(at 179.07 89.535 0)
 			(effects
@@
 			(project "gdp"
 				(path "/95aff260-2720-4733-a81d-a7a2136fdd14/123266b5-995d-4527-ad06-2cb8a9732efd"
-					(reference "R11")
+					(reference "R41")
 					(unit 1)
 				)
@@
 		(on_board yes)
 		(dnp no)
-		(property "Reference" "R37"
+		(property "Reference" "R30"
 			(at 151.765 43.815 0)
 			(effects
@@
 			(project "gdp"
 				(path "/95aff260-2720-4733-a81d-a7a2136fdd14/123266b5-995d-4527-ad06-2cb8a9732efd"
-					(reference "R37")
+					(reference "R30")
 					(unit 1)
 				)
@@
 		(on_board yes)
 		(dnp no)
-		(property "Reference" "R11"
+		(property "Reference" "R41"
 			(at 176.53 114.3 0)
 			(effects
@@
 			)
 		)
-		(property "Value" "120R"
+		(property "Value" "1K2"
 			(at 179.07 114.3 0)
 			(effects
@@
 			(project "gdp"
 				(path "/95aff260-2720-4733-a81d-a7a2136fdd14/123266b5-995d-4527-ad06-2cb8a9732efd"
-					(reference "R11")
-					(unit 1)
-				)
+					(reference "R41")
+					(unit 1)
+				)

Commit message: Adds Sheet 11
Other:
- title: PARTNER GDP -> PARTNER GDP: VIDEOMIX
Changed lines of the file:
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@@
 	(paper "A4")
 	(title_block
-		(title "PARTNER GDP")
+		(title "PARTNER GDP: VIDEOMIX")
 		(company "Oddbit Retro")
+		(comment 1 "NARISAL: MIHA GRČAR")
 	)
 	(junction

Commit message: Fixes (component refs...)
Parts:
- renumbered R32 to R38, R40 to R42, R41 to R44, R39 to R45
Changed lines of the file:
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@@
 		(on_board yes)
 		(dnp no)
-		(property "Reference" "R40"
+		(property "Reference" "R42"
 			(at 176.53 81.28 0)
 			(effects
@@
 			(project "gdp"
 				(path "/95aff260-2720-4733-a81d-a7a2136fdd14/123266b5-995d-4527-ad06-2cb8a9732efd"
-					(reference "R40")
+					(reference "R42")
 					(unit 1)
 				)
@@
 		(on_board yes)
 		(dnp no)
-		(property "Reference" "R39"
+		(property "Reference" "R45"
 			(at 176.53 106.045 0)
 			(effects
@@
 			(project "gdp"
 				(path "/95aff260-2720-4733-a81d-a7a2136fdd14/123266b5-995d-4527-ad06-2cb8a9732efd"
-					(reference "R39")
+					(reference "R45")
 					(unit 1)
 				)
@@
 		(on_board yes)
 		(dnp no)
-		(property "Reference" "R32"
+		(property "Reference" "R38"
 			(at 176.53 97.79 0)
 			(effects
@@
 			(project "gdp"
 				(path "/95aff260-2720-4733-a81d-a7a2136fdd14/123266b5-995d-4527-ad06-2cb8a9732efd"
-					(reference "R32")
+					(reference "R38")
 					(unit 1)
 				)
@@
 		(on_board yes)
 		(dnp no)
-		(property "Reference" "R41"
+		(property "Reference" "R44"
 			(at 176.53 89.535 0)
 			(effects
@@
 			(project "gdp"
 				(path "/95aff260-2720-4733-a81d-a7a2136fdd14/123266b5-995d-4527-ad06-2cb8a9732efd"
-					(reference "R41")
-					(unit 1)
-				)
+					(reference "R44")
+					(unit 1)
+				)

Commit message: Adds Sheet 14 (WIP)
Parts:
- IC72: value 74S04 -> 74LS04
Connections:
- net HCSYNC- renamed ~{HCSYNC}
- net VSYNC- renamed ~{VSYNC}
Changed lines of the file:
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@@
 		)
 	)
-	(global_label "HCSYNC-"
+	(global_label "~{HCSYNC}"
 		(shape input)
 		(at 91.44 115.57 180)
@@
 		)
 		(property "Intersheetrefs" "${INTERSHEET_REFS}"
-			(at 79.3833 115.57 0)
+			(at 80.9557 115.57 0)
 			(effects
 				(font
@@
 		)
 	)
-	(global_label "VSYNC-"
+	(global_label "~{VSYNC}"
 		(shape input)
 		(at 91.44 152.4 180)
@@
 		)
 		(property "Intersheetrefs" "${INTERSHEET_REFS}"
-			(at 80.8952 152.4 0)
+			(at 82.4676 152.4 0)
 			(effects
 				(font
@@
 			)
 		)
-		(property "Value" "74S04"
+		(property "Value" "74LS04"
 			(at 98.425 75.565 0)
 			(effects
@@
 			)
 		)
-		(property "Description" ""
+		(property "Description" "Hex Inverter"
 			(at 99.06 74.295 0)
 			(effects

Commit message: Initial footprint assignment
Parts:
- CK5: renamed from CK53; footprint (none) -> Capacitor_THT:C_Disc_D4.3mm_W1.9mm_P5.00mm
- IC66: renamed from IC72; footprint (none) -> Package_DIP:DIP-14_W7.62mm
- IC67: renamed from IC63; footprint (none) -> Package_DIP:DIP-14_W7.62mm
- R34: renamed from R29; footprint (none) -> Resistor_THT:R_Axial_DIN0207_L6.3mm_D2.5mm_P7.62mm_Horizontal
- R35: renamed from R43; footprint (none) -> Resistor_THT:R_Axial_DIN0207_L6.3mm_D2.5mm_P7.62mm_Horizontal
- R36: renamed from R25; footprint (none) -> Resistor_THT:R_Axial_DIN0207_L6.3mm_D2.5mm_P7.62mm_Horizontal
- R37: renamed from R46; footprint (none) -> Resistor_THT:R_Axial_DIN0207_L6.3mm_D2.5mm_P7.62mm_Horizontal
- R38: renamed from R30; footprint (none) -> Resistor_THT:R_Axial_DIN0207_L6.3mm_D2.5mm_P7.62mm_Horizontal
- R39: renamed from R37; footprint (none) -> Resistor_THT:R_Axial_DIN0207_L6.3mm_D2.5mm_P7.62mm_Horizontal
- R40: renamed from R47; footprint (none) -> Resistor_THT:R_Axial_DIN0207_L6.3mm_D2.5mm_P7.62mm_Horizontal
- R41: renamed from R24; footprint (none) -> Resistor_THT:R_Axial_DIN0207_L6.3mm_D2.5mm_P7.62mm_Horizontal
- R42, R45: footprint (none) -> Resistor_THT:R_Axial_DIN0207_L6.3mm_D2.5mm_P7.62mm_Horizontal
- R43: renamed from R44; footprint (none) -> Resistor_THT:R_Axial_DIN0207_L6.3mm_D2.5mm_P7.62mm_Horizontal
- R44: renamed from R38; footprint (none) -> Resistor_THT:R_Axial_DIN0207_L6.3mm_D2.5mm_P7.62mm_Horizontal
- R46: renamed from R41; footprint (none) -> Resistor_THT:R_Axial_DIN0207_L6.3mm_D2.5mm_P7.62mm_Horizontal
- R47: renamed from R39; footprint (none) -> Resistor_THT:R_Axial_DIN0207_L6.3mm_D2.5mm_P7.62mm_Horizontal
- R48: renamed from R40; footprint (none) -> Resistor_THT:R_Axial_DIN0207_L6.3mm_D2.5mm_P7.62mm_Horizontal
- R49: renamed from R31; footprint (none) -> Resistor_THT:R_Axial_DIN0207_L6.3mm_D2.5mm_P7.62mm_Horizontal
- SH13: renamed from SH19; footprint (none) -> Connector_PinHeader_2.54mm:PinHeader_1x02_P2.54mm_Vertical
- SH14: renamed from SH18; footprint (none) -> Connector_PinHeader_2.54mm:PinHeader_1x02_P2.54mm_Vertical
- SH15: renamed from SH16; footprint (none) -> Connector_PinHeader_2.54mm:PinHeader_1x02_P2.54mm_Vertical
- SH16: renamed from SH17; footprint (none) -> Connector_PinHeader_2.54mm:PinHeader_1x02_P2.54mm_Vertical
- SH17: renamed from SH15; footprint (none) -> Connector_PinHeader_2.54mm:PinHeader_1x02_P2.54mm_Vertical
- ST6: value Conn_01x03 -> 3; footprint (none) -> Connector_PinHeader_2.54mm:PinHeader_1x03_P2.54mm_Vertical
- ST7: value MODU2-10 -> 10; footprint (none) -> Connector_PinHeader_2.54mm:PinHeader_1x10_P2.54mm_Vertical
- T1, T2: footprint (none) -> Package_TO_SOT_THT:TO-92_Wide

Commit message: Results of some measurements
Connections:
- net at ST7.8 (Pin_8): now also R41.2, T1.1 (C)
- net at ST7.9 (Pin_9): now also SH15.2 (B), SH16.2 (B)
Other:
- moved on the sheet: CK5, IC66C, IC67A, IC67C, IC67E, R34, R35, R37, R38, R40, R41, R43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
