File: gdp/3.kicad_sch (KiCad schematic)
At the start: 0 parts

Commit message: Adds pages 4, 7, 10 (still WIP)
Other:
- title: Partner GDP -> (none)
Changed lines of the file:
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@@
 (kicad_sch (version 20230121) (generator eeschema)
   (paper "A4")
-  (title_block
-    (title "Partner GDP")
-  )
 )

Commit message: Adds Sheet 3
Parts:
- added IC22: PAL16L8, symbol Logic_Programmable:PAL16L8
- added IC23: EF9367, Package_DIP:DIP-40_W15.24mm, symbol MCU_Parallax:P8X32A-D40
- added IC24: PAL10L8, symbol Logic_Programmable:PAL16L8
- added IC49: PAL16R4, symbol Logic_Programmable:PAL16L8
- added R22, R23, R36, R52, R7: 2K2, symbol Device:R
Connections:
- new net: IC24.8 (I8), R23.1
- new net: IC24.11 (I10), R52.1
- new net: IC22.9 (I9), IC23.25 (BLK), IC49.5 (I4)
- new net: IC23.35 (MSL3), IC49.6 (I5)
- new net: IC24.9 (I9), R22.1
- new net: IC23.15 (DIN), IC24.7 (I7)
- new net: IC22.2 (I2), IC23.24 (MW)
- new net: IC22.18 (IO2), IC23.8 (FMAT)
- new net +5V: IC22.20 (VCC), IC23.40 (VCC), IC24.20 (VCC), IC49.20 (VCC), R22.2, R23.2, R36.1, R52.2
- new net A0: IC23.9 (A0)
- new net A1: IC23.10 (A1)
- new net A2: IC23.11 (A2)
- new net A3: IC23.12 (A3)
- new net ALL1: IC24.14 (O6)
- new net D0: IC23.33 (D0)
- new net D1: IC23.32 (D1)
- new net D2: IC23.31 (D2)
- new net D3: IC23.D3 (30)
- new net D4: IC23.29 (D4)
- new net D5: IC23.28 (D5)
- new net D6: IC23.27 (D6)
- new net D7: IC23.26 (D7)
- new net DAD0: IC23.37 (DAD0)
- new net DAD1: IC23.39 (DAD1)
- new net DAD2: IC23.38 (DAD2)
- new net DAD3: IC23.4 (DAD3)
- new net DAD4: IC23.3 (DAD4)
- new net DAD5: IC23.2 (DAD5), IC49.2 (I1)
- new net DAD6: IC23.5 (DAD6), IC49.3 (I2)
- new net DOUT: IC24.15 (O5), IC24.5 (I5)
- new net DOUT1: IC24.3 (I3)
- new net DOUT2: IC24.4 (I4)
- new net EOC: IC22.11 (I10)
- new net FM0: IC22.7 (I7)
- new net FM1: IC22.8 (I8)
- new net GA7: IC49.18 (IO2)
- new net GDPSYNC: IC23.34 (SYNC)
- new net GND: IC22.10 (GND), IC23.20 (GND), IC24.10 (GND), IC49.10 (GND), IC49.11 (~{OE}), R7.1
- new net LOAD: IC22.17 (I03)
- new net MUX1: IC24.2 (I2)
- new net PO: IC49.19 (IO1)
- new net QA: IC22.4 (I4)
- new net QB: IC22.5 (I5)
- new net RBNK: IC49.7 (I6)
- new net SCRLM: IC49.9 (I8)
- new net SHLD: IC22.19 (IO1)
- new net SOUT: IC49.13 (IO7)
- new net WBNK: IC49.8 (I7)
- new net X0: IC23.6 (MSL0)
- new net X1: IC23.36 (MSL1)
- new net X2: IC23.7 (MSL2)
- new net X3: IC49.17 (O3)
- new net X9: IC23.19 (X9)
- new net XORM: IC24.6 (I6)
- new net ~{ALL16}: IC22.14 (IO6)
- new net ~{ALL}: IC22.3 (I3), IC23.22 (ALL), IC24.1 (I1)
- new net ~{CAS}: IC22.15 (IO5)
- new net ~{DINX}: IC24.16 (O4)
- new net ~{ENS}: IC22.13 (IO7)
- new net ~{GDPINT}: IC49.14 (O6)
- new net ~{GDP}: IC23.17 (E)
- new net ~{GINT}: IC23.13 (IRQ), IC49.12 (IO8), R36.2
- new net ~{NORM}: IC24.13 (O7)
- new net ~{SHIFT}: IC24.12 (O8)
- new net ~{WHITE}: IC22.12 (IO8)
- new net ~{WRITE}: IC22.16 (IO4)
- new net ~{WR}: IC23.18 (R/W)
- no-connect marks 0 -> 6

Commit message: Adds Sheet 5
Other:
- company: (none) -> Oddbit Retro
- title: (none) -> PARTNER GDP: GDP + CONTROL
Changed lines of the file:
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@@
 	(generator_version "8.0")
 	(paper "A4")
+	(title_block
+		(title "PARTNER GDP: GDP + CONTROL")
+		(company "Oddbit Retro")
+		(comment 1 "NARISAL: MIHA GRČAR")
+	)
 	(junction
 		(at 180.34 99.06)

Commit message: Adds Sheet 12
Changed lines of the file:
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@@
 	)
 	(bus_entry
-		(at 245.11 139.7)
+		(at 241.3 139.7)
 		(size 2.54 2.54)
 		(stroke
@@
 	)
 	(bus_entry
-		(at 245.11 88.9)
+		(at 241.3 88.9)
 		(size 2.54 2.54)
 		(stroke
@@
 	)
 	(bus_entry
-		(at 245.11 40.64)
+		(at 241.3 40.64)
 		(size 2.54 2.54)
 		(stroke
@@
 	)
 	(bus_entry
-		(at 245.11 86.36)
+		(at 241.3 86.36)
 		(size 2.54 2.54)
 		(stroke
@@
 	(wire
 		(pts
-			(xy 245.11 86.36) (xy 214.63 86.36)
+			(xy 241.3 86.36) (xy 214.63 86.36)
 		)
 		(stroke
@@
 	(bus
 		(pts
-			(xy 247.65 157.48) (xy 252.73 157.48)
+			(xy 243.84 157.48) (xy 248.92 157.48)
 		)
 		(stroke
@@
 	(wire
 		(pts
-			(xy 214.63 88.9) (xy 245.11 88.9)
+			(xy 214.63 88.9) (xy 241.3 88.9)
 		)
 		(stroke
@@
 	(bus
 		(pts
-			(xy 247.65 43.18) (xy 247.65 88.9)
+			(xy 243.84 43.18) (xy 243.84 88.9)
 		)
 		(stroke
@@
 	(wire
 		(pts
-			(xy 214.63 40.64) (xy 245.11 40.64)
+			(xy 214.63 40.64) (xy 241.3 40.64)
 		)
 		(stroke
@@
 	(bus
 		(pts
-			(xy 247.65 142.24) (xy 247.65 157.48)
-		)
-		(stroke
-			(width 0)
-			(type default)
-		)
-	)
-	(wire
-		(pts
-			(xy 214.63 139.7) (xy 245.11 139.7)
+			(xy 243.84 142.24) (xy 243.84 157.48)
+		)
+		(stroke
+			(width 0)
+			(type default)
+		)
+	)
+	(wire
+		(pts
+			(xy 214.63 139.7) (xy 241.3 139.7)
 		)
 		(stroke
@@
 	(bus
 		(pts
-			(xy 247.65 88.9) (xy 247.65 91.44)
+			(xy 243.84 88.9) (xy 243.84 91.44)
 		)
 		(stroke
@@
 	(bus
 		(pts
-			(xy 247.65 91.44) (xy 247.65 142.24)
+			(xy 243.84 91.44) (xy 243.84 142.24)
 		)
 		(stroke
@@
 	)
 	(label "GA7"
-		(at 238.76 139.7 0)
+		(at 237.49 139.7 0)
 		(fields_autoplaced yes)
 		(effects
@@
 	(global_label "{GA7 ~{WRITE} ~{CAS} ~{DINX}}"
 		(shape output)
-		(at 252.73 157.48 0)
+		(at 248.92 157.48 0)
 		(fields_autoplaced yes)
 		(effects
@@
 		)
 		(property "Intersheetrefs" "${INTERSHEET_REFS}"
-			(at 277.3052 157.48 0)
-			(effects
-				(font
+			(at 273.4952 157.48 0)
+			(effects
+				(font

Commit message: Small fixes
Connections:
- net GND: now also IC23.23 (W0)
- net LPEN: now also IC23.21 (LPCK), R7.2
- net MUX1: now also IC49.4 (I3)
- net QC: now also IC22.6 (I6), IC23.1 (CK), IC49.1 (CLK)

Commit message: Initial footprint assignment
Parts:
- IC10: renamed from IC49; footprint (none) -> Package_DIP:DIP-20_W7.62mm
- IC8: renamed from IC24; footprint (none) -> Package_DIP:DIP-20_W7.62mm
- IC9: renamed from IC22; footprint (none) -> Package_DIP:DIP-20_W7.62mm
- R13: renamed from R7; footprint (none) -> Resistor_THT:R_Axial_DIN0207_L6.3mm_D2.5mm_P7.62mm_Horizontal
- R14: renamed from R36; footprint (none) -> Resistor_THT:R_Axial_DIN0207_L6.3mm_D2.5mm_P7.62mm_Horizontal
- R15: renamed from R23; footprint (none) -> Resistor_THT:R_Axial_DIN0207_L6.3mm_D2.5mm_P7.62mm_Horizontal
- R16: renamed from R22; footprint (none) -> Resistor_THT:R_Axial_DIN0207_L6.3mm_D2.5mm_P7.62mm_Horizontal
- R17: renamed from R52; footprint (none) -> Resistor_THT:R_Axial_DIN0207_L6.3mm_D2.5mm_P7.62mm_Horizontal
- renumbered IC23 to IC7

Commit message: Several fixes
Connections:
- net D3: now also IC7.30 (D3); no longer IC7.D3 (30)
Changed lines of the file:
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@@
 		(pin "12"
 		)
-		(pin "D3"
+		(pin "30"
 		)
 		(pin "21"
