File: gdp/3.kicad_sch (KiCad schematic)
At the start: 9 parts, among them IC10 PAL16R4, IC7 EF9367, IC8 PAL10L8, IC9 PAL16L8

Commit message: Fixes refs
Parts:
- renumbered IC9 to IC22, IC7 to IC23, IC8 to IC24, IC10 to IC49, R16 to R22, R15 to R23, R14 to R36, R17 to R52, R13 to R7
Changed lines of the file:
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@@
 		(on_board yes)
 		(dnp no)
-		(property "Reference" "R15"
+		(property "Reference" "R23"
 			(at 144.78 62.23 0)
 			(effects
@@
 			(project "gdp"
 				(path "/95aff260-2720-4733-a81d-a7a2136fdd14/a792f856-eda0-4c7e-9974-4020eb15499f"
-					(reference  "R23")
+					(reference "R23")
 					(unit 1)
 				)
@@
 		(on_board yes)
 		(dnp no)
-		(property "Reference" "R17"
+		(property "Reference" "R52"
 			(at 168.91 62.23 0)
 			(effects
@@
 			(project "gdp"
 				(path "/95aff260-2720-4733-a81d-a7a2136fdd14/a792f856-eda0-4c7e-9974-4020eb15499f"
-					(reference  "R52")
+					(reference "R52")
 					(unit 1)
 				)
@@
 		(dnp no)
 		(fields_autoplaced yes)
-		(property "Reference" "IC10"
+		(property "Reference" "IC49"
 			(at 204.1241 118.11 0)
 			(effects
@@
 			(project ""
 				(path "/95aff260-2720-4733-a81d-a7a2136fdd14/a792f856-eda0-4c7e-9974-4020eb15499f"
-					(reference  "IC49")
+					(reference "IC49")
 					(unit 1)
 				)
@@
 		(on_board yes)
 		(dnp no)
-		(property "Reference" "R14"
+		(property "Reference" "R36"
 			(at 104.14 62.23 0)
 			(effects
@@
 			(project "gdp"
 				(path "/95aff260-2720-4733-a81d-a7a2136fdd14/a792f856-eda0-4c7e-9974-4020eb15499f"
-					(reference  "R36")
+					(reference "R36")
 					(unit 1)
 				)
@@
 		(on_board yes)
 		(dnp no)
-		(property "Reference" "R16"
+		(property "Reference" "R22"
 			(at 157.48 62.23 0)
 			(effects
@@
 			(project "gdp"
 				(path "/95aff260-2720-4733-a81d-a7a2136fdd14/a792f856-eda0-4c7e-9974-4020eb15499f"
-					(reference  "R22")
+					(reference "R22")
 					(unit 1)
 				)
@@
 		(on_board yes)
 		(dnp no)
-		(property "Reference" "IC7"
+		(property "Reference" "IC23"
 			(at 81.28 109.22 0)
 			(effects
@@
 			(project "gdp"
 				(path "/95aff260-2720-4733-a81d-a7a2136fdd14/a792f856-eda0-4c7e-9974-4020eb15499f"
-					(reference  "IC23")
+					(reference "IC23")
 					(unit 1)
 				)
@@
 		(dnp no)
 		(fields_autoplaced yes)
-		(property "Reference" "IC9"
+		(property "Reference" "IC22"
 			(at 204.1241 72.39 0)
 			(effects
@@
 			(project ""
 				(path "/95aff260-2720-4733-a81d-a7a2136fdd14/a792f856-eda0-4c7e-9974-4020eb15499f"
-					(reference  "IC22")
+					(reference "IC22")
 					(unit 1)
 				)
@@
 		(dnp no)
 		(fields_autoplaced yes)
-		(property "Reference" "IC8"
+		(property "Reference" "IC24"
 			(at 204.1241 26.67 0)
 			(effects
@@
 			(project ""
 				(path "/95aff260-2720-4733-a81d-a7a2136fdd14/a792f856-eda0-4c7e-9974-4020eb15499f"
-					(reference  "IC24")
+					(reference "IC24")
 					(unit 1)
 				)
@@
 		(on_board yes)
 		(dnp no)
-		(property "Reference" "R13"
+		(property "Reference" "R7"
 			(at 44.45 81.28 0)
 			(effects
@@
 			(project "gdp"
 				(path "/95aff260-2720-4733-a81d-a7a2136fdd14/a792f856-eda0-4c7e-9974-4020eb15499f"
-					(reference  "R7")
-					(unit 1)
-				)
+					(reference "R7")
+					(unit 1)
+				)

Commit message: Placing footprints...
Parts:
- R22, R23, R36, R52, R7: footprint Resistor_THT:R_Axial_DIN0207_L6.3mm_D2.5mm_P7.62mm_Horizontal -> Resistor_THT:R_Axial_DIN0207_L6.3mm_D2.5mm_P10.16mm_Horizontal
Changed lines of the file:
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@@
 			)
 		)
-		(property "Footprint" "Resistor_THT:R_Axial_DIN0207_L6.3mm_D2.5mm_P7.62mm_Horizontal"
+		(property "Footprint" "Resistor_THT:R_Axial_DIN0207_L6.3mm_D2.5mm_P10.16mm_Horizontal"
 			(at 141.732 63.5 90)
 			(effects
@@
 			)
 		)
-		(property "Footprint" "Resistor_THT:R_Axial_DIN0207_L6.3mm_D2.5mm_P7.62mm_Horizontal"
+		(property "Footprint" "Resistor_THT:R_Axial_DIN0207_L6.3mm_D2.5mm_P10.16mm_Horizontal"
 			(at 165.862 63.5 90)
 			(effects
@@
 			)
 		)
-		(property "Footprint" "Resistor_THT:R_Axial_DIN0207_L6.3mm_D2.5mm_P7.62mm_Horizontal"
+		(property "Footprint" "Resistor_THT:R_Axial_DIN0207_L6.3mm_D2.5mm_P10.16mm_Horizontal"
 			(at 101.092 63.5 90)
 			(effects
@@
 			)
 		)
-		(property "Footprint" "Resistor_THT:R_Axial_DIN0207_L6.3mm_D2.5mm_P7.62mm_Horizontal"
+		(property "Footprint" "Resistor_THT:R_Axial_DIN0207_L6.3mm_D2.5mm_P10.16mm_Horizontal"
 			(at 154.432 63.5 90)
 			(effects
@@
 			)
 		)
-		(property "Footprint" "Resistor_THT:R_Axial_DIN0207_L6.3mm_D2.5mm_P7.62mm_Horizontal"
+		(property "Footprint" "Resistor_THT:R_Axial_DIN0207_L6.3mm_D2.5mm_P10.16mm_Horizontal"
 			(at 41.402 82.55 90)
 			(effects

Commit message: Maps footprints PCB -> sch
Parts:
- R23: footprint Resistor_THT:R_Axial_DIN0207_L6.3mm_D2.5mm_P10.16mm_Horizontal -> Package_DIP:DIP-20_W7.62mm
- R52, R7: footprint Resistor_THT:R_Axial_DIN0207_L6.3mm_D2.5mm_P10.16mm_Horizontal -> GDP:R_XL
Changed lines of the file:
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@@
 			)
 		)
-		(property "Footprint" "Resistor_THT:R_Axial_DIN0207_L6.3mm_D2.5mm_P10.16mm_Horizontal"
+		(property "Footprint" "Package_DIP:DIP-20_W7.62mm"
 			(at 141.732 63.5 90)
 			(effects
@@
 			)
 		)
-		(property "Footprint" "Resistor_THT:R_Axial_DIN0207_L6.3mm_D2.5mm_P10.16mm_Horizontal"
+		(property "Footprint" "GDP:R_XL"
 			(at 165.862 63.5 90)
 			(effects
@@
 			)
 		)
-		(property "Footprint" "Resistor_THT:R_Axial_DIN0207_L6.3mm_D2.5mm_P10.16mm_Horizontal"
+		(property "Footprint" "GDP:R_XL"
 			(at 41.402 82.55 90)
 			(effects

Commit message: Fixes footprint references in sch
Parts:
- R22, R36: footprint Resistor_THT:R_Axial_DIN0207_L6.3mm_D2.5mm_P10.16mm_Horizontal -> GDP:R_XL
- R23: footprint Package_DIP:DIP-20_W7.62mm -> GDP:R_XL
Changed lines of the file:
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@@
 			)
 		)
-		(property "Footprint" "Package_DIP:DIP-20_W7.62mm"
+		(property "Footprint" "GDP:R_XL"
 			(at 141.732 63.5 90)
 			(effects
@@
 			)
 		)
-		(property "Footprint" "Resistor_THT:R_Axial_DIN0207_L6.3mm_D2.5mm_P10.16mm_Horizontal"
+		(property "Footprint" "GDP:R_XL"
 			(at 101.092 63.5 90)
 			(effects
@@
 			)
 		)
-		(property "Footprint" "Resistor_THT:R_Axial_DIN0207_L6.3mm_D2.5mm_P10.16mm_Horizontal"
+		(property "Footprint" "GDP:R_XL"
 			(at 154.432 63.5 90)
 			(effects

Commit message: Adds more copper
Connections:
- net at IC23.14 (DW): now also IC22.1 (I1)
Changed lines of the file:
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@@
-	(wire
-		(pts
-			(xy 101.6 104.14) (xy 132.08 104.14)
-		)
-		(stroke
-			(width 0)
-			(type default)
-		)
-	)
 	(wire
 		(pts
@@
 		)
 		(stroke
+			(width 0)
+			(type default)
+		)
+	)
+	(wire
+		(pts
+			(xy 100.33 104.14) (xy 132.08 104.14)
+		)
+		(stroke

Commit message: Fixes resistor footprints
Parts:
- R22, R23, R36: footprint GDP:R_XL -> GDP:R_XL_narrow
Changed lines of the file:
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@@
 			)
 		)
-		(property "Footprint" "GDP:R_XL"
+		(property "Footprint" "GDP:R_XL_narrow"
 			(at 141.732 63.5 90)
 			(effects
@@
 			)
 		)
-		(property "Footprint" "GDP:R_XL"
+		(property "Footprint" "GDP:R_XL_narrow"
 			(at 101.092 63.5 90)
 			(effects
@@
 			)
 		)
-		(property "Footprint" "GDP:R_XL"
+		(property "Footprint" "GDP:R_XL_narrow"
 			(at 154.432 63.5 90)
 			(effects
