File: gdp/10.kicad_sch (KiCad schematic)
At the start: 8 parts, among them IC46 2732, IC47 HM6116, IC50 SCB2675

Commit message: Adds pg 13 (WIP)
Connections:
- net ADOUBLE: now also IC50.14 (ADBL)
- net ATTD0: now also IC50.16 (ABLNK)
- net ATTD1: now also IC50.19 (AVL)
- net ATTD4: now also IC50.25 (ARF)
- net ATTD5: now also IC50.18 (AGB)
- net ATTD6: now also IC50.22 (ABB)
- net ATTD7: now also IC50.21 (ARB)
- net CA3: now also IC50.23 (ABF)
- net CA4: now also IC50.17 (AGF)
- net CHD0: now also IC50.39 (D0)
- net CHD1: now also IC50.2 (D1)
- net CHD2: now also IC50.38 (D2)
- net CHD3: now also IC50.3 (D3)
- net CHD4: now also IC50.37 (D4)
- net CHD5: now also IC50.4 (D5)
- net CHD6: now also IC50.36 (D6)
- net CHD7: now also IC50.5 (D7), IC50.6 (D8)

Commit message: Some minor edits
Other:
- company: (none) -> Oddbit Retro
Changed lines of the file:
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@@
   (title_block
     (title "PARTNER GDP")
+    (company "Oddbit Retro")
   )
   (junction (at 129.54 125.095) (diameter 0) (color 0 0 0 0)

Commit message: Adds Sheet 3
Parts:
- gave numbers to parts that had none: 4
- renumbered CK23 to CK2/CK40

Commit message: Adds Sheet 9
Parts:
- CK40: renamed from CK2/CK40; value 10U?? -> 10U
- renumbered R25/R26 to R26, R22/R32 to R32, R24/R33 to R33, R23/R35 to R35
Other:
- title: PARTNER GDP -> PARTNER GDP: CHAR GEN + CMAC
Changed lines of the file:
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@@
 	(paper "A4")
 	(title_block
-		(title "PARTNER GDP")
+		(title "PARTNER GDP: CHAR GEN + CMAC")
 		(company "Oddbit Retro")
+		(comment 1 "NARISAL: MIHA GRČAR")
 	)
 	(junction
@@
 		(on_board yes)
 		(dnp no)
-		(property "Reference" "R24/R33"
-			(at 236.855 129.54 0)
+		(property "Reference" "R33"
+			(at 237.49 129.54 0)
 			(effects
 				(font
@@
 			(project "gdp"
 				(path "/95aff260-2720-4733-a81d-a7a2136fdd14/ba395ee3-de2f-4f14-bf28-234301706162"
-					(reference "R24/R33")
+					(reference "R33")
 					(unit 1)
 				)
@@
 		(on_board yes)
 		(dnp no)
-		(property "Reference" "CK2/CK40"
+		(property "Reference" "CK40"
 			(at 192.405 43.815 0)
 			(effects
@@
 			)
 		)
-		(property "Value" "10U??"
+		(property "Value" "10U"
 			(at 192.405 46.355 0)
 			(effects
@@
 			(project "gdp"
 				(path "/95aff260-2720-4733-a81d-a7a2136fdd14/ba395ee3-de2f-4f14-bf28-234301706162"
-					(reference "CK2/CK40")
+					(reference "CK40")
 					(unit 1)
 				)
@@
 		(on_board yes)
 		(dnp no)
-		(property "Reference" "R22/R32"
+		(property "Reference" "R32"
 			(at 227.965 129.54 0)
 			(effects
@@
 			(project "gdp"
 				(path "/95aff260-2720-4733-a81d-a7a2136fdd14/ba395ee3-de2f-4f14-bf28-234301706162"
-					(reference "R22/R32")
+					(reference "R32")
 					(unit 1)
 				)
@@
 		(on_board yes)
 		(dnp no)
-		(property "Reference" "R25/R26"
+		(property "Reference" "R26"
 			(at 212.09 43.815 0)
 			(effects
@@
 			(project "gdp"
 				(path "/95aff260-2720-4733-a81d-a7a2136fdd14/ba395ee3-de2f-4f14-bf28-234301706162"
-					(reference "R25/R26")
+					(reference "R26")
 					(unit 1)
 				)
@@
 		(on_board yes)
 		(dnp no)
-		(property "Reference" "R23/R35"
+		(property "Reference" "R35"
 			(at 188.595 129.54 0)
 			(effects
@@
 			(project "gdp"
 				(path "/95aff260-2720-4733-a81d-a7a2136fdd14/ba395ee3-de2f-4f14-bf28-234301706162"
-					(reference "R23/R35")
+					(reference "R35")
 					(unit 1)
 				)

Commit message: Initial footprint assignment
Parts:
- CK2: renamed from CK40; footprint (none) -> Capacitor_THT:C_Disc_D4.3mm_W1.9mm_P5.00mm
- IC54: renamed from IC47; footprint Package_DIP:DIP-28_W15.24mm -> Package_DIP:DIP-24_W15.24mm
- IC55: renamed from IC46; footprint Package_DIP:DIP-28_W15.24mm -> Package_DIP:DIP-24_W15.24mm
- R27: renamed from R35; footprint (none) -> Resistor_THT:R_Axial_DIN0207_L6.3mm_D2.5mm_P7.62mm_Horizontal
- R28: renamed from R26; footprint (none) -> Resistor_THT:R_Axial_DIN0207_L6.3mm_D2.5mm_P7.62mm_Horizontal
- R29: renamed from R32; footprint (none) -> Resistor_THT:R_Axial_DIN0207_L6.3mm_D2.5mm_P7.62mm_Horizontal
- R30: renamed from R33; footprint (none) -> Resistor_THT:R_Axial_DIN0207_L6.3mm_D2.5mm_P7.62mm_Horizontal
- renumbered IC50 to IC56
Changed lines of the file:
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@@
 		(on_board yes)
 		(dnp no)
-		(property "Reference" "#PWR052"
+		(property "Reference" "#PWR0136"
 			(at 208.915 64.135 0)
 			(effects
@@
 			(project "gdp"
 				(path "/95aff260-2720-4733-a81d-a7a2136fdd14/ba395ee3-de2f-4f14-bf28-234301706162"
-					(reference "#PWR052")
+					(reference "#PWR0136")
 					(unit 1)
 				)
@@
 		(dnp no)
 		(fields_autoplaced yes)
-		(property "Reference" "#PWR049"
+		(property "Reference" "#PWR0131"
 			(at 109.22 93.345 0)
 			(effects
@@
 			(project "gdp"
 				(path "/95aff260-2720-4733-a81d-a7a2136fdd14/ba395ee3-de2f-4f14-bf28-234301706162"
-					(reference "#PWR049")
+					(reference "#PWR0131")
 					(unit 1)
 				)
@@
 		(dnp no)
 		(fields_autoplaced yes)
-		(property "Reference" "#PWR051"
+		(property "Reference" "#PWR0135"
 			(at 206.375 123.825 0)
 			(effects
@@
 			(project "gdp"
 				(path "/95aff260-2720-4733-a81d-a7a2136fdd14/ba395ee3-de2f-4f14-bf28-234301706162"
-					(reference "#PWR051")
+					(reference "#PWR0135")
 					(unit 1)
 				)
@@
 		(on_board yes)
 		(dnp no)
-		(property "Reference" "#PWR048"
+		(property "Reference" "#PWR0132"
 			(at 109.22 100.965 0)
 			(effects
@@
 			(project "gdp"
 				(path "/95aff260-2720-4733-a81d-a7a2136fdd14/ba395ee3-de2f-4f14-bf28-234301706162"
-					(reference "#PWR048")
+					(reference "#PWR0132")
 					(unit 1)
 				)
@@
 		(on_board yes)
 		(dnp no)
-		(property "Reference" "IC47"
+		(property "Reference" "IC54"
 			(at 109.22 50.8 0)
 			(effects
@@
 			)
 		)
-		(property "Footprint" "Package_DIP:DIP-28_W15.24mm"
+		(property "Footprint" "Package_DIP:DIP-24_W15.24mm"
 			(at 109.22 59.055 0)
 			(effects
@@
 			)
 		)
-		(property "Datasheet" "https://downloads.reactivemicro.com/Electronics/ROM/2764%20EPROM.pdf"
+		(property "Datasheet" "N/A"
 			(at 109.22 59.055 0)
 			(effects
@@
 			)
 		)
-		(property "Description" ""
+		(property "Description" "N/A"
 			(at 109.22 62.865 0)
 			(effects
@@
 			(project "gdp"
 				(path "/95aff260-2720-4733-a81d-a7a2136fdd14/ba395ee3-de2f-4f14-bf28-234301706162"
-					(reference "IC47")
+					(reference "IC54")
 					(unit 1)
 				)
@@
 		(on_board yes)
 		(dnp no)
-		(property "Reference" "R33"
+		(property "Reference" "R30"
 			(at 237.49 129.54 0)
 			(effects
@@
 			)
 		)
-		(property "Footprint" ""
+		(property "Footprint" "Resistor_THT:R_Axial_DIN0207_L6.3mm_D2.5mm_P7.62mm_Horizontal"
 			(at 234.442 130.81 90)
 			(effects
@@
 			)
 		)
-		(property "Datasheet" "~"
+		(property "Datasheet" "N/A"
 			(at 236.22 130.81 0)
 			(effects
@@
 			)
 		)
-		(property "Description" ""
+		(property "Description" "N/A"
 			(at 236.22 130.81 0)
 			(effects
@@
 			(project "gdp"
 				(path "/95aff260-2720-4733-a81d-a7a2136fdd14/ba395ee3-de2f-4f14-bf28-234301706162"
-					(reference "R33")
+					(reference "R30")
 					(unit 1)
 				)
@@
 		(on_board yes)
 		(dnp no)
-		(property "Reference" "CK40"
+		(property "Reference" "CK2"
 			(at 192.405 43.815 0)
 			(effects
@@
 			)
 		)
-		(property "Footprint" ""
+		(property "Footprint" "Capacitor_THT:C_Disc_D4.3mm_W1.9mm_P5.00mm"
 			(at 196.85 45.085 0)
 			(effects
@@
 			)
 		)
-		(property "Datasheet" "~"
+		(property "Datasheet" "N/A"
 			(at 196.85 45.085 0)
 			(effects
@@
 			)
 		)
-		(property "Description" ""
+		(property "Description" "N/A"
 			(at 196.85 45.085 0)
 			(effects
@@
 			(project "gdp"
 				(path "/95aff260-2720-4733-a81d-a7a2136fdd14/ba395ee3-de2f-4f14-bf28-234301706162"
-					(reference "CK40")
+					(reference "CK2")
 					(unit 1)
 				)
@@
 		(on_board yes)
 		(dnp no)
-		(property "Reference" "#PWR055"
+		(property "Reference" "#PWR0137"
 			(at 210.82 45.085 0)
 			(effects
@@
 			(project "gdp"
 				(path "/95aff260-2720-4733-a81d-a7a2136fdd14/ba395ee3-de2f-4f14-bf28-234301706162"
-					(reference "#PWR055")
+					(reference "#PWR0137")
 					(unit 1)
 				)
@@
 		(dnp no)
 		(fields_autoplaced yes)
-		(property "Reference" "#PWR050"
+		(property "Reference" "#PWR0133"
 			(at 109.22 151.765 0)
 			(effects
@@
 			(project "gdp"
 				(path "/95aff260-2720-4733-a81d-a7a2136fdd14/ba395ee3-de2f-4f14-bf28-234301706162"
-					(reference "#PWR050")
+					(reference "#PWR0133")
 					(unit 1)
 				)
@@
 		(on_board yes)
 		(dnp no)
-		(property "Reference" "#PWR054"
+		(property "Reference" "#PWR0139"
 			(at 245.745 138.43 0)
 			(effects
@@
 			(project "gdp"
 				(path "/95aff260-2720-4733-a81d-a7a2136fdd14/ba395ee3-de2f-4f14-bf28-234301706162"
-					(reference "#PWR054")
+					(reference "#PWR0139")
 					(unit 1)
 				)
@@
 		(on_board yes)
 		(dnp no)
-		(property "Reference" "R32"
+		(property "Reference" "R29"
 			(at 227.965 129.54 0)
 			(effects
@@
 			)
 		)
-		(property "Footprint" ""
+		(property "Footprint" "Resistor_THT:R_Axial_DIN0207_L6.3mm_D2.5mm_P7.62mm_Horizontal"
 			(at 224.917 130.81 90)
 			(effects
@@
 			)
 		)
-		(property "Datasheet" "~"
+		(property "Datasheet" "N/A"
 			(at 226.695 130.81 0)
 			(effects
@@
 			)
 		)
-		(property "Description" ""
+		(property "Description" "N/A"
 			(at 226.695 130.81 0)
 			(effects
@@
 			(project "gdp"
 				(path "/95aff260-2720-4733-a81d-a7a2136fdd14/ba395ee3-de2f-4f14-bf28-234301706162"
-					(reference "R32")
+					(reference "R29")
 					(unit 1)
 				)
@@
 		(on_board yes)
 		(dnp no)
-		(property "Reference" "IC46"
+		(property "Reference" "IC55"
 			(at 109.22 109.22 0)
 			(effects
@@
 			)
 		)
-		(property "Footprint" "Package_DIP:DIP-28_W15.24mm"
+		(property "Footprint" "Package_DIP:DIP-24_W15.24mm"
 			(at 109.22 117.475 0)
 			(effects
@@
 			)
 		)
-		(property "Datasheet" "https://downloads.reactivemicro.com/Electronics/ROM/2764%20EPROM.pdf"
+		(property "Datasheet" "N/A"
 			(at 109.22 117.475 0)
 			(effects
@@
 			)
 		)
-		(property "Description" ""
+		(property "Description" "N/A"
 			(at 109.22 121.285 0)
 			(effects
@@
 			(project "gdp"
 				(path "/95aff260-2720-4733-a81d-a7a2136fdd14/ba395ee3-de2f-4f14-bf28-234301706162"
-					(reference "IC46")
+					(reference "IC55")
 					(unit 1)
 				)
@@
 		(on_board yes)
 		(dnp no)
-		(property "Reference" "R26"
+		(property "Reference" "R28"
 			(at 212.09 43.815 0)
 			(effects
@@
 			)
 		)
-		(property "Footprint" ""
+		(property "Footprint" "Resistor_THT:R_Axial_DIN0207_L6.3mm_D2.5mm_P7.62mm_Horizontal"
 			(at 209.042 45.085 90)
 			(effects
@@
 			)
 		)
-		(property "Datasheet" "~"
+		(property "Datasheet" "N/A"
 			(at 210.82 45.085 0)
 			(effects
@@
 			)
 		)
-		(property "Description" ""
+		(property "Description" "N/A"
 			(at 210.82 45.085 0)
 			(effects
@@
 			(project "gdp"
 				(path "/95aff260-2720-4733-a81d-a7a2136fdd14/ba395ee3-de2f-4f14-bf28-234301706162"
-					(reference "R26")
+					(reference "R28")
 					(unit 1)
 				)
@@
 		(on_board yes)
 		(dnp no)
-		(property "Reference" "R35"
+		(property "Reference" "R27"
 			(at 188.595 129.54 0)
 			(effects
@@
 			)
 		)
-		(property "Footprint" ""
+		(property "Footprint" "Resistor_THT:R_Axial_DIN0207_L6.3mm_D2.5mm_P7.62mm_Horizontal"
 			(at 185.547 130.81 90)
 			(effects
@@
 			)
 		)
-		(property "Datasheet" "~"
+		(property "Datasheet" "N/A"
 			(at 187.325 130.81 0)
 			(effects
@@
 			)
 		)
-		(property "Description" ""
+		(property "Description" "N/A"
 			(at 187.325 130.81 0)
 			(effects
@@
 			(project "gdp"
 				(path "/95aff260-2720-4733-a81d-a7a2136fdd14/ba395ee3-de2f-4f14-bf28-234301706162"
-					(reference "R35")
+					(reference "R27")
 					(unit 1)
 				)
@@
 		(on_board yes)
 		(dnp no)
-		(property "Reference" "IC50"
+		(property "Reference" "IC56"
 			(at 206.375 81.915 0)
 			(effects
@@
 			)
 		)
-		(property "Description" ""
+		(property "Description" "N/A"
 			(at 206.375 89.535 0)
 			(effects
@@
 			(project "gdp"
 				(path "/95aff260-2720-4733-a81d-a7a2136fdd14/ba395ee3-de2f-4f14-bf28-234301706162"
-					(reference "IC50")
+					(reference "IC56")
 					(unit 1)
 				)
@@
 		(dnp no)
 		(fields_autoplaced yes)
-		(property "Reference" "#PWR056"
+		(property "Reference" "#PWR0134"
 			(at 196.85 36.195 0)
 			(effects
@@
 			(project "gdp"
 				(path "/95aff260-2720-4733-a81d-a7a2136fdd14/ba395ee3-de2f-4f14-bf28-234301706162"
-					(reference "#PWR056")
+					(reference "#PWR0134")
 					(unit 1)
 				)
@@
 		(dnp no)
 		(fields_autoplaced yes)
-		(property "Reference" "#PWR053"
+		(property "Reference" "#PWR0138"
 			(at 225.425 88.265 0)
 			(effects
@@
 			(project "gdp"
 				(path "/95aff260-2720-4733-a81d-a7a2136fdd14/ba395ee3-de2f-4f14-bf28-234301706162"
-					(reference "#PWR053")
+					(reference "#PWR0138")
 					(unit 1)
 				)
@@
 		(on_board yes)
 		(dnp no)
-		(property "Reference" "#PWR047"
+		(property "Reference" "#PWR0130"
 			(at 109.22 42.545 0)
 			(effects
@@
 			(project "gdp"
 				(path "/95aff260-2720-4733-a81d-a7a2136fdd14/ba395ee3-de2f-4f14-bf28-234301706162"
-					(reference "#PWR047")
-					(unit 1)
-				)
+					(reference "#PWR0130")
+					(unit 1)
+				)
