File: gdp/10.kicad_sch (KiCad schematic)
At the start: 8 parts, among them IC54 HM6116, IC55 2732, IC56 SCB2675

Commit message: Fixes refs
Parts:
- renumbered CK2 to CK40, IC55 to IC46, IC54 to IC47, IC56 to IC50, R28 to R26, R29 to R32, R30 to R33, R27 to R35
Changed lines of the file:
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@@
 		(on_board yes)
 		(dnp no)
-		(property "Reference" "IC54"
+		(property "Reference" "IC47"
 			(at 109.22 50.8 0)
 			(effects
@@
 			(project "gdp"
 				(path "/95aff260-2720-4733-a81d-a7a2136fdd14/ba395ee3-de2f-4f14-bf28-234301706162"
-					(reference  "IC47")
+					(reference "IC47")
 					(unit 1)
 				)
@@
 		(on_board yes)
 		(dnp no)
-		(property "Reference" "R30"
+		(property "Reference" "R33"
 			(at 237.49 129.54 0)
 			(effects
@@
 			(project "gdp"
 				(path "/95aff260-2720-4733-a81d-a7a2136fdd14/ba395ee3-de2f-4f14-bf28-234301706162"
-					(reference  "R33")
+					(reference "R33")
 					(unit 1)
 				)
@@
 		(on_board yes)
 		(dnp no)
-		(property "Reference" "CK2"
+		(property "Reference" "CK40"
 			(at 192.405 43.815 0)
 			(effects
@@
 			(project "gdp"
 				(path "/95aff260-2720-4733-a81d-a7a2136fdd14/ba395ee3-de2f-4f14-bf28-234301706162"
-					(reference  "CK40")
+					(reference "CK40")
 					(unit 1)
 				)
@@
 		(on_board yes)
 		(dnp no)
-		(property "Reference" "R29"
+		(property "Reference" "R32"
 			(at 227.965 129.54 0)
 			(effects
@@
 			(project "gdp"
 				(path "/95aff260-2720-4733-a81d-a7a2136fdd14/ba395ee3-de2f-4f14-bf28-234301706162"
-					(reference  "R32")
+					(reference "R32")
 					(unit 1)
 				)
@@
 		(on_board yes)
 		(dnp no)
-		(property "Reference" "IC55"
+		(property "Reference" "IC46"
 			(at 109.22 109.22 0)
 			(effects
@@
 			(project "gdp"
 				(path "/95aff260-2720-4733-a81d-a7a2136fdd14/ba395ee3-de2f-4f14-bf28-234301706162"
-					(reference  "IC46")
+					(reference "IC46")
 					(unit 1)
 				)
@@
 		(on_board yes)
 		(dnp no)
-		(property "Reference" "R28"
+		(property "Reference" "R26"
 			(at 212.09 43.815 0)
 			(effects
@@
 			(project "gdp"
 				(path "/95aff260-2720-4733-a81d-a7a2136fdd14/ba395ee3-de2f-4f14-bf28-234301706162"
-					(reference  "R26")
+					(reference "R26")
 					(unit 1)
 				)
@@
 		(on_board yes)
 		(dnp no)
-		(property "Reference" "R27"
+		(property "Reference" "R35"
 			(at 188.595 129.54 0)
 			(effects
@@
 			(project "gdp"
 				(path "/95aff260-2720-4733-a81d-a7a2136fdd14/ba395ee3-de2f-4f14-bf28-234301706162"
-					(reference  "R35")
+					(reference "R35")
 					(unit 1)
 				)
@@
 		(on_board yes)
 		(dnp no)
-		(property "Reference" "IC56"
+		(property "Reference" "IC50"
 			(at 206.375 81.915 0)
 			(effects
@@
 			(project "gdp"
 				(path "/95aff260-2720-4733-a81d-a7a2136fdd14/ba395ee3-de2f-4f14-bf28-234301706162"
-					(reference  "IC50")
-					(unit 1)
-				)
+					(reference "IC50")
+					(unit 1)
+				)

Commit message: Placing footprints...
Parts:
- R26, R32, R33, R35: footprint Resistor_THT:R_Axial_DIN0207_L6.3mm_D2.5mm_P7.62mm_Horizontal -> Resistor_THT:R_Axial_DIN0207_L6.3mm_D2.5mm_P10.16mm_Horizontal
Changed lines of the file:
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@@
 			)
 		)
-		(property "Footprint" "Resistor_THT:R_Axial_DIN0207_L6.3mm_D2.5mm_P7.62mm_Horizontal"
+		(property "Footprint" "Resistor_THT:R_Axial_DIN0207_L6.3mm_D2.5mm_P10.16mm_Horizontal"
 			(at 234.442 130.81 90)
 			(effects
@@
 			)
 		)
-		(property "Footprint" "Resistor_THT:R_Axial_DIN0207_L6.3mm_D2.5mm_P7.62mm_Horizontal"
+		(property "Footprint" "Resistor_THT:R_Axial_DIN0207_L6.3mm_D2.5mm_P10.16mm_Horizontal"
 			(at 224.917 130.81 90)
 			(effects
@@
 			)
 		)
-		(property "Footprint" "Resistor_THT:R_Axial_DIN0207_L6.3mm_D2.5mm_P7.62mm_Horizontal"
+		(property "Footprint" "Resistor_THT:R_Axial_DIN0207_L6.3mm_D2.5mm_P10.16mm_Horizontal"
 			(at 209.042 45.085 90)
 			(effects
@@
 			)
 		)
-		(property "Footprint" "Resistor_THT:R_Axial_DIN0207_L6.3mm_D2.5mm_P7.62mm_Horizontal"
+		(property "Footprint" "Resistor_THT:R_Axial_DIN0207_L6.3mm_D2.5mm_P10.16mm_Horizontal"
 			(at 185.547 130.81 90)
 			(effects

Commit message: Maps footprints PCB -> sch
Parts:
- R26: footprint Resistor_THT:R_Axial_DIN0207_L6.3mm_D2.5mm_P10.16mm_Horizontal -> GDP:R_XXL
- R33: footprint Resistor_THT:R_Axial_DIN0207_L6.3mm_D2.5mm_P10.16mm_Horizontal -> GDP:R_L
- R35: footprint Resistor_THT:R_Axial_DIN0207_L6.3mm_D2.5mm_P10.16mm_Horizontal -> GDP:R_XL
Changed lines of the file:
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@@
 			)
 		)
-		(property "Footprint" "Resistor_THT:R_Axial_DIN0207_L6.3mm_D2.5mm_P10.16mm_Horizontal"
+		(property "Footprint" "GDP:R_L"
 			(at 234.442 130.81 90)
 			(effects
@@
 			)
 		)
-		(property "Footprint" "Resistor_THT:R_Axial_DIN0207_L6.3mm_D2.5mm_P10.16mm_Horizontal"
+		(property "Footprint" "GDP:R_XXL"
 			(at 209.042 45.085 90)
 			(effects
@@
 			)
 		)
-		(property "Footprint" "Resistor_THT:R_Axial_DIN0207_L6.3mm_D2.5mm_P10.16mm_Horizontal"
+		(property "Footprint" "GDP:R_XL"
 			(at 185.547 130.81 90)
 			(effects

Commit message: Fixes footprint references in sch
Parts:
- R32: footprint Resistor_THT:R_Axial_DIN0207_L6.3mm_D2.5mm_P10.16mm_Horizontal -> GDP:R_L
Changed lines of the file:
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@@
 			)
 		)
-		(property "Footprint" "Resistor_THT:R_Axial_DIN0207_L6.3mm_D2.5mm_P10.16mm_Horizontal"
+		(property "Footprint" "GDP:R_L"
 			(at 224.917 130.81 90)
 			(effects

Commit message: Fixes labels
Connections:
- net TTLY1 renamed TTLV1
- net TTLY2 renamed TTLV2
- net YIDGP1 renamed VIDGP1
- net YIDGP2 renamed VIDGP2
Changed lines of the file:
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@@
 		)
 	)
-	(global_label "YIDGP2"
+	(global_label "VIDGP2"
 		(shape output)
 		(at 238.125 71.755 0)
@@
 		)
 	)
-	(global_label "YIDGP1"
+	(global_label "VIDGP1"
 		(shape output)
 		(at 238.125 69.215 0)
@@
 		)
 	)
-	(global_label "TTLY2"
+	(global_label "TTLV2"
 		(shape output)
 		(at 238.125 64.135 0)
@@
 		)
 	)
-	(global_label "TTLY1"
+	(global_label "TTLV1"
 		(shape output)
 		(at 238.125 66.675 0)

Commit message: Adds decoupling capacitors
Parts:
- CK40: value 10U -> U10
Changed lines of the file:
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@@
 			)
 		)
-		(property "Value" "10U"
+		(property "Value" "U10"
 			(at 192.405 46.355 0)
 			(effects

Commit message: Fixes GND issue (R32)
Connections:
- net +5V: no longer R32.2
- net GNDD: now also R32.2
Other:
- moved on the sheet: CK40, IC46, IC47, IC50, R26, R32, R35
