File: gdp/11.kicad_sch (KiCad schematic)
At the start: 0 parts

Commit message: Adds Sheet 11
Parts:
- added IC15B: 74LS367, symbol 74xx_IEEE:74LS244
- added IC26, IC27: 74LS374, symbol 74xx:74LS374
- added IC33, IC34: 74LS244, symbol 74xx_IEEE:74LS244
Connections:
- new net +5V: IC15B.20 (VCC), IC26.20 (VCC), IC27.20 (VCC), IC33.20 (VCC), IC33.20 (VCC), IC34.20 (VCC), IC34.20 (VCC)
- new net ADOUBLE: IC26.2 (O0)
- new net ASCD0: IC27.3 (D0), IC34.11 (I0)
- new net ASCD1: IC27.4 (D1), IC34.13 (I1)
- new net ASCD2: IC27.7 (D2), IC34.15 (I2)
- new net ASCD3: IC27.8 (D3), IC34.17 (I3)
- new net ASCD4: IC27.13 (D4), IC33.11 (I0)
- new net ASCD5: IC27.14 (D5), IC33.13 (I1)
- new net ASCD6: IC27.17 (D6), IC33.15 (I2)
- new net ASCD7: IC27.18 (D7), IC33.17 (I3)
- new net CCLK+: IC27.11 (Cp)
- new net CH0: IC26.12 (O4)
- new net CH1: IC26.15 (O5)
- new net CH10: IC27.16 (O6), IC33.14 (O2)
- new net CH11: IC27.19 (O7), IC33.12 (O3)
- new net CH2: IC26.16 (O6)
- new net CH3: IC26.19 (O7)
- new net CH4: IC27.2 (O0)
- new net CH5: IC27.5 (O1)
- new net CH6: IC27.6 (O2)
- new net CH7: IC27.9 (O3)
- new net CH8: IC27.12 (O4), IC33.18 (O0)
- new net CH9: IC27.15 (O5), IC33.16 (O1)
- new net CHD0: IC15B.3, IC34.9 (O0)
- new net CHD1: IC15B.5, IC34.7 (O1)
- new net CHD2: IC15B.7, IC34.5 (O2)
- new net CHD3: IC15B.9, IC34.3 (O3)
- new net CHD4: IC33.9 (O0), IC34.18 (O0)
- new net CHD5: IC33.7 (O1), IC34.16 (O1)
- new net CHD6: IC33.5 (O2), IC34.14 (O2)
- new net CHD7: IC33.3 (O3), IC34.12 (O3)
- new net DA0: IC15B.2
- new net DA1: IC15B.4, IC26.7 (D2)
- new net DA10: IC33.6 (I2)
- new net DA11: IC33.8 (I3)
- new net DA13: IC26.4 (D1)
- new net DA2: IC15B.6, IC26.8 (D3)
- new net DA3: IC15B.10
- new net DA4: IC26.13 (D4), IC34.2 (I0)
- new net DA5: IC26.14 (D5), IC34.4 (I1)
- new net DA6: IC26.17 (D6), IC34.6 (I2)
- new net DA7: IC26.18 (D7), IC34.8 (I3)
- new net DA8: IC33.2 (I0)
- new net DA9: IC26.3 (D0), IC33.4 (I1)
- new net GNDD: IC15B.10, IC26.10 (GND), IC27.10 (GND), IC33.10 (GND), IC33.10 (GND), IC34.10 (GND), IC34.10 (GND)
- new net ~{BLNK}: IC26.11 (Cp)
- new net ~{DSPEN}: IC26.1 (OE), IC27.1 (OE)
- new net ~{LDEN}: IC15B.1, IC33.1 (~{OE}), IC33.19 (~{OE}), IC34.1 (~{OE}), IC34.19 (~{OE})
- new net ~{RESTRICT}: IC26.5 (O1)
- no-connect marks 0 -> 2
Other:
- company: (none) -> Oddbit Retro
- title: (none) -> PARTNER GDP: CHAR DATA

Commit message: Fixes IC15
Parts:
- removed IC15B: 74LS367, symbol 74xx_IEEE:74LS244
- added IC15: 74LS367, symbol 74xx_IEEE:74LS367
Connections:
- net +5V: now also IC15.20 (VCC)
- net CHD0: now also IC15.3 (1Y1)
- net CHD1: now also IC15.5 (1Y2)
- net CHD2: now also IC15.7 (1Y3)
- net CHD3: now also IC15.9 (1Y4)
- net DA0: now also IC15.2 (1I1)
- net DA1: now also IC15.4 (1I2)
- net DA2: now also IC15.6 (1I3)
- net DA3: now also IC15.10 (1I4)
- net GNDD: now also IC15.10 (1I4)
- net ~{LDEN}: now also IC15.1 (~{1G})
Changed lines of the file:
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@@
-	)
-	(symbol
-		(lib_name "74LS244_3")
-		(lib_id "74xx_IEEE:74LS244")
-		(at 99.06 91.44 0)
-		(unit 1)
-		(exclude_from_sim no)
-		(in_bom yes)
-		(on_board yes)
-		(dnp no)
-		(fields_autoplaced yes)
-		(property "Reference" "IC15B"
-			(at 99.06 86.614 0)
-			(effects
-				(font
-					(size 1.27 1.27)
-				)
-			)
-		)
-		(property "Value" "74LS367"
-			(at 99.06 89.154 0)
-			(effects
-				(font
-					(size 1.27 1.27)
-				)
-			)
-		)
-		(property "Footprint" ""
-			(at 99.06 91.44 0)
-			(effects
-				(font
-					(size 1.27 1.27)
-				)
-				(hide yes)
-			)
-		)
-		(property "Datasheet" ""
-			(at 44.196 78.994 0)
-			(effects
-				(font
-					(size 1.27 1.27)
-				)
-				(hide yes)
-			)
-		)
-		(property "Description" ""
-			(at 33.02 81.28 0)
-			(effects
-				(font
-					(size 1.27 1.27)
-				)
-				(hide yes)
-			)
-		)
-		(pin "10"
-		)
-		(pin "7"
-		)
-		(pin "5"
-		)
-		(pin "6"
-		)
-		(pin "2"
-		)
-		(pin "20"
-		)
-		(pin "10"
-		)
-		(pin "1"
-		)
-		(pin "3"
-		)
-		(pin "9"
-		)
-		(pin "4"
-		)
-		(instances
-			(project "gdp"
-				(path "/95aff260-2720-4733-a81d-a7a2136fdd14/d6b86f16-da3f-4420-ad10-a48d1b11a79a"
-					(reference "IC15B")
-					(unit 1)
-				)
-			)
-		)
 	)
 	(symbol
@@
 				)
 			)
+		)
+	)
+	(symbol
+		(lib_id "74xx_IEEE:74LS367")
+		(at 99.06 91.44 0)
+		(unit 2)
+		(exclude_from_sim no)
+		(in_bom yes)
+		(on_board yes)
+		(dnp no)
+		(property "Reference" "IC15"
+			(at 98.806 87.63 0)
+			(effects
+				(font
+					(size 1.27 1.27)
+				)
+			)
+		)
+		(property "Value" "74LS367"
+			(at 98.806 89.535 0)
+			(effects
+				(font
+					(size 1.27 1.27)
+				)
+			)
+		)
+		(property "Footprint" ""
+			(at 148.59 110.49 0)
+			(effects
+				(font
+					(size 1.27 1.27)
+				)
+				(hide yes)
+			)
+		)
+		(property "Datasheet" ""
+			(at 148.59 110.49 0)
+			(effects
+				(font
+					(size 1.27 1.27)
+				)
+				(hide yes)
+			)
+		)
+		(property "Description" ""
+			(at 98.806 88.9 0)
+			(effects
+				(font
+					(size 1.27 1.27)
+				)
+				(hide yes)
+			)
+		)
+		(pin "16"
+		)
+		(pin "8"
+		)
+		(pin "11"
+		)
+		(pin "12"
+		)
+		(pin "13"
+		)
+		(pin "14"
+		)
+		(pin "15"
+		)
+		(pin "10"
+		)
+		(pin "20"
+		)
+		(pin "1"
+		)
+		(pin "10"
+		)
+		(pin "2"
+		)
+		(pin "3"
+		)
+		(pin "16"
+		)
+		(pin "14"
+		)
+		(pin "4"
+		)
+		(pin "11"
+		)
+		(pin "8"
+		)
+		(pin "15"
+		)
+		(pin "7"
+		)
+		(pin "5"
+		)
+		(pin "13"
+		)
+		(pin "9"
+		)
+		(pin "12"
+		)
+		(pin "6"
+		)
+		(instances
+			(project "gdp"
+				(path "/95aff260-2720-4733-a81d-a7a2136fdd14/d6b86f16-da3f-4420-ad10-a48d1b11a79a"
+					(reference "IC15")
+					(unit 2)
+				)
+			)

Commit message: Initial footprint assignment
Parts:
- IC42: renamed from IC15; footprint (none) -> Package_DIP:DIP-16_W7.62mm
- IC57: renamed from IC26; footprint (none) -> Package_DIP:DIP-20_W7.62mm
- IC58: renamed from IC34; footprint (none) -> Package_DIP:DIP-20_W7.62mm
- IC59: renamed from IC33; footprint (none) -> Package_DIP:DIP-20_W7.62mm
- IC60: renamed from IC27; footprint (none) -> Package_DIP:DIP-20_W7.62mm

Commit message: Several fixes
Connections:
- net +5V: now also IC42.16 (VCC); no longer IC42.20 (VCC)
- net GNDD: now also IC42.8 (GND); no longer IC42.10 (1I4)
Changed lines of the file:
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@@
 		(pin "15"
 		)
-		(pin "10"
+		(pin "8"
 		)
-		(pin "20"
+		(pin "16"
 		)
 		(pin "1"
