File: gdp/11.kicad_sch (KiCad schematic)
At the start: 5 parts, among them IC42 74LS367, IC57 74LS374, IC58 74LS244, IC59 74LS244, IC60 74LS374

Commit message: Fixes refs
Parts:
- renumbered IC42 to IC15, IC57 to IC26, IC60 to IC27, IC59 to IC33, IC58 to IC33, IC59 to IC34, IC58 to IC34
Changed lines of the file:
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@@
 		(dnp no)
 		(fields_autoplaced yes)
-		(property "Reference" "IC59"
+		(property "Reference" "IC34"
 			(at 99.06 169.164 0)
 			(do_not_autoplace yes)
@@
 			(project "gdp"
 				(path "/95aff260-2720-4733-a81d-a7a2136fdd14/d6b86f16-da3f-4420-ad10-a48d1b11a79a"
-					(reference  "IC33")
+					(reference "IC34")
 					(unit 1)
 				)
@@
 		(dnp no)
 		(fields_autoplaced yes)
-		(property "Reference" "IC59"
+		(property "Reference" "IC33"
 			(at 208.28 125.984 0)
 			(effects
@@
 			(project "gdp"
 				(path "/95aff260-2720-4733-a81d-a7a2136fdd14/d6b86f16-da3f-4420-ad10-a48d1b11a79a"
-					(reference  "IC33")
+					(reference "IC33")
 					(unit 2)
 				)
@@
 		(dnp no)
 		(fields_autoplaced yes)
-		(property "Reference" "IC60"
+		(property "Reference" "IC27"
 			(at 210.4741 21.59 0)
 			(effects
@@
 			(project ""
 				(path "/95aff260-2720-4733-a81d-a7a2136fdd14/d6b86f16-da3f-4420-ad10-a48d1b11a79a"
-					(reference  "IC27")
+					(reference "IC27")
 					(unit 1)
 				)
@@
 		(dnp no)
 		(fields_autoplaced yes)
-		(property "Reference" "IC58"
+		(property "Reference" "IC33"
 			(at 99.06 129.794 0)
 			(do_not_autoplace yes)
@@
 			(project "gdp"
 				(path "/95aff260-2720-4733-a81d-a7a2136fdd14/d6b86f16-da3f-4420-ad10-a48d1b11a79a"
-					(reference  "IC34")
+					(reference "IC33")
 					(unit 1)
 				)
@@
 		(on_board yes)
 		(dnp no)
-		(property "Reference" "IC42"
+		(property "Reference" "IC15"
 			(at 98.806 87.63 0)
 			(effects
@@
 			(project "gdp"
 				(path "/95aff260-2720-4733-a81d-a7a2136fdd14/d6b86f16-da3f-4420-ad10-a48d1b11a79a"
-					(reference  "IC15")
+					(reference "IC15")
 					(unit 2)
 				)
@@
 		(dnp no)
 		(fields_autoplaced yes)
-		(property "Reference" "IC58"
+		(property "Reference" "IC34"
 			(at 208.28 86.614 0)
 			(effects
@@
 			(project "gdp"
 				(path "/95aff260-2720-4733-a81d-a7a2136fdd14/d6b86f16-da3f-4420-ad10-a48d1b11a79a"
-					(reference  "IC34")
+					(reference "IC34")
 					(unit 2)
 				)
@@
 		(dnp no)
 		(fields_autoplaced yes)
-		(property "Reference" "IC57"
+		(property "Reference" "IC26"
 			(at 101.2541 21.59 0)
 			(effects
@@
 			(project "gdp"
 				(path "/95aff260-2720-4733-a81d-a7a2136fdd14/d6b86f16-da3f-4420-ad10-a48d1b11a79a"
-					(reference  "IC26")
-					(unit 1)
-				)
+					(reference "IC26")
+					(unit 1)
+				)

Commit message: Bug fix
Connections:
- net CH0: now also IC15.3 (1Y1)
- net CH1: now also IC15.5 (1Y2)
- net CH2: now also IC15.7 (1Y3)
- net CH3: now also IC15.9 (1Y4)
- net CH4: now also IC33.18 (O0)
- net CH5: now also IC33.16 (O1)
- net CH6: now also IC33.14 (O2)
- net CH7: now also IC33.12 (O3)
- net CHD0: no longer IC15.3 (1Y1)
- net CHD1: no longer IC15.5 (1Y2)
- net CHD2: no longer IC15.7 (1Y3)
- net CHD3: no longer IC15.9 (1Y4)
- net CHD4: no longer IC33.18 (O0)
- net CHD5: no longer IC33.16 (O1)
- net CHD6: no longer IC33.14 (O2)
- net CHD7: no longer IC33.12 (O3)
