File: gdp/12.kicad_sch (KiCad schematic)
At the start: 0 parts

Commit message: Adds Sheet 12
Parts:
- added CK3: 10U, symbol Device:C_Small
- added CK5: 2N2, symbol Device:C_Small
- added IC1: 74LS74, symbol 74xx:74LS74
- added IC12: PAL16R4, symbol Logic_Programmable:PAL16L8
- added IC51: 74LS14, symbol 74xx:74LS14
- added IC64: 74LS123, symbol 74xx:74LS123
- added IC66: 74S00, symbol 74xx:74LS00
- added IC71: 74LS04, symbol 74xx:74LS04
- added R2, R48: 1K0, symbol Device:R
- added R27: 220R, symbol Device:R
- added SH10, SH11, SH13, SH14, SH4, SH5, SH_4, SH_5: SCHALT, symbol Switch:SW_DPST_x2
Connections:
- new net: IC12.9 (I8), R2.1
- new net: IC1.11 (C), SH4.2 (B), SH5.2 (B)
- new net: IC64.10 (B), SH13.2 (B), SH14.2 (B)
- new net: CK3.1, IC51.1, R27.1
- new net: CK5.1, IC64.6 (Cext)
- new net: CK5.2, IC64.7 (RCext), R48.1
- new net +5V: IC1.10 (~{S}), IC1.12 (D), IC12.20 (VCC), IC64.11 (Clr), R2.2, R48.2, SH_4.1 (A)
- new net AHSYNC: SH5.1 (A)
- new net ATTD2: IC12.8 (I7)
- new net AVSCS: SH10.1 (A), SH14.1 (A)
- new net BLANK: IC66.2, IC71.3
- new net CCLK+: IC12.1 (CLK), IC71.6
- new net CLKEN: IC1.8 (~{Q})
- new net CURSOR: IC66.1
- new net DA11: IC12.3 (I2)
- new net DA12: IC12.4 (I3)
- new net DA13: IC12.5 (I4)
- new net GDPSYNC: SH11.1 (A)
- new net GNDD: CK3.2, IC12.10 (GND), IC12.11 (~{OE}), IC64.9 (A), SH4.1 (A)
- new net HCSYNC+: IC51.5, SH10.2 (B), SH11.2 (B)
- new net LROW: IC64.5 (Q)
- new net MASTER: SH_4.2 (B), SH_5.2 (B)
- new net VSYNC+: IC51.2, IC51.3, SH13.1 (A), SH_5.1 (A)
- new net ~{AVDINT}: IC12.15 (Q3)
- new net ~{AVINT}: IC12.2 (I1)
- new net ~{BCE}: IC12.6 (I5)
- new net ~{BLNK}: IC71.4
- new net ~{CCLK}: IC71.5
- new net ~{CRAMEN}: IC12.16 (Q2)
- new net ~{CRAM}: IC12.13 (IO3)
- new net ~{CRH}: IC12.19 (IO1)
- new net ~{CRL}: IC12.18 (IO2)
- new net ~{CROM}: IC12.17 (Q1)
- new net ~{DSPEN}: IC71.2
- new net ~{HCSYNC}: IC1.13 (~{R}), IC51.6, R27.2
- new net ~{LDEN}: IC12.12 (IO4), IC71.1
- new net ~{ROW}: IC66.3
- new net ~{VSYNC}: IC51.4
- new net ~{WDB}: IC12.7 (I6)
- no-connect marks 0 -> 3
Other:
- company: (none) -> Oddbit Retro
- title: (none) -> PARTNER GDP: SYNC + CONTROL

Commit message: Fixes (component refs...)
Parts:
- R17: renamed from R2; value 1K0 -> 2K2
- renumbered CK5 to CK55
Changed lines of the file:
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@@
 		(on_board yes)
 		(dnp no)
-		(property "Reference" "R2"
+		(property "Reference" "R17"
 			(at 95.25 163.83 0)
 			(effects
@@
 			)
 		)
-		(property "Value" "1K0"
+		(property "Value" "2K2"
 			(at 95.25 166.37 0)
 			(effects
@@
 			(project "gdp"
 				(path "/95aff260-2720-4733-a81d-a7a2136fdd14/7e43dd6e-b5cb-462f-9bfd-3d0ee9fd8751"
-					(reference "R2")
+					(reference "R17")
 					(unit 1)
 				)
@@
 		(on_board yes)
 		(dnp no)
-		(property "Reference" "CK5"
+		(property "Reference" "CK55"
 			(at 190.5 112.395 0)
 			(effects
@@
 			(project "gdp"
 				(path "/95aff260-2720-4733-a81d-a7a2136fdd14/7e43dd6e-b5cb-462f-9bfd-3d0ee9fd8751"
-					(reference "CK5")
-					(unit 1)
-				)
+					(reference "CK55")
+					(unit 1)
+				)

Commit message: Adds Sheet 14 (WIP)
Parts:
- renumbered CK3 to CK50
Changed lines of the file:
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@@
 		(on_board yes)
 		(dnp no)
-		(property "Reference" "CK3"
+		(property "Reference" "CK50"
 			(at 154.305 55.88 0)
 			(effects
@@
 			(project "gdp"
 				(path "/95aff260-2720-4733-a81d-a7a2136fdd14/7e43dd6e-b5cb-462f-9bfd-3d0ee9fd8751"
-					(reference "CK3")
+					(reference "CK50")
 					(unit 1)
 				)

Commit message: Initial footprint assignment
Parts:
- CK3: renamed from CK50; footprint (none) -> Capacitor_THT:C_Disc_D4.3mm_W1.9mm_P5.00mm
- CK4: renamed from CK55; footprint (none) -> Capacitor_THT:C_Disc_D4.3mm_W1.9mm_P5.00mm
- IC41: renamed from IC1; footprint (none) -> Package_DIP:DIP-14_W7.62mm
- IC61: renamed from IC71; footprint (none) -> Package_DIP:DIP-14_W7.62mm
- IC62: renamed from IC12; footprint (none) -> Package_DIP:DIP-20_W7.62mm
- IC63: renamed from IC51; footprint (none) -> Package_DIP:DIP-14_W7.62mm
- IC64: renamed from IC66; footprint (none) -> Package_DIP:DIP-14_W7.62mm
- IC65: renamed from IC64; footprint (none) -> Package_DIP:DIP-16_W7.62mm
- R31: renamed from R17; footprint (none) -> Resistor_THT:R_Axial_DIN0207_L6.3mm_D2.5mm_P7.62mm_Horizontal
- R32: renamed from R27; footprint (none) -> Resistor_THT:R_Axial_DIN0207_L6.3mm_D2.5mm_P7.62mm_Horizontal
- R33: renamed from R48; footprint (none) -> Resistor_THT:R_Axial_DIN0207_L6.3mm_D2.5mm_P7.62mm_Horizontal
- SH10: renamed from SH5; footprint (none) -> Connector_PinHeader_2.54mm:PinHeader_1x02_P2.54mm_Vertical
- SH11: renamed from SH13; footprint (none) -> Connector_PinHeader_2.54mm:PinHeader_1x02_P2.54mm_Vertical
- SH12: renamed from SH14; footprint (none) -> Connector_PinHeader_2.54mm:PinHeader_1x02_P2.54mm_Vertical
- SH7: renamed from SH11; footprint (none) -> Connector_PinHeader_2.54mm:PinHeader_1x02_P2.54mm_Vertical
- SH8: renamed from SH10; footprint (none) -> Connector_PinHeader_2.54mm:PinHeader_1x02_P2.54mm_Vertical
- SH9: renamed from SH4; footprint (none) -> Connector_PinHeader_2.54mm:PinHeader_1x02_P2.54mm_Vertical
- SH_1: renamed from SH_4; footprint (none) -> Connector_PinHeader_2.54mm:PinHeader_1x02_P2.54mm_Vertical
- SH_2: renamed from SH_5; footprint (none) -> Connector_PinHeader_2.54mm:PinHeader_1x02_P2.54mm_Vertical

Commit message: Results of some measurements
Changed lines of the file:
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@@
 	(wire
 		(pts
-			(xy 87.63 167.64) (xy 87.63 171.45)
+			(xy 87.63 167.64) (xy 87.63 168.91)
 		)
 		(stroke
@@
 	(wire
 		(pts
-			(xy 93.98 168.91) (xy 93.98 171.45)
-		)
-		(stroke
-			(width 0)
-			(type default)
-		)
-	)
-	(wire
-		(pts
-			(xy 93.98 171.45) (xy 87.63 171.45)
-		)
-		(stroke
+			(xy 93.98 168.91) (xy 87.63 168.91)
+		)
+		(stroke

Commit message: Adds VCC/GND
Parts:
- added unit 7 of IC61
- added unit 7 of IC63
- added unit 5 of IC64
- added unit 3 of IC65
- added IC66: 74LS74, Package_DIP:DIP-14_W7.62mm, symbol 74xx:74LS74
- renumbered IC41 to IC38
Connections:
- net +5V: now also IC61.14 (VCC), IC63.14 (VCC), IC64.14 (VCC), IC65.16 (VCC), IC66.14 (VCC)
- net GNDD: now also IC61.7 (GND), IC63.7 (GND), IC64.7 (GND), IC65.8 (GND), IC66.7 (GND)
