File: gdp/12.kicad_sch (KiCad schematic)
At the start: 20 parts, among them IC38 74LS74, IC61 74LS04, IC62 PAL16R4, IC63 74LS14, IC64 74S00, IC65 74LS123, IC66 74LS74

Commit message: Fixes refs
Parts:
- renumbered CK3 to CK50, CK4 to CK55, IC38 to IC1, IC62 to IC12, IC63 to IC51, IC65 to IC64, IC64 to IC66, IC61 to IC71, IC66 to IC72, R31 to R17, R32 to R27, R33 to R48, SH8 to SH10, SH7 to SH11, SH11 to SH13, SH12 to SH14, SH9 to SH4, SH10 to SH5, SH_1 to SH_4, SH_2 to SH_5
Changed lines of the file:
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@@
 		(dnp no)
 		(fields_autoplaced yes)
-		(property "Reference" "IC63"
+		(property "Reference" "IC51"
 			(at 179.07 48.26 0)
 			(effects
@@
 			(project "gdp"
 				(path "/95aff260-2720-4733-a81d-a7a2136fdd14/7e43dd6e-b5cb-462f-9bfd-3d0ee9fd8751"
-					(reference  "IC51")
+					(reference "IC51")
 					(unit 2)
 				)
@@
 		(on_board yes)
 		(dnp no)
-		(property "Reference" "R31"
+		(property "Reference" "R17"
 			(at 95.25 163.83 0)
 			(effects
@@
 			(project "gdp"
 				(path "/95aff260-2720-4733-a81d-a7a2136fdd14/7e43dd6e-b5cb-462f-9bfd-3d0ee9fd8751"
-					(reference  "R17")
+					(reference "R17")
 					(unit 1)
 				)
@@
 		(dnp no)
 		(fields_autoplaced yes)
-		(property "Reference" "IC61"
+		(property "Reference" "IC71"
 			(at 111.76 109.22 0)
 			(effects
@@
 			(project "gdp"
 				(path "/95aff260-2720-4733-a81d-a7a2136fdd14/7e43dd6e-b5cb-462f-9bfd-3d0ee9fd8751"
-					(reference  "IC71")
+					(reference "IC71")
 					(unit 3)
 				)
@@
 		(on_board yes)
 		(dnp no)
-		(property "Reference" "IC66"
+		(property "Reference" "IC72"
 			(at 252.73 52.07 0)
 			(effects
@@
 			(project "gdp"
 				(path "/95aff260-2720-4733-a81d-a7a2136fdd14/7e43dd6e-b5cb-462f-9bfd-3d0ee9fd8751"
-					(reference  "IC72")
+					(reference "IC72")
 					(unit 3)
 				)
@@
 		(on_board yes)
 		(dnp no)
-		(property "Reference" "SH10"
+		(property "Reference" "SH5"
 			(at 111.76 81.28 0)
 			(effects
@@
 			(project "gdp"
 				(path "/95aff260-2720-4733-a81d-a7a2136fdd14/7e43dd6e-b5cb-462f-9bfd-3d0ee9fd8751"
-					(reference  "SH5")
+					(reference "SH5")
 					(unit 1)
 				)
@@
 		(on_board yes)
 		(dnp no)
-		(property "Reference" "IC65"
+		(property "Reference" "IC64"
 			(at 252.73 123.19 0)
 			(effects
@@
 			(project "gdp"
 				(path "/95aff260-2720-4733-a81d-a7a2136fdd14/7e43dd6e-b5cb-462f-9bfd-3d0ee9fd8751"
-					(reference  "IC64")
+					(reference "IC64")
 					(unit 3)
 				)
@@
 		(dnp no)
 		(fields_autoplaced yes)
-		(property "Reference" "IC63"
+		(property "Reference" "IC51"
 			(at 124.46 36.83 0)
 			(effects
@@
 			(project ""
 				(path "/95aff260-2720-4733-a81d-a7a2136fdd14/7e43dd6e-b5cb-462f-9bfd-3d0ee9fd8751"
-					(reference  "IC51")
+					(reference "IC51")
 					(unit 3)
 				)
@@
 		(dnp no)
 		(fields_autoplaced yes)
-		(property "Reference" "IC61"
+		(property "Reference" "IC71"
 			(at 111.76 92.71 0)
 			(effects
@@
 			(project ""
 				(path "/95aff260-2720-4733-a81d-a7a2136fdd14/7e43dd6e-b5cb-462f-9bfd-3d0ee9fd8751"
-					(reference  "IC71")
+					(reference "IC71")
 					(unit 2)
 				)
@@
 		(on_board yes)
 		(dnp no)
-		(property "Reference" "IC61"
+		(property "Reference" "IC71"
 			(at 264.16 123.19 0)
 			(effects
@@
 			(project "gdp"
 				(path "/95aff260-2720-4733-a81d-a7a2136fdd14/7e43dd6e-b5cb-462f-9bfd-3d0ee9fd8751"
-					(reference  "IC71")
+					(reference "IC71")
 					(unit 7)
 				)
@@
 		(on_board yes)
 		(dnp no)
-		(property "Reference" "SH12"
+		(property "Reference" "SH14"
 			(at 177.8 100.33 0)
 			(effects
@@
 			(project "gdp"
 				(path "/95aff260-2720-4733-a81d-a7a2136fdd14/7e43dd6e-b5cb-462f-9bfd-3d0ee9fd8751"
-					(reference  "SH14")
+					(reference "SH14")
 					(unit 1)
 				)
@@
 		(dnp no)
 		(fields_autoplaced yes)
-		(property "Reference" "IC61"
+		(property "Reference" "IC71"
 			(at 137.16 124.46 0)
 			(effects
@@
 			(project "gdp"
 				(path "/95aff260-2720-4733-a81d-a7a2136fdd14/7e43dd6e-b5cb-462f-9bfd-3d0ee9fd8751"
-					(reference  "IC71")
+					(reference "IC71")
 					(unit 1)
 				)
@@
 		(on_board yes)
 		(dnp no)
-		(property "Reference" "SH11"
+		(property "Reference" "SH13"
 			(at 177.8 91.44 0)
 			(effects
@@
 			(project "gdp"
 				(path "/95aff260-2720-4733-a81d-a7a2136fdd14/7e43dd6e-b5cb-462f-9bfd-3d0ee9fd8751"
-					(reference  "SH13")
+					(reference "SH13")
 					(unit 1)
 				)
@@
 		(on_board yes)
 		(dnp no)
-		(property "Reference" "SH9"
+		(property "Reference" "SH4"
 			(at 111.76 71.12 0)
 			(effects
@@
 			(project "gdp"
 				(path "/95aff260-2720-4733-a81d-a7a2136fdd14/7e43dd6e-b5cb-462f-9bfd-3d0ee9fd8751"
-					(reference  "SH4")
+					(reference "SH4")
 					(unit 1)
 				)
@@
 		(on_board yes)
 		(dnp no)
-		(property "Reference" "CK3"
+		(property "Reference" "CK50"
 			(at 154.305 55.88 0)
 			(effects
@@
 			(project "gdp"
 				(path "/95aff260-2720-4733-a81d-a7a2136fdd14/7e43dd6e-b5cb-462f-9bfd-3d0ee9fd8751"
-					(reference  "CK50")
+					(reference "CK50")
 					(unit 1)
 				)
@@
 		(dnp no)
 		(fields_autoplaced yes)
-		(property "Reference" "IC64"
+		(property "Reference" "IC66"
 			(at 208.2717 134.62 0)
 			(effects
@@
 			(project ""
 				(path "/95aff260-2720-4733-a81d-a7a2136fdd14/7e43dd6e-b5cb-462f-9bfd-3d0ee9fd8751"
-					(reference  "IC66")
+					(reference "IC66")
 					(unit 1)
 				)
@@
 		(on_board yes)
 		(dnp no)
-		(property "Reference" "SH_1"
+		(property "Reference" "SH_4"
 			(at 180.34 31.75 0)
 			(effects
@@
 			(project "gdp"
 				(path "/95aff260-2720-4733-a81d-a7a2136fdd14/7e43dd6e-b5cb-462f-9bfd-3d0ee9fd8751"
-					(reference  "SH_4")
+					(reference "SH_4")
 					(unit 1)
 				)
@@
 		(on_board yes)
 		(dnp no)
-		(property "Reference" "R32"
+		(property "Reference" "R27"
 			(at 143.51 46.99 0)
 			(effects
@@
 			(project "gdp"
 				(path "/95aff260-2720-4733-a81d-a7a2136fdd14/7e43dd6e-b5cb-462f-9bfd-3d0ee9fd8751"
-					(reference  "R27")
+					(reference "R27")
 					(unit 1)
 				)
@@
 		(on_board yes)
 		(dnp no)
-		(property "Reference" "SH8"
+		(property "Reference" "SH10"
 			(at 102.87 48.26 0)
 			(effects
@@
 			(project "gdp"
 				(path "/95aff260-2720-4733-a81d-a7a2136fdd14/7e43dd6e-b5cb-462f-9bfd-3d0ee9fd8751"
-					(reference  "SH10")
+					(reference "SH10")
 					(unit 1)
 				)
@@
 		(on_board yes)
 		(dnp no)
-		(property "Reference" "CK4"
+		(property "Reference" "CK55"
 			(at 190.5 112.395 0)
 			(effects
@@
 			(project "gdp"
 				(path "/95aff260-2720-4733-a81d-a7a2136fdd14/7e43dd6e-b5cb-462f-9bfd-3d0ee9fd8751"
-					(reference  "CK55")
+					(reference "CK55")
 					(unit 1)
 				)
@@
 		(dnp no)
 		(fields_autoplaced yes)
-		(property "Reference" "IC38"
-			(at 146.9741 67.31 0)
+		(property "Reference" "IC1"
+			(at 144.78 67.31 0)
 			(effects
 				(font
 					(size 1.27 1.27)
 				)
-				(justify left)
 			)
 		)
 		(property "Value" "74LS74"
-			(at 146.9741 69.85 0)
+			(at 144.78 69.85 0)
 			(effects
 				(font
 					(size 1.27 1.27)
 				)
-				(justify left)
 			)
 		)
@@
 			(project ""
 				(path "/95aff260-2720-4733-a81d-a7a2136fdd14/7e43dd6e-b5cb-462f-9bfd-3d0ee9fd8751"
-					(reference  "IC21")
+					(reference "IC1")
 					(unit 2)
 				)
@@
 		(dnp no)
 		(fields_autoplaced yes)
-		(property "Reference" "IC62"
+		(property "Reference" "IC12"
 			(at 113.9541 132.08 0)
 			(effects
@@
 			(project "gdp"
 				(path "/95aff260-2720-4733-a81d-a7a2136fdd14/7e43dd6e-b5cb-462f-9bfd-3d0ee9fd8751"
-					(reference  "IC12")
+					(reference "IC12")
 					(unit 1)
 				)
@@
 		(on_board yes)
 		(dnp no)
-		(property "Reference" "SH_2"
+		(property "Reference" "SH_5"
 			(at 180.34 39.37 0)
 			(effects
@@
 			(project "gdp"
 				(path "/95aff260-2720-4733-a81d-a7a2136fdd14/7e43dd6e-b5cb-462f-9bfd-3d0ee9fd8751"
-					(reference  "SH_5")
+					(reference "SH_5")
 					(unit 1)
 				)
@@
 		(on_board yes)
 		(dnp no)
-		(property "Reference" "R33"
+		(property "Reference" "R48"
 			(at 180.34 109.22 0)
 			(effects
@@
 			(project "gdp"
 				(path "/95aff260-2720-4733-a81d-a7a2136fdd14/7e43dd6e-b5cb-462f-9bfd-3d0ee9fd8751"
-					(reference  "R48")
+					(reference "R48")
 					(unit 1)
 				)
@@
 		(on_board yes)
 		(dnp no)
-		(property "Reference" "SH7"
+		(property "Reference" "SH11"
 			(at 102.87 38.1 0)
 			(effects
@@
 			(project "gdp"
 				(path "/95aff260-2720-4733-a81d-a7a2136fdd14/7e43dd6e-b5cb-462f-9bfd-3d0ee9fd8751"
-					(reference  "SH11")
+					(reference "SH11")
 					(unit 1)
 				)
@@
 		(on_board yes)
 		(dnp no)
-		(property "Reference" "IC63"
+		(property "Reference" "IC51"
 			(at 264.16 86.36 0)
 			(effects
@@
 			(project "gdp"
 				(path "/95aff260-2720-4733-a81d-a7a2136fdd14/7e43dd6e-b5cb-462f-9bfd-3d0ee9fd8751"
-					(reference  "IC51")
+					(reference "IC51")
 					(unit 7)
 				)
@@
 		(dnp no)
 		(fields_autoplaced yes)
-		(property "Reference" "IC65"
+		(property "Reference" "IC64"
 			(at 209.55 88.9 0)
 			(effects
@@
 			(project ""
 				(path "/95aff260-2720-4733-a81d-a7a2136fdd14/7e43dd6e-b5cb-462f-9bfd-3d0ee9fd8751"
-					(reference  "IC64")
+					(reference "IC64")
 					(unit 2)
 				)
@@
 		(dnp no)
 		(fields_autoplaced yes)
-		(property "Reference" "IC63"
+		(property "Reference" "IC51"
 			(at 161.29 36.83 0)
 			(effects
@@
 			(project "gdp"
 				(path "/95aff260-2720-4733-a81d-a7a2136fdd14/7e43dd6e-b5cb-462f-9bfd-3d0ee9fd8751"
-					(reference  "IC51")
+					(reference "IC51")
 					(unit 1)
 				)
@@
 		(on_board yes)
 		(dnp no)
-		(property "Reference" "IC64"
+		(property "Reference" "IC66"
 			(at 252.73 86.36 0)
 			(effects
@@
 			(project "gdp"
 				(path "/95aff260-2720-4733-a81d-a7a2136fdd14/7e43dd6e-b5cb-462f-9bfd-3d0ee9fd8751"
-					(reference  "IC66")
+					(reference "IC66")
 					(unit 5)
 				)

Commit message: Placing footprints...
Parts:
- R17, R27, R48: footprint Resistor_THT:R_Axial_DIN0207_L6.3mm_D2.5mm_P7.62mm_Horizontal -> Resistor_THT:R_Axial_DIN0207_L6.3mm_D2.5mm_P10.16mm_Horizontal
Changed lines of the file:
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@@
 			)
 		)
-		(property "Footprint" "Resistor_THT:R_Axial_DIN0207_L6.3mm_D2.5mm_P7.62mm_Horizontal"
+		(property "Footprint" "Resistor_THT:R_Axial_DIN0207_L6.3mm_D2.5mm_P10.16mm_Horizontal"
 			(at 92.202 165.1 90)
 			(effects
@@
 			)
 		)
-		(property "Footprint" "Resistor_THT:R_Axial_DIN0207_L6.3mm_D2.5mm_P7.62mm_Horizontal"
+		(property "Footprint" "Resistor_THT:R_Axial_DIN0207_L6.3mm_D2.5mm_P10.16mm_Horizontal"
 			(at 142.24 43.942 90)
 			(effects
@@
 			)
 		)
-		(property "Footprint" "Resistor_THT:R_Axial_DIN0207_L6.3mm_D2.5mm_P7.62mm_Horizontal"
+		(property "Footprint" "Resistor_THT:R_Axial_DIN0207_L6.3mm_D2.5mm_P10.16mm_Horizontal"
 			(at 179.07 106.172 90)
 			(effects

Commit message: Maps footprints PCB -> sch
Parts:
- R27: footprint Resistor_THT:R_Axial_DIN0207_L6.3mm_D2.5mm_P10.16mm_Horizontal -> GDP:R_XL
Changed lines of the file:
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@@
 			)
 		)
-		(property "Footprint" "Resistor_THT:R_Axial_DIN0207_L6.3mm_D2.5mm_P10.16mm_Horizontal"
+		(property "Footprint" "GDP:R_XL"
 			(at 142.24 43.942 90)
 			(effects

Commit message: Fixes footprint references in sch
Parts:
- R17: footprint Resistor_THT:R_Axial_DIN0207_L6.3mm_D2.5mm_P10.16mm_Horizontal -> GDP:R_XL
Changed lines of the file:
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@@
 			)
 		)
-		(property "Footprint" "Resistor_THT:R_Axial_DIN0207_L6.3mm_D2.5mm_P10.16mm_Horizontal"
+		(property "Footprint" "GDP:R_XL"
 			(at 92.202 165.1 90)
 			(effects

Commit message: Re-annotates symbols
Parts:
- renumbered IC72 to IC1
Changed lines of the file:
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@@
 		(on_board yes)
 		(dnp no)
-		(property "Reference" "IC72"
+		(property "Reference" "IC1"
 			(at 252.73 52.07 0)
 			(effects
@@
 			(project "gdp"
 				(path "/95aff260-2720-4733-a81d-a7a2136fdd14/7e43dd6e-b5cb-462f-9bfd-3d0ee9fd8751"
-					(reference "IC72")
+					(reference "IC1")
 					(unit 3)
 				)

Commit message: Fixes footprints R34 R27
Parts:
- R27: footprint GDP:R_XL -> GDP:R_XL_narrow
Changed lines of the file:
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@@
 			)
 		)
-		(property "Footprint" "GDP:R_XL"
+		(property "Footprint" "GDP:R_XL_narrow"
 			(at 142.24 43.942 90)
 			(effects

Commit message: Fixes resistor footprints
Connections:
- net ~{CRH} renamed ~{CHR}
- net ~{CRL} renamed ~{CLR}
Changed lines of the file:
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@@
 		)
 	)
-	(global_label "~{CRH}"
+	(global_label "~{CHR}"
 		(shape output)
 		(at 133.35 158.75 0)
@@
 		)
 	)
-	(global_label "~{CRL}"
+	(global_label "~{CLR}"
 		(shape output)
 		(at 133.35 156.21 0)
