File: gdp/12.kicad_sch (KiCad schematic)
At the start: 19 parts, among them IC1 74LS74, IC12 PAL16R4, IC51 74LS14, IC64 74LS123, IC66 74S00, IC71 74LS04

Commit message: Fixes SH ref
Parts:
- renumbered SH_5 to SH12, SH_4 to SH6
Changed lines of the file:
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@@
 		(on_board yes)
 		(dnp no)
-		(property "Reference" "SH_4"
+		(property "Reference" "SH6"
 			(at 180.34 31.75 0)
 			(effects
@@
 			(project "gdp"
 				(path "/95aff260-2720-4733-a81d-a7a2136fdd14/7e43dd6e-b5cb-462f-9bfd-3d0ee9fd8751"
-					(reference "SH_4")
+					(reference "SH6")
 					(unit 1)
 				)
@@
 		(on_board yes)
 		(dnp no)
-		(property "Reference" "SH_5"
+		(property "Reference" "SH12"
 			(at 180.34 39.37 0)
 			(effects
@@
 			(project "gdp"
 				(path "/95aff260-2720-4733-a81d-a7a2136fdd14/7e43dd6e-b5cb-462f-9bfd-3d0ee9fd8751"
-					(reference "SH_5")
-					(unit 1)
-				)
+					(reference "SH12")
+					(unit 1)
+				)

Commit message: Adds decoupling capacitors
Parts:
- CK50: value 10U -> U10
Changed lines of the file:
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@@
 			)
 		)
-		(property "Value" "10U"
+		(property "Value" "U10"
 			(at 154.305 53.34 0)
 			(effects

Commit message: Fixes "CA0" issue in schematics
Changed lines of the file:
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@@
 (kicad_sch
-	(version 20231120)
+	(version 20250114)
 	(generator "eeschema")
-	(generator_version "8.0")
+	(generator_version "9.0")
 	(paper "A4")
 	(title_block
