File: gdp/14.kicad_sch (KiCad schematic)
At the start: 16 parts, among them IC63 74LS14, IC64 74S00, IC65 74LS123, IC66 74LS74, IC67 74LS04, IC69 74LS163, IC70 74LS00

Commit message: Fixes refs
Parts:
- renumbered CK8 to CK52, CK7 to CK62, CK6 to CK63, IC63 to IC51, IC70 to IC52, IC69 to IC61, IC67 to IC63, IC65 to IC64, IC64 to IC66, IC66 to IC72, R53 to R28, R52 to R34, R54 to R51, R51 to R54
Changed lines of the file:
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@@
 		(dnp no)
 		(fields_autoplaced yes)
-		(property "Reference" "IC67"
+		(property "Reference" "IC63"
 			(at 120.65 41.91 0)
 			(effects
@@
 			(project "gdp"
 				(path "/95aff260-2720-4733-a81d-a7a2136fdd14/b2d99a56-eb50-41cd-94b5-019756774957"
-					(reference  "IC63")
+					(reference "IC63")
 					(unit 2)
 				)
@@
 		(dnp no)
 		(fields_autoplaced yes)
-		(property "Reference" "IC70"
+		(property "Reference" "IC52"
 			(at 189.2217 127 0)
 			(effects
@@
 			(project ""
 				(path "/95aff260-2720-4733-a81d-a7a2136fdd14/b2d99a56-eb50-41cd-94b5-019756774957"
-					(reference  "IC52")
+					(reference "IC52")
 					(unit 4)
 				)
@@
 		(on_board yes)
 		(dnp no)
-		(property "Reference" "R53"
+		(property "Reference" "R28"
 			(at 134.62 34.29 0)
 			(effects
@@
 			(project "gdp"
 				(path "/95aff260-2720-4733-a81d-a7a2136fdd14/b2d99a56-eb50-41cd-94b5-019756774957"
-					(reference  "R28")
+					(reference "R28")
 					(unit 1)
 				)
@@
 		(dnp no)
 		(fields_autoplaced yes)
-		(property "Reference" "IC70"
+		(property "Reference" "IC52"
 			(at 233.6717 132.08 0)
 			(effects
@@
 			(project "gdp"
 				(path "/95aff260-2720-4733-a81d-a7a2136fdd14/b2d99a56-eb50-41cd-94b5-019756774957"
-					(reference  "IC52")
+					(reference "IC52")
 					(unit 1)
 				)
@@
 		(dnp no)
 		(fields_autoplaced yes)
-		(property "Reference" "IC70"
+		(property "Reference" "IC52"
 			(at 189.2217 143.51 0)
 			(effects
@@
 			(project "gdp"
 				(path "/95aff260-2720-4733-a81d-a7a2136fdd14/b2d99a56-eb50-41cd-94b5-019756774957"
-					(reference  "IC52")
+					(reference "IC52")
 					(unit 2)
 				)
@@
 		(dnp no)
 		(fields_autoplaced yes)
-		(property "Reference" "IC64"
+		(property "Reference" "IC66"
 			(at 91.4317 86.36 0)
 			(effects
@@
 			(project ""
 				(path "/95aff260-2720-4733-a81d-a7a2136fdd14/b2d99a56-eb50-41cd-94b5-019756774957"
-					(reference  "IC66")
+					(reference "IC66")
 					(unit 2)
 				)
@@
 		(dnp no)
 		(fields_autoplaced yes)
-		(property "Reference" "IC67"
+		(property "Reference" "IC63"
 			(at 95.25 41.91 0)
 			(effects
@@
 			(project "gdp"
 				(path "/95aff260-2720-4733-a81d-a7a2136fdd14/b2d99a56-eb50-41cd-94b5-019756774957"
-					(reference  "IC63")
+					(reference "IC63")
 					(unit 1)
 				)
@@
 		(on_board yes)
 		(dnp no)
-		(property "Reference" "CK8"
+		(property "Reference" "CK52"
 			(at 125.095 119.38 0)
 			(effects
@@
 			(project "gdp"
 				(path "/95aff260-2720-4733-a81d-a7a2136fdd14/b2d99a56-eb50-41cd-94b5-019756774957"
-					(reference  "CK52")
+					(reference "CK52")
 					(unit 1)
 				)
@@
 		(on_board yes)
 		(dnp no)
-		(property "Reference" "IC70"
+		(property "Reference" "IC52"
 			(at 234.95 106.68 0)
 			(effects
@@
 			(project "gdp"
 				(path "/95aff260-2720-4733-a81d-a7a2136fdd14/b2d99a56-eb50-41cd-94b5-019756774957"
-					(reference  "IC52")
+					(reference "IC52")
 					(unit 5)
 				)
@@
 		(on_board yes)
 		(dnp no)
-		(property "Reference" "R52"
+		(property "Reference" "R34"
 			(at 116.84 119.38 0)
 			(effects
@@
 			(project "gdp"
 				(path "/95aff260-2720-4733-a81d-a7a2136fdd14/b2d99a56-eb50-41cd-94b5-019756774957"
-					(reference  "R34")
+					(reference "R34")
 					(unit 1)
 				)
@@
 		(on_board yes)
 		(dnp no)
-		(property "Reference" "R51"
+		(property "Reference" "R54"
 			(at 95.25 30.48 90)
 			(effects
@@
 			(project "gdp"
 				(path "/95aff260-2720-4733-a81d-a7a2136fdd14/b2d99a56-eb50-41cd-94b5-019756774957"
-					(reference  "R54")
+					(reference "R54")
 					(unit 1)
 				)
@@
 		(dnp no)
 		(fields_autoplaced yes)
-		(property "Reference" "IC67"
+		(property "Reference" "IC63"
 			(at 59.69 41.91 0)
 			(effects
@@
 			(project ""
 				(path "/95aff260-2720-4733-a81d-a7a2136fdd14/b2d99a56-eb50-41cd-94b5-019756774957"
-					(reference  "IC63")
+					(reference "IC63")
 					(unit 6)
 				)
@@
 		(dnp no)
 		(fields_autoplaced yes)
-		(property "Reference" "IC64"
+		(property "Reference" "IC66"
 			(at 91.4317 101.6 0)
 			(effects
@@
 			(project "gdp"
 				(path "/95aff260-2720-4733-a81d-a7a2136fdd14/b2d99a56-eb50-41cd-94b5-019756774957"
-					(reference  "IC66")
+					(reference "IC66")
 					(unit 4)
 				)
@@
 		(on_board yes)
 		(dnp no)
-		(property "Reference" "CK6"
+		(property "Reference" "CK63"
 			(at 52.705 68.58 0)
 			(effects
@@
 			(project "gdp"
 				(path "/95aff260-2720-4733-a81d-a7a2136fdd14/b2d99a56-eb50-41cd-94b5-019756774957"
-					(reference  "CK63")
+					(reference "CK63")
 					(unit 1)
 				)
@@
 		(on_board yes)
 		(dnp no)
-		(property "Reference" "R54"
+		(property "Reference" "R51"
 			(at 162.56 38.1 0)
 			(effects
@@
 			(project "gdp"
 				(path "/95aff260-2720-4733-a81d-a7a2136fdd14/b2d99a56-eb50-41cd-94b5-019756774957"
-					(reference  "R51")
+					(reference "R51")
 					(unit 1)
 				)
@@
 		(dnp no)
 		(fields_autoplaced yes)
-		(property "Reference" "IC70"
+		(property "Reference" "IC52"
 			(at 212.0817 129.54 0)
 			(effects
@@
 			(project "gdp"
 				(path "/95aff260-2720-4733-a81d-a7a2136fdd14/b2d99a56-eb50-41cd-94b5-019756774957"
-					(reference  "IC52")
+					(reference "IC52")
 					(unit 3)
 				)
@@
 		(dnp no)
 		(fields_autoplaced yes)
-		(property "Reference" "IC69"
+		(property "Reference" "IC61"
 			(at 185.0741 38.1 0)
 			(effects
@@
 			(project ""
 				(path "/95aff260-2720-4733-a81d-a7a2136fdd14/b2d99a56-eb50-41cd-94b5-019756774957"
-					(reference  "IC61")
+					(reference "IC61")
 					(unit 1)
 				)
@@
 		(dnp no)
 		(fields_autoplaced yes)
-		(property "Reference" "IC67"
+		(property "Reference" "IC63"
 			(at 165.1 129.54 0)
 			(effects
@@
 			(project ""
 				(path "/95aff260-2720-4733-a81d-a7a2136fdd14/b2d99a56-eb50-41cd-94b5-019756774957"
-					(reference  "IC63")
+					(reference "IC63")
 					(unit 5)
 				)
@@
 		(dnp no)
 		(fields_autoplaced yes)
-		(property "Reference" "IC64"
+		(property "Reference" "IC66"
 			(at 115.5617 93.98 0)
 			(effects
@@
 			(project "gdp"
 				(path "/95aff260-2720-4733-a81d-a7a2136fdd14/b2d99a56-eb50-41cd-94b5-019756774957"
-					(reference  "IC66")
+					(reference "IC66")
 					(unit 3)
 				)
@@
 		(dnp no)
 		(fields_autoplaced yes)
-		(property "Reference" "IC63"
+		(property "Reference" "IC51"
 			(at 171.45 104.14 0)
 			(effects
@@
 			(project ""
 				(path "/95aff260-2720-4733-a81d-a7a2136fdd14/b2d99a56-eb50-41cd-94b5-019756774957"
-					(reference  "IC51")
+					(reference "IC51")
 					(unit 4)
 				)
@@
 		(dnp no)
 		(fields_autoplaced yes)
-		(property "Reference" "IC66"
+		(property "Reference" "IC72"
 			(at 59.69 95.25 0)
 			(effects
@@
 			(project "gdp"
 				(path "/95aff260-2720-4733-a81d-a7a2136fdd14/b2d99a56-eb50-41cd-94b5-019756774957"
-					(reference  "IC72")
+					(reference "IC72")
 					(unit 1)
 				)
@@
 		(on_board yes)
 		(dnp no)
-		(property "Reference" "CK7"
+		(property "Reference" "CK62"
 			(at 77.47 45.085 90)
 			(effects
@@
 			(project "gdp"
 				(path "/95aff260-2720-4733-a81d-a7a2136fdd14/b2d99a56-eb50-41cd-94b5-019756774957"
-					(reference  "CK62")
+					(reference "CK62")
 					(unit 1)
 				)
@@
 		(dnp no)
 		(fields_autoplaced yes)
-		(property "Reference" "IC66"
+		(property "Reference" "IC72"
 			(at 214.63 38.1 0)
 			(effects
@@
 			(project ""
 				(path "/95aff260-2720-4733-a81d-a7a2136fdd14/b2d99a56-eb50-41cd-94b5-019756774957"
-					(reference  "IC72")
+					(reference "IC72")
 					(unit 2)
 				)
@@
 		(dnp no)
 		(fields_autoplaced yes)
-		(property "Reference" "IC67"
+		(property "Reference" "IC63"
 			(at 146.05 41.91 0)
 			(effects
@@
 			(project "gdp"
 				(path "/95aff260-2720-4733-a81d-a7a2136fdd14/b2d99a56-eb50-41cd-94b5-019756774957"
-					(reference  "IC63")
+					(reference "IC63")
 					(unit 4)
 				)
@@
 		(dnp no)
 		(fields_autoplaced yes)
-		(property "Reference" "IC65"
+		(property "Reference" "IC64"
 			(at 146.05 93.98 0)
 			(effects
@@
 			(project ""
 				(path "/95aff260-2720-4733-a81d-a7a2136fdd14/b2d99a56-eb50-41cd-94b5-019756774957"
-					(reference  "IC64")
+					(reference "IC64")
 					(unit 1)
 				)

Commit message: Placing footprints...
Parts:
- R28, R34, R50, R51, R54: footprint Resistor_THT:R_Axial_DIN0207_L6.3mm_D2.5mm_P7.62mm_Horizontal -> Resistor_THT:R_Axial_DIN0207_L6.3mm_D2.5mm_P10.16mm_Horizontal
Changed lines of the file:
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@@
 			)
 		)
-		(property "Footprint" "Resistor_THT:R_Axial_DIN0207_L6.3mm_D2.5mm_P7.62mm_Horizontal"
+		(property "Footprint" "Resistor_THT:R_Axial_DIN0207_L6.3mm_D2.5mm_P10.16mm_Horizontal"
 			(at 131.572 35.56 90)
 			(effects
@@
 			)
 		)
-		(property "Footprint" "Resistor_THT:R_Axial_DIN0207_L6.3mm_D2.5mm_P7.62mm_Horizontal"
+		(property "Footprint" "Resistor_THT:R_Axial_DIN0207_L6.3mm_D2.5mm_P10.16mm_Horizontal"
 			(at 113.792 120.65 90)
 			(effects
@@
 			)
 		)
-		(property "Footprint" "Resistor_THT:R_Axial_DIN0207_L6.3mm_D2.5mm_P7.62mm_Horizontal"
+		(property "Footprint" "Resistor_THT:R_Axial_DIN0207_L6.3mm_D2.5mm_P10.16mm_Horizontal"
 			(at 95.25 37.338 90)
 			(effects
@@
 			)
 		)
-		(property "Footprint" "Resistor_THT:R_Axial_DIN0207_L6.3mm_D2.5mm_P7.62mm_Horizontal"
+		(property "Footprint" "Resistor_THT:R_Axial_DIN0207_L6.3mm_D2.5mm_P10.16mm_Horizontal"
 			(at 59.69 37.338 90)
 			(effects
@@
 			)
 		)
-		(property "Footprint" "Resistor_THT:R_Axial_DIN0207_L6.3mm_D2.5mm_P7.62mm_Horizontal"
+		(property "Footprint" "Resistor_THT:R_Axial_DIN0207_L6.3mm_D2.5mm_P10.16mm_Horizontal"
 			(at 159.512 39.37 90)
 			(effects

Commit message: Maps footprints PCB -> sch
Parts:
- R28: footprint Resistor_THT:R_Axial_DIN0207_L6.3mm_D2.5mm_P10.16mm_Horizontal -> GDP:R_S
- R50: footprint Resistor_THT:R_Axial_DIN0207_L6.3mm_D2.5mm_P10.16mm_Horizontal -> GDP:R_XL
Changed lines of the file:
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@@
 			)
 		)
-		(property "Footprint" "Resistor_THT:R_Axial_DIN0207_L6.3mm_D2.5mm_P10.16mm_Horizontal"
+		(property "Footprint" "GDP:R_S"
 			(at 131.572 35.56 90)
 			(effects
@@
 			)
 		)
-		(property "Footprint" "Resistor_THT:R_Axial_DIN0207_L6.3mm_D2.5mm_P10.16mm_Horizontal"
+		(property "Footprint" "GDP:R_XL"
 			(at 59.69 37.338 90)
 			(effects

Commit message: Fixes footprint references in sch
Parts:
- R34, R54: footprint Resistor_THT:R_Axial_DIN0207_L6.3mm_D2.5mm_P10.16mm_Horizontal -> GDP:R_XL
Changed lines of the file:
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@@
 			)
 		)
-		(property "Footprint" "Resistor_THT:R_Axial_DIN0207_L6.3mm_D2.5mm_P10.16mm_Horizontal"
+		(property "Footprint" "GDP:R_XL"
 			(at 113.792 120.65 90)
 			(effects
@@
 			)
 		)
-		(property "Footprint" "Resistor_THT:R_Axial_DIN0207_L6.3mm_D2.5mm_P10.16mm_Horizontal"
+		(property "Footprint" "GDP:R_XL"
 			(at 95.25 37.338 90)
 			(effects

Commit message: Schema fixes
Parts:
- renumbered IC72 to IC65
Changed lines of the file:
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@@
 		(dnp no)
 		(fields_autoplaced yes)
-		(property "Reference" "IC72"
+		(property "Reference" "IC65"
 			(at 214.63 38.1 0)
 			(effects
@@
 			(project ""
 				(path "/95aff260-2720-4733-a81d-a7a2136fdd14/b2d99a56-eb50-41cd-94b5-019756774957"
-					(reference "IC72")
+					(reference "IC65")
 					(unit 2)
 				)

Commit message: Re-annotates symbols
Parts:
- renumbered IC72 to IC65, IC63 to IC72
Changed lines of the file:
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@@
 		(dnp no)
 		(fields_autoplaced yes)
-		(property "Reference" "IC63"
+		(property "Reference" "IC72"
 			(at 120.65 41.91 0)
 			(effects
@@
 			(project "gdp"
 				(path "/95aff260-2720-4733-a81d-a7a2136fdd14/b2d99a56-eb50-41cd-94b5-019756774957"
-					(reference "IC63")
+					(reference "IC72")
 					(unit 2)
 				)
@@
 		(dnp no)
 		(fields_autoplaced yes)
-		(property "Reference" "IC63"
+		(property "Reference" "IC72"
 			(at 95.25 41.91 0)
 			(effects
@@
 			(project "gdp"
 				(path "/95aff260-2720-4733-a81d-a7a2136fdd14/b2d99a56-eb50-41cd-94b5-019756774957"
-					(reference "IC63")
+					(reference "IC72")
 					(unit 1)
 				)
@@
 		(dnp no)
 		(fields_autoplaced yes)
-		(property "Reference" "IC63"
+		(property "Reference" "IC72"
 			(at 59.69 41.91 0)
 			(effects
@@
 			(project ""
 				(path "/95aff260-2720-4733-a81d-a7a2136fdd14/b2d99a56-eb50-41cd-94b5-019756774957"
-					(reference "IC63")
+					(reference "IC72")
 					(unit 6)
 				)
@@
 		(dnp no)
 		(fields_autoplaced yes)
-		(property "Reference" "IC63"
+		(property "Reference" "IC72"
 			(at 165.1 129.54 0)
 			(effects
@@
 			(project ""
 				(path "/95aff260-2720-4733-a81d-a7a2136fdd14/b2d99a56-eb50-41cd-94b5-019756774957"
-					(reference "IC63")
+					(reference "IC72")
 					(unit 5)
 				)
@@
 		(dnp no)
 		(fields_autoplaced yes)
-		(property "Reference" "IC72"
+		(property "Reference" "IC65"
 			(at 59.69 95.25 0)
 			(effects
@@
 			(project "gdp"
 				(path "/95aff260-2720-4733-a81d-a7a2136fdd14/b2d99a56-eb50-41cd-94b5-019756774957"
-					(reference "IC72")
+					(reference "IC65")
 					(unit 1)
 				)
@@
 		(dnp no)
 		(fields_autoplaced yes)
-		(property "Reference" "IC63"
+		(property "Reference" "IC72"
 			(at 146.05 41.91 0)
 			(effects
@@
 			(project "gdp"
 				(path "/95aff260-2720-4733-a81d-a7a2136fdd14/b2d99a56-eb50-41cd-94b5-019756774957"
-					(reference "IC63")
+					(reference "IC72")
 					(unit 4)
 				)

Commit message: Fixes footprints R34 R27
Parts:
- R34: footprint GDP:R_XL -> GDP:R_XL_narrow
Changed lines of the file:
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@@
 			)
 		)
-		(property "Footprint" "GDP:R_XL"
+		(property "Footprint" "GDP:R_XL_narrow"
 			(at 113.792 120.65 90)
 			(effects
