File: gdp/9.kicad_sch (KiCad schematic)
At the start: 0 parts

Commit message: Adds pages 4, 7, 10 (still WIP)
Other:
- title: Partner GDP -> (none)
Changed lines of the file:
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@@
 (kicad_sch (version 20230121) (generator eeschema)
   (paper "A4")
-  (title_block
-    (title "Partner GDP")
-  )
 )

Commit message: Fixes Sheet 5
Other:
- company: (none) -> Oddbit Retro
- title: (none) -> PARTNER GDP: MEMORY
Changed lines of the file:
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@@
 	(generator_version "8.0")
 	(paper "A4")
+	(title_block
+		(title "PARTNER GDP: MEMORY")
+		(company "Oddbit Retro")
+		(comment 1 "NARISAL: MIHA GRČAR")
+	)
 )

Commit message: Adds Sheet 9
Parts:
- added IC19, IC20, IC44, IC45: HM6116, Package_DIP:DIP-28_W15.24mm, symbol Memory_EPROM:2764
Connections:
- new net +5V: IC19.24 (VCC), IC20.24 (VCC), IC44.24 (VCC), IC45.24 (VCC)
- new net ASCD0: IC19.9 (D0), IC20.9 (D0)
- new net ASCD1: IC19.10 (D1), IC20.10 (D1)
- new net ASCD2: IC19.11 (D2), IC20.11 (D2)
- new net ASCD3: IC19.13 (D3), IC20.13 (D3)
- new net ASCD4: IC19.14 (D4), IC20.14 (D4)
- new net ASCD5: IC19.15 (D5), IC20.15 (D5)
- new net ASCD6: IC19.16 (D6), IC20.16 (D6)
- new net ASCD7: IC19.17 (D7), IC20.17 (D7)
- new net ATTD0: IC44.9 (D0), IC45.9 (D0)
- new net ATTD1: IC44.10 (D1), IC45.10 (D1)
- new net ATTD2: IC44.11 (D2), IC45.11 (D2)
- new net ATTD3: IC44.13 (D3), IC45.13 (D3)
- new net ATTD4: IC44.14 (D4), IC45.14 (D4)
- new net ATTD5: IC44.15 (D5), IC45.15 (D5)
- new net ATTD6: IC44.16 (D6), IC45.16 (D6)
- new net ATTD7: IC44.17 (D7), IC45.17 (D7)
- new net DA0: IC19.8 (A0), IC20.8 (A0), IC44.8 (A0), IC45.8 (A0)
- new net DA1: IC19.7 (A1), IC20.7 (A1), IC44.7 (A1), IC45.7 (A1)
- new net DA10: IC19.19 (A10), IC20.19 (A10), IC44.19 (A10), IC45.19 (A10)
- new net DA2: IC19.6 (A2), IC20.6 (A2), IC44.6 (A2), IC45.6 (A2)
- new net DA3: IC19.5 (A3), IC20.5 (A3), IC44.5 (A3), IC45.5 (A3)
- new net DA4: IC19.4 (A4), IC20.4 (A4), IC44.4 (A4), IC45.4 (A4)
- new net DA5: IC19.3 (A5), IC20.3 (A5), IC44.3 (A5), IC45.3 (A5)
- new net DA6: IC19.2 (A6), IC20.2 (A6), IC44.2 (A6), IC45.2 (A6)
- new net DA7: IC19.1 (A7), IC20.1 (A7), IC44.1 (A7), IC45.1 (A7)
- new net DA8: IC19.23 (A8), IC20.23 (A8), IC44.23 (A8), IC45.23 (A8)
- new net DA9: IC19.22 (A9), IC20.22 (A9), IC44.22 (A9), IC45.22 (A9)
- new net GNDD: IC19.12 (GND), IC19.20 (~{OE}), IC20.12 (GND), IC20.20 (~{OE}), IC44.12 (GND), IC44.20 (~{OE}), IC45.12 (GND), IC45.20 (~{OE})
- new net ~{CHR}: IC19.18 (~{CS}), IC44.18 (~{CS})
- new net ~{CLR}: IC20.18 (~{CS}), IC45.18 (~{CS})
- new net ~{WDB}: IC19.21 (~{WE}), IC20.21 (~{WE}), IC44.21 (~{WE}), IC45.21 (~{WE})
Other:
- title: PARTNER GDP: MEMORY -> PARTNER GDP: AVDC MEMORY

Commit message: Initial footprint assignment
Parts:
- IC50: renamed from IC45; footprint Package_DIP:DIP-28_W15.24mm -> Package_DIP:DIP-24_W15.24mm
- IC51: renamed from IC20; footprint Package_DIP:DIP-28_W15.24mm -> Package_DIP:DIP-24_W15.24mm
- IC52: renamed from IC44; footprint Package_DIP:DIP-28_W15.24mm -> Package_DIP:DIP-24_W15.24mm
- IC53: renamed from IC19; footprint Package_DIP:DIP-28_W15.24mm -> Package_DIP:DIP-24_W15.24mm
Changed lines of the file:
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@@
 		(dnp no)
 		(fields_autoplaced yes)
-		(property "Reference" "#PWR0135"
+		(property "Reference" "#PWR0123"
 			(at 102.87 151.13 0)
 			(effects
@@
 			(project "gdp"
 				(path "/95aff260-2720-4733-a81d-a7a2136fdd14/5420fe53-9172-4320-b1ae-7476e0c7581b"
-					(reference "#PWR0135")
+					(reference "#PWR0123")
 					(unit 1)
 				)
@@
 		(on_board yes)
 		(dnp no)
-		(property "Reference" "#PWR0143"
+		(property "Reference" "#PWR0128"
 			(at 184.15 100.33 0)
 			(effects
@@
 			(project "gdp"
 				(path "/95aff260-2720-4733-a81d-a7a2136fdd14/5420fe53-9172-4320-b1ae-7476e0c7581b"
-					(reference "#PWR0143")
+					(reference "#PWR0128")
 					(unit 1)
 				)
@@
 		(on_board yes)
 		(dnp no)
-		(property "Reference" "IC44"
+		(property "Reference" "IC52"
 			(at 184.15 50.165 0)
 			(effects
@@
 			)
 		)
-		(property "Footprint" "Package_DIP:DIP-28_W15.24mm"
+		(property "Footprint" "Package_DIP:DIP-24_W15.24mm"
 			(at 184.15 58.42 0)
 			(effects
@@
 			)
 		)
-		(property "Datasheet" "https://downloads.reactivemicro.com/Electronics/ROM/2764%20EPROM.pdf"
+		(property "Datasheet" "N/A"
 			(at 184.15 58.42 0)
 			(effects
@@
 			)
 		)
-		(property "Description" ""
+		(property "Description" "N/A"
 			(at 184.15 62.23 0)
 			(effects
@@
 			(project "gdp"
 				(path "/95aff260-2720-4733-a81d-a7a2136fdd14/5420fe53-9172-4320-b1ae-7476e0c7581b"
-					(reference "IC44")
+					(reference "IC52")
 					(unit 1)
 				)
@@
 		(dnp no)
 		(fields_autoplaced yes)
-		(property "Reference" "#PWR0141"
+		(property "Reference" "#PWR0118"
 			(at 90.17 92.71 0)
 			(effects
@@
 			(project "gdp"
 				(path "/95aff260-2720-4733-a81d-a7a2136fdd14/5420fe53-9172-4320-b1ae-7476e0c7581b"
-					(reference "#PWR0141")
+					(reference "#PWR0118")
 					(unit 1)
 				)
@@
 		(dnp no)
 		(fields_autoplaced yes)
-		(property "Reference" "#PWR0138"
+		(property "Reference" "#PWR0129"
 			(at 184.15 151.13 0)
 			(effects
@@
 			(project "gdp"
 				(path "/95aff260-2720-4733-a81d-a7a2136fdd14/5420fe53-9172-4320-b1ae-7476e0c7581b"
-					(reference "#PWR0138")
+					(reference "#PWR0129")
 					(unit 1)
 				)
@@
 		(on_board yes)
 		(dnp no)
-		(property "Reference" "#PWR0145"
+		(property "Reference" "#PWR0120"
 			(at 102.87 41.91 0)
 			(effects
@@
 			(project "gdp"
 				(path "/95aff260-2720-4733-a81d-a7a2136fdd14/5420fe53-9172-4320-b1ae-7476e0c7581b"
-					(reference "#PWR0145")
+					(reference "#PWR0120")
 					(unit 1)
 				)
@@
 		(dnp no)
 		(fields_autoplaced yes)
-		(property "Reference" "#PWR0136"
+		(property "Reference" "#PWR0119"
 			(at 90.17 151.13 0)
 			(effects
@@
 			(project "gdp"
 				(path "/95aff260-2720-4733-a81d-a7a2136fdd14/5420fe53-9172-4320-b1ae-7476e0c7581b"
-					(reference "#PWR0136")
+					(reference "#PWR0119")
 					(unit 1)
 				)
@@
 		(dnp no)
 		(fields_autoplaced yes)
-		(property "Reference" "#PWR0137"
+		(property "Reference" "#PWR0125"
 			(at 171.45 151.13 0)
 			(effects
@@
 			(project "gdp"
 				(path "/95aff260-2720-4733-a81d-a7a2136fdd14/5420fe53-9172-4320-b1ae-7476e0c7581b"
-					(reference "#PWR0137")
+					(reference "#PWR0125")
 					(unit 1)
 				)
@@
 		(dnp no)
 		(fields_autoplaced yes)
-		(property "Reference" "#PWR0140"
+		(property "Reference" "#PWR0127"
 			(at 184.15 92.71 0)
 			(effects
@@
 			(project "gdp"
 				(path "/95aff260-2720-4733-a81d-a7a2136fdd14/5420fe53-9172-4320-b1ae-7476e0c7581b"
-					(reference "#PWR0140")
+					(reference "#PWR0127")
 					(unit 1)
 				)
@@
 		(dnp no)
 		(fields_autoplaced yes)
-		(property "Reference" "#PWR0142"
+		(property "Reference" "#PWR0121"
 			(at 102.87 92.71 0)
 			(effects
@@
 			(project "gdp"
 				(path "/95aff260-2720-4733-a81d-a7a2136fdd14/5420fe53-9172-4320-b1ae-7476e0c7581b"
-					(reference "#PWR0142")
+					(reference "#PWR0121")
 					(unit 1)
 				)
@@
 		(on_board yes)
 		(dnp no)
-		(property "Reference" "#PWR0144"
+		(property "Reference" "#PWR0126"
 			(at 184.15 41.91 0)
 			(effects
@@
 			(project "gdp"
 				(path "/95aff260-2720-4733-a81d-a7a2136fdd14/5420fe53-9172-4320-b1ae-7476e0c7581b"
-					(reference "#PWR0144")
+					(reference "#PWR0126")
 					(unit 1)
 				)
@@
 		(on_board yes)
 		(dnp no)
-		(property "Reference" "IC19"
+		(property "Reference" "IC53"
 			(at 184.15 108.585 0)
 			(effects
@@
 			)
 		)
-		(property "Footprint" "Package_DIP:DIP-28_W15.24mm"
+		(property "Footprint" "Package_DIP:DIP-24_W15.24mm"
 			(at 184.15 116.84 0)
 			(effects
@@
 			)
 		)
-		(property "Datasheet" "https://downloads.reactivemicro.com/Electronics/ROM/2764%20EPROM.pdf"
+		(property "Datasheet" "N/A"
 			(at 184.15 116.84 0)
 			(effects
@@
 			)
 		)
-		(property "Description" ""
+		(property "Description" "N/A"
 			(at 184.15 120.65 0)
 			(effects
@@
 			(project "gdp"
 				(path "/95aff260-2720-4733-a81d-a7a2136fdd14/5420fe53-9172-4320-b1ae-7476e0c7581b"
-					(reference "IC19")
+					(reference "IC53")
 					(unit 1)
 				)
@@
 		(on_board yes)
 		(dnp no)
-		(property "Reference" "IC20"
+		(property "Reference" "IC51"
 			(at 102.87 108.585 0)
 			(effects
@@
 			)
 		)
-		(property "Footprint" "Package_DIP:DIP-28_W15.24mm"
+		(property "Footprint" "Package_DIP:DIP-24_W15.24mm"
 			(at 102.87 116.84 0)
 			(effects
@@
 			)
 		)
-		(property "Datasheet" "https://downloads.reactivemicro.com/Electronics/ROM/2764%20EPROM.pdf"
+		(property "Datasheet" "N/A"
 			(at 102.87 116.84 0)
 			(effects
@@
 			)
 		)
-		(property "Description" ""
+		(property "Description" "N/A"
 			(at 102.87 120.65 0)
 			(effects
@@
 			(project "gdp"
 				(path "/95aff260-2720-4733-a81d-a7a2136fdd14/5420fe53-9172-4320-b1ae-7476e0c7581b"
-					(reference "IC20")
+					(reference "IC51")
 					(unit 1)
 				)
@@
 		(on_board yes)
 		(dnp no)
-		(property "Reference" "#PWR0146"
+		(property "Reference" "#PWR0122"
 			(at 102.87 100.33 0)
 			(effects
@@
 			(project "gdp"
 				(path "/95aff260-2720-4733-a81d-a7a2136fdd14/5420fe53-9172-4320-b1ae-7476e0c7581b"
-					(reference "#PWR0146")
+					(reference "#PWR0122")
 					(unit 1)
 				)
@@
 		(on_board yes)
 		(dnp no)
-		(property "Reference" "IC45"
+		(property "Reference" "IC50"
 			(at 102.87 50.165 0)
 			(effects
@@
 			)
 		)
-		(property "Footprint" "Package_DIP:DIP-28_W15.24mm"
+		(property "Footprint" "Package_DIP:DIP-24_W15.24mm"
 			(at 102.87 58.42 0)
 			(effects
@@
 			)
 		)
-		(property "Datasheet" "https://downloads.reactivemicro.com/Electronics/ROM/2764%20EPROM.pdf"
+		(property "Datasheet" "N/A"
 			(at 102.87 58.42 0)
 			(effects
@@
 			)
 		)
-		(property "Description" ""
+		(property "Description" "N/A"
 			(at 102.87 62.23 0)
 			(effects
@@
 			(project "gdp"
 				(path "/95aff260-2720-4733-a81d-a7a2136fdd14/5420fe53-9172-4320-b1ae-7476e0c7581b"
-					(reference "IC45")
+					(reference "IC50")
 					(unit 1)
 				)
@@
 		(dnp no)
 		(fields_autoplaced yes)
-		(property "Reference" "#PWR0139"
+		(property "Reference" "#PWR0124"
 			(at 171.45 92.71 0)
 			(effects
@@
 			(project "gdp"
 				(path "/95aff260-2720-4733-a81d-a7a2136fdd14/5420fe53-9172-4320-b1ae-7476e0c7581b"
-					(reference "#PWR0139")
-					(unit 1)
-				)
+					(reference "#PWR0124")
+					(unit 1)
+				)
