File: gdp/9.kicad_sch (KiCad schematic)
At the start: 4 parts, among them IC50 HM6116, IC51 HM6116, IC52 HM6116, IC53 HM6116

Commit message: Fixes refs
Parts:
- renumbered IC53 to IC19, IC51 to IC20, IC52 to IC44, IC50 to IC45
Changed lines of the file:
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@@
 		(on_board yes)
 		(dnp no)
-		(property "Reference" "IC52"
+		(property "Reference" "IC44"
 			(at 184.15 50.165 0)
 			(effects
@@
 			(project "gdp"
 				(path "/95aff260-2720-4733-a81d-a7a2136fdd14/5420fe53-9172-4320-b1ae-7476e0c7581b"
-					(reference  "IC44")
+					(reference "IC44")
 					(unit 1)
 				)
@@
 		(on_board yes)
 		(dnp no)
-		(property "Reference" "IC53"
+		(property "Reference" "IC19"
 			(at 184.15 108.585 0)
 			(effects
@@
 			(project "gdp"
 				(path "/95aff260-2720-4733-a81d-a7a2136fdd14/5420fe53-9172-4320-b1ae-7476e0c7581b"
-					(reference  "IC19")
+					(reference "IC19")
 					(unit 1)
 				)
@@
 		(on_board yes)
 		(dnp no)
-		(property "Reference" "IC51"
+		(property "Reference" "IC20"
 			(at 102.87 108.585 0)
 			(effects
@@
 			(project "gdp"
 				(path "/95aff260-2720-4733-a81d-a7a2136fdd14/5420fe53-9172-4320-b1ae-7476e0c7581b"
-					(reference  "IC20")
+					(reference "IC20")
 					(unit 1)
 				)
@@
 		(on_board yes)
 		(dnp no)
-		(property "Reference" "IC50"
+		(property "Reference" "IC45"
 			(at 102.87 50.165 0)
 			(effects
@@
 			(project "gdp"
 				(path "/95aff260-2720-4733-a81d-a7a2136fdd14/5420fe53-9172-4320-b1ae-7476e0c7581b"
-					(reference  "IC45")
-					(unit 1)
-				)
+					(reference "IC45")
+					(unit 1)
+				)
