File: gdp/15.kicad_sch (KiCad schematic)
At the start: 55 parts

Commit message: Adds R55 & R56
Parts:
- added R55, R56: 2K2, GDP:R_XL, symbol Device:R
Connections:
- net GNDD: now also R55.2, R56.2
- new net ATTD6: R56.1
- new net ATTD7: R55.1
