File: gdp/15.kicad_sch (KiCad schematic)
At the start: 58 parts

Commit message: Got myself into a mess.... :(
Parts:
- added IC65: 74LS14, Package_DIP:DIP-14_W7.62mm, symbol 74xx:74LS14
Connections:
- no-connect marks 0 -> 4
Changed lines of the file:
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@@
 		(color 0 0 0 0)
+	)
+	(no_connect
+		(at 113.03 82.55)
+	)
+	(no_connect
+		(at 97.79 97.79)
+	)
+	(no_connect
+		(at 97.79 82.55)
+	)
+	(no_connect
+		(at 113.03 97.79)
 	)
 	(wire
@@
 	)
 	(symbol
+		(lib_id "74xx:74LS14")
+		(at 105.41 97.79 0)
+		(unit 5)
+		(exclude_from_sim no)
+		(in_bom yes)
+		(on_board yes)
+		(dnp no)
+		(fields_autoplaced yes)
+		(property "Reference" "IC65"
+			(at 105.41 88.9 0)
+			(effects
+				(font
+					(size 1.27 1.27)
+				)
+			)
+		)
+		(property "Value" "74LS14"
+			(at 105.41 91.44 0)
+			(effects
+				(font
+					(size 1.27 1.27)
+				)
+			)
+		)
+		(property "Footprint" "Package_DIP:DIP-14_W7.62mm"
+			(at 105.41 97.79 0)
+			(effects
+				(font
+					(size 1.27 1.27)
+				)
+				(hide yes)
+			)
+		)
+		(property "Datasheet" "N/A"
+			(at 105.41 97.79 0)
+			(effects
+				(font
+					(size 1.27 1.27)
+				)
+				(hide yes)
+			)
+		)
+		(property "Description" "N/A"
+			(at 105.41 97.79 0)
+			(effects
+				(font
+					(size 1.27 1.27)
+				)
+				(hide yes)
+			)
+		)
+		(pin "1"
+		)
+		(pin "3"
+		)
+		(pin "4"
+		)
+		(pin "5"
+		)
+		(pin "6"
+		)
+		(pin "8"
+		)
+		(pin "9"
+		)
+		(pin "2"
+		)
+		(pin "11"
+		)
+		(pin "12"
+		)
+		(pin "10"
+		)
+		(pin "7"
+		)
+		(pin "13"
+		)
+		(pin "14"
+		)
+		(instances
+			(project "gdp"
+				(path "/95aff260-2720-4733-a81d-a7a2136fdd14/44a9780b-71f6-40f0-9057-b92b2aeabcf0"
+					(reference "IC65")
+					(unit 5)
+				)
+			)
+		)
+	)
+	(symbol
 		(lib_id "Device:C_Small")
 		(at 35.56 93.98 90)
@@
 				)
 			)
+		)
+	)
+	(symbol
+		(lib_id "74xx:74LS14")
+		(at 105.41 82.55 0)
+		(unit 6)
+		(exclude_from_sim no)
+		(in_bom yes)
+		(on_board yes)
+		(dnp no)
+		(fields_autoplaced yes)
+		(property "Reference" "IC65"
+			(at 105.41 73.66 0)
+			(effects
+				(font
+					(size 1.27 1.27)
+				)
+			)
+		)
+		(property "Value" "74LS14"
+			(at 105.41 76.2 0)
+			(effects
+				(font
+					(size 1.27 1.27)
+				)
+			)
+		)
+		(property "Footprint" "Package_DIP:DIP-14_W7.62mm"
+			(at 105.41 82.55 0)
+			(effects
+				(font
+					(size 1.27 1.27)
+				)
+				(hide yes)
+			)
+		)
+		(property "Datasheet" "N/A"
+			(at 105.41 82.55 0)
+			(effects
+				(font
+					(size 1.27 1.27)
+				)
+				(hide yes)
+			)
+		)
+		(property "Description" "N/A"
+			(at 105.41 82.55 0)
+			(effects
+				(font
+					(size 1.27 1.27)
+				)
+				(hide yes)
+			)
+		)
+		(pin "1"
+		)
+		(pin "3"
+		)
+		(pin "4"
+		)
+		(pin "5"
+		)
+		(pin "6"
+		)
+		(pin "8"
+		)
+		(pin "9"
+		)
+		(pin "2"
+		)
+		(pin "11"
+		)
+		(pin "12"
+		)
+		(pin "10"
+		)
+		(pin "7"
+		)
+		(pin "13"
+		)
+		(pin "14"
+		)
+		(instances
+			(project "gdp"
+				(path "/95aff260-2720-4733-a81d-a7a2136fdd14/44a9780b-71f6-40f0-9057-b92b2aeabcf0"
+					(reference "IC65")
+					(unit 6)
+				)
+			)

Commit message: Fixes unconnected pads
Parts:
- added IC11: 7406, Package_DIP:DIP-14_W7.62mm, symbol 74xx:74LS06
- added IC71: 74LS04, Package_DIP:DIP-14_W7.62mm, symbol 74xx:74LS04
- renumbered IC65 to IC51
Connections:
- no-connect marks 4 -> 12

Commit message: Some polishing
Connections:
- no-connect marks 12 -> 18
Changed lines of the file:
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@@
+	)
+	(no_connect
+		(at 97.79 132.08)
+	)
+	(no_connect
+		(at 97.79 116.84)
 	)
 	(no_connect
@@
 	)
 	(no_connect
+		(at 97.79 147.32)
+	)
+	(no_connect
 		(at 72.39 105.41)
+	)
+	(no_connect
+		(at 113.03 147.32)
 	)
 	(no_connect
@@
 	)
 	(no_connect
+		(at 113.03 132.08)
+	)
+	(no_connect
 		(at 72.39 118.11)
 	)
 	(no_connect
+		(at 113.03 116.84)
+	)
+	(no_connect
